File: moteurs_brushless_elec/PCB/power_part.sch (KiCad schematic (older format))
At the start: 20 parts, among them J3 FAN, U4 B_Plug_5mm, U5 LM317_SOT223, U6 LM317_SOT223

Commit message: routing...
Parts:
- U5, U6: footprint TO_SOT_Packages_THT:TO-220_Horizontal -> TO_SOT_Packages_SMD:SOT-223-3Lead_TabPin2
Changed lines of the file:
@@
 $EndDescr
 $Comp
-L VCC #PWR038
+L VCC #PWR042
 U 1 1 5962E5D8
 P 4650 2300
-F 0 "#PWR038" H 4650 2150 50  0001 C CNN
+F 0 "#PWR042" H 4650 2150 50  0001 C CNN
 F 1 "VCC" H 4650 2450 50  0000 C CNN
 F 2 "" H 4650 2300 50  0001 C CNN
@@
 $EndComp
 $Comp
-L +3.3V #PWR039
+L +3.3V #PWR043
 U 1 1 5962E5EC
 P 10450 2450
-F 0 "#PWR039" H 10450 2300 50  0001 C CNN
+F 0 "#PWR043" H 10450 2300 50  0001 C CNN
 F 1 "+3.3V" H 10450 2590 50  0000 C CNN
 F 2 "" H 10450 2450 50  0001 C CNN
@@
 $EndComp
 $Comp
-L GND #PWR040
+L GND #PWR044
 U 1 1 5962E732
 P 3650 2900
-F 0 "#PWR040" H 3650 2650 50  0001 C CNN
+F 0 "#PWR044" H 3650 2650 50  0001 C CNN
 F 1 "GND" H 3650 2750 50  0000 C CNN
 F 2 "" H 3650 2900 50  0001 C CNN
@@
 $EndComp
 $Comp
-L GND #PWR041
+L GND #PWR045
 U 1 1 5962E829
 P 4250 3000
-F 0 "#PWR041" H 4250 2750 50  0001 C CNN
+F 0 "#PWR045" H 4250 2750 50  0001 C CNN
 F 1 "GND" H 4250 2850 50  0000 C CNN
 F 2 "" H 4250 3000 50  0001 C CNN
@@
 	3650 2650 3650 2900
 $Comp
-L PWR_FLAG #FLG042
+L PWR_FLAG #FLG046
 U 1 1 5962EB73
 P 4500 2400
-F 0 "#FLG042" H 4500 2475 50  0001 C CNN
+F 0 "#FLG046" H 4500 2475 50  0001 C CNN
 F 1 "PWR_FLAG" H 4500 2550 50  0000 C CNN
 F 2 "" H 4500 2400 50  0001 C CNN
@@
 $EndComp
 $Comp
-L PWR_FLAG #FLG043
+L PWR_FLAG #FLG047
 U 1 1 5962EBA1
 P 3800 2850
-F 0 "#FLG043" H 3800 2925 50  0001 C CNN
+F 0 "#FLG047" H 3800 2925 50  0001 C CNN
 F 1 "PWR_FLAG" H 3800 3000 50  0000 C CNN
 F 2 "" H 3800 2850 50  0001 C CNN
@@
 Connection ~ 3650 2850
 $Comp
-L +5V #PWR044
+L +5V #PWR048
 U 1 1 5962ECD4
 P 7900 2450
-F 0 "#PWR044" H 7900 2300 50  0001 C CNN
+F 0 "#PWR048" H 7900 2300 50  0001 C CNN
 F 1 "+5V" H 7900 2590 50  0000 C CNN
 F 2 "" H 7900 2450 50  0001 C CNN
@@
 F 0 "U5" H 7000 3000 50  0000 C CNN
 F 1 "LM317_SOT223" H 7050 2450 50  0000 L CNN
-F 2 "TO_SOT_Packages_THT:TO-220_Horizontal" H 7000 2700 50  0001 C CNN
+F 2 "TO_SOT_Packages_SMD:SOT-223-3Lead_TabPin2" H 7000 2700 50  0001 C CNN
 F 3 "" H 7000 2700 50  0001 C CNN
 	1    7000 2700
@@
 F 0 "U6" H 9650 2950 50  0000 C CNN
 F 1 "LM317_SOT223" H 9700 2400 50  0000 L CNN
-F 2 "TO_SOT_Packages_THT:TO-220_Horizontal" H 9650 2650 50  0001 C CNN
+F 2 "TO_SOT_Packages_SMD:SOT-223-3Lead_TabPin2" H 9650 2650 50  0001 C CNN
 F 3 "" H 9650 2650 50  0001 C CNN
 	1    9650 2650
@@
 $EndComp
 $Comp
-L VCC #PWR045
+L VCC #PWR049
 U 1 1 5962F11A
 P 6450 2450
-F 0 "#PWR045" H 6450 2300 50  0001 C CNN
+F 0 "#PWR049" H 6450 2300 50  0001 C CNN
 F 1 "VCC" H 6450 2600 50  0000 C CNN
 F 2 "" H 6450 2450 50  0001 C CNN
@@
 $EndComp
 $Comp
-L VCC #PWR046
+L VCC #PWR050
 U 1 1 5962F138
 P 9050 2450
-F 0 "#PWR046" H 9050 2300 50  0001 C CNN
+F 0 "#PWR050" H 9050 2300 50  0001 C CNN
 F 1 "VCC" H 9050 2600 50  0000 C CNN
 F 2 "" H 9050 2450 50  0001 C CNN
@@
 $EndComp
 $Comp
-L GND #PWR047
+L GND #PWR051
 U 1 1 5962F3CB
 P 7000 3600
-F 0 "#PWR047" H 7000 3350 50  0001 C CNN
+F 0 "#PWR051" H 7000 3350 50  0001 C CNN
 F 1 "GND" H 7000 3450 50  0000 C CNN
 F 2 "" H 7000 3600 50  0001 C CNN
@@
 $EndComp
 $Comp
-L GND #PWR048
+L GND #PWR052
 U 1 1 5962F3F1
 P 9650 3600
-F 0 "#PWR048" H 9650 3350 50  0001 C CNN
+F 0 "#PWR052" H 9650 3350 50  0001 C CNN
 F 1 "GND" H 9650 3450 50  0000 C CNN
 F 2 "" H 9650 3600 50  0001 C CNN
@@
 $EndComp
 $Comp
-L GND #PWR049
+L GND #PWR053
 U 1 1 5963063C
 P 5450 3000
-F 0 "#PWR049" H 5450 2750 50  0001 C CNN
+F 0 "#PWR053" H 5450 2750 50  0001 C CNN
 F 1 "GND" H 5450 2850 50  0000 C CNN
 F 2 "" H 5450 3000 50  0001 C CNN
@@
 $EndComp
 $Comp
-L GND #PWR050
+L GND #PWR054
 U 1 1 5963066E
 P 8400 3100
-F 0 "#PWR050" H 8400 2850 50  0001 C CNN
+F 0 "#PWR054" H 8400 2850 50  0001 C CNN
 F 1 "GND" H 8400 2950 50  0000 C CNN
 F 2 "" H 8400 3100 50  0001 C CNN
@@
 $EndComp
 $Comp
-L GND #PWR051
+L GND #PWR055
 U 1 1 596306A0
 P 10850 3100
-F 0 "#PWR051" H 10850 2850 50  0001 C CNN
+F 0 "#PWR055" H 10850 2850 50  0001 C CNN
 F 1 "GND" H 10850 2950 50  0000 C CNN
 F 2 "" H 10850 3100 50  0001 C CNN
@@
 $EndComp
 $Comp
-L GND #PWR052
+L GND #PWR056
 U 1 1 596262B8
 P 7900 3300
-F 0 "#PWR052" H 7900 3050 50  0001 C CNN
+F 0 "#PWR056" H 7900 3050 50  0001 C CNN
 F 1 "GND" H 7900 3150 50  0000 C CNN
 F 2 "" H 7900 3300 50  0001 C CNN
@@
 $EndComp
 $Comp
-L GND #PWR053
+L GND #PWR057
 U 1 1 5962633A
 P 10450 3350
-F 0 "#PWR053" H 10450 3100 50  0001 C CNN
+F 0 "#PWR057" H 10450 3100 50  0001 C CNN
 F 1 "GND" H 10450 3200 50  0000 C CNN
 F 2 "" H 10450 3350 50  0001 C CNN
@@
 $EndComp
 $Comp
-L GND #PWR054
+L GND #PWR058
 U 1 1 596AA4A9
 P 5500 2050
-F 0 "#PWR054" H 5500 1800 50  0001 C CNN
+F 0 "#PWR058" H 5500 1800 50  0001 C CNN
 F 1 "GND" H 5500 1900 50  0000 C CNN
 F 2 "" H 5500 2050 50  0001 C CNN
@@
 $EndComp
 $Comp
-L VCC #PWR055
+L VCC #PWR059
 U 1 1 596AA4E5
 P 5500 1850
-F 0 "#PWR055" H 5500 1700 50  0001 C CNN
+F 0 "#PWR059" H 5500 1700 50  0001 C CNN
 F 1 "VCC" H 5500 2000 50  0000 C CNN
 F 2 "" H 5500 1850 50  0001 C CNN
