File: moteurs_brushless_elec/PCB/uC.sch (KiCad schematic (older format))
At the start: 14 parts, among them J1 CONN_SERIAL, J2 swdio, P1 CONN_I2C, P2 CONN_FREE, U3 stm32f303k8t6, Y1 Crystal_8MHz

Commit message: routing...
Parts:
- added P3: CONN_CAN, Connectors_Molex:Molex_KK-6410-02_02x2.54mm_Straight, symbol CONN_01X02
- added R15: R, Resistors_SMD:R_1206_HandSoldering, symbol R
- added U9: MCP2562, Housings_SOIC:SOIC-8_3.9x4.9mm_Pitch1.27mm, symbol MCP2562
Connections:
- net +3V3: now also U9.5 (VIO)
- net GND: now also U9.2 (VSS), U9.8 (STBY)
- net RX: now also U9.4 (RXD)
- net TX: now also U9.1 (TXD)
- new net: P3.2 (P2), R15.2, U9.6 (CANL)
- new net: P3.1 (P1), R15.1, U9.7 (CANH)
- new net +5V: U9.3 (VDD)
Changed lines of the file:
@@
 Wire Wire Line
 	4300 2800 4950 2800
+$Comp
+L MCP2562 U9
+U 1 1 59C2F137
+P 3500 5300
+F 0 "U9" H 3500 5400 60  0000 C CNN
+F 1 "MCP2562" H 3500 5300 60  0000 C CNN
+F 2 "Housings_SOIC:SOIC-8_3.9x4.9mm_Pitch1.27mm" H 3750 5300 60  0001 C CNN
+F 3 "" H 3750 5300 60  0000 C CNN
+	1    3500 5300
+	1    0    0    -1
+$EndComp
+$Comp
+L +3.3V #PWR038
+U 1 1 59C2F346
+P 3300 4500
+F 0 "#PWR038" H 3300 4350 50  0001 C CNN
+F 1 "+3.3V" H 3300 4640 50  0000 C CNN
+F 2 "" H 3300 4500 50  0000 C CNN
+F 3 "" H 3300 4500 50  0000 C CNN
+	1    3300 4500
+	1    0    0    -1
+$EndComp
+$Comp
+L +5V #PWR039
+U 1 1 59C2F5FE
+P 3700 4500
+F 0 "#PWR039" H 3700 4350 50  0001 C CNN
+F 1 "+5V" H 3700 4640 50  0000 C CNN
+F 2 "" H 3700 4500 50  0000 C CNN
+F 3 "" H 3700 4500 50  0000 C CNN
+	1    3700 4500
+	1    0    0    -1
+$EndComp
+$Comp
+L GND #PWR040
+U 1 1 59C2F720
+P 3500 6100
+F 0 "#PWR040" H 3500 5850 50  0001 C CNN
+F 1 "GND" H 3500 5950 50  0000 C CNN
+F 2 "" H 3500 6100 50  0000 C CNN
+F 3 "" H 3500 6100 50  0000 C CNN
+	1    3500 6100
+	1    0    0    -1
+$EndComp
+$Comp
+L GND #PWR041
+U 1 1 59C2F752
+P 2550 5650
+F 0 "#PWR041" H 2550 5400 50  0001 C CNN
+F 1 "GND" H 2550 5500 50  0000 C CNN
+F 2 "" H 2550 5650 50  0000 C CNN
+F 3 "" H 2550 5650 50  0000 C CNN
+	1    2550 5650
+	1    0    0    -1
+$EndComp
+Wire Wire Line
+	2550 5650 2550 5500
+Wire Wire Line
+	2550 5500 2800 5500
+Wire Wire Line
+	3500 6100 3500 5900
+Text Label 2450 5100 0    60   ~ 0
+TX
+Text Label 2450 5300 0    60   ~ 0
+RX
+Wire Wire Line
+	2450 5100 2800 5100
+Wire Wire Line
+	2450 5300 2800 5300
+Wire Wire Line
+	3300 4500 3300 4600
+Wire Wire Line
+	3700 4500 3700 4600
+$Comp
+L CONN_01X02 P3
+U 1 1 59C2FCB1
+P 4850 5350
+F 0 "P3" H 4850 5500 50  0000 C CNN
+F 1 "CONN_CAN" V 4950 5350 50  0000 C CNN
+F 2 "Connectors_Molex:Molex_KK-6410-02_02x2.54mm_Straight" H 4850 5350 50  0001 C CNN
+F 3 "" H 4850 5350 50  0000 C CNN
+	1    4850 5350
+	1    0    0    -1
+$EndComp
+$Comp
+L R R15
+U 1 1 59C2FCEC
+P 4450 5300
+F 0 "R15" V 4530 5300 50  0000 C CNN
+F 1 "R" V 4450 5300 50  0000 C CNN
+F 2 "Resistors_SMD:R_1206_HandSoldering" V 4380 5300 50  0001 C CNN
+F 3 "" H 4450 5300 50  0000 C CNN
+	1    4450 5300
+	1    0    0    -1
+$EndComp
+Wire Wire Line
+	4200 5500 4650 5500
+Wire Wire Line
+	4650 5500 4650 5400
+Wire Wire Line
+	4450 5450 4450 5500
+Connection ~ 4450 5500
+Wire Wire Line
+	4200 5100 4650 5100
+Wire Wire Line
+	4450 5100 4450 5150
+Wire Wire Line
+	4650 5100 4650 5300
+Connection ~ 4450 5100
 $EndSCHEMATC
