File: moteurs_brushless_elec/PCB/motor_part.sch (KiCad schematic (older format))
At the start: 36 parts, among them K1 Maxon-200142, K2 Maxon-200142, U1 L6235D, U2 L6235D

Commit message: routing...
Parts:
- U1, U2: footprint Housings_SOIC:SOIC-24_7.5x15.4mm_Pitch1.27mm -> Housings_SOIC:SOIC-24W_7.5x15.4mm_Pitch1.27mm
Changed lines of the file:
@@
 F 0 "U1" H 4300 2350 60  0000 C CNN
 F 1 "L6235D" H 4300 2550 60  0000 C CNN
-F 2 "Housings_SOIC:SOIC-24_7.5x15.4mm_Pitch1.27mm" H 4000 2600 60  0001 C CNN
+F 2 "Housings_SOIC:SOIC-24W_7.5x15.4mm_Pitch1.27mm" H 4000 2600 60  0001 C CNN
 F 3 "" H 4000 2600 60  0001 C CNN
 	1    4300 2350
@@
 F 0 "U2" H 11450 2250 60  0000 C CNN
 F 1 "L6235D" H 11450 2450 60  0000 C CNN
-F 2 "Housings_SOIC:SOIC-24_7.5x15.4mm_Pitch1.27mm" H 11150 2500 60  0001 C CNN
+F 2 "Housings_SOIC:SOIC-24W_7.5x15.4mm_Pitch1.27mm" H 11150 2500 60  0001 C CNN
 F 3 "" H 11150 2500 60  0001 C CNN
 	1    11450 2250
