File: moteurs_brushless_elec/PCB/carte_moteurs.kicad_pcb (KiCad board)
At the start: 2 copper layers, 75 parts, among them J1 CONN_SERIAL, J2 swdio, J3 FAN, K1 Maxon-200142, K2 Maxon-200142, P1 CONN_I2C, P2 CONN_FREE, P3 CONN_CAN, P4 encoder_2, P5 encoder_1, U1 L6235D, U2 L6235D, U3 stm32f303k8t6, U4 B_Plug_5mm, U5 LM317_SOT223, U6 LM317_SOT223, U9 MCP2562, Y1 Crystal_8MHz

Commit message: driver_1_done
Parts:
- C2, Cboot1, Cboot2, Cen1, Cen2, Coff1, Coff2, Cp1, Cp2, Cpul1, Cpul2, D1, D2, D3, D4, R1, R2, Rdd1, Rdd2, Ren1, Ren2, Roff1, Roff2, Rp1, Rp2, Rpul1, Rpul2: moved to B.Cu
- moved D9 181.3 mm to (41.1, 101.6)
- moved Rsense1 143.6 mm to (263.2, 53.0)
- moved C8 135.1 mm to (54.7, 123.0)
- moved D7 135.1 mm to (57.7, 142.3)
- moved F1 135.1 mm to (27.7, 114.9)
- moved R10 135.1 mm to (85.5, 117.3)
- moved R8 135.1 mm to (66.3, 138.8)
- moved C6 135.1 mm to (68.9, 112.6)
- moved C7 135.1 mm to (28.9, 142.9)
- moved C9 135.1 mm to (43.6, 129.9)
- moved D8 135.1 mm to (57.7, 134.1)
- moved R11 135.1 mm to (66.3, 132.9)
- moved R13 135.1 mm to (35.9, 143.0)
- moved R7 135.1 mm to (83.2, 123.1)
- moved U5 135.1 mm to (46.6, 141.8)
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Routing:
- net GND: track 0.00 -> 75.4 mm, vias 0 -> 1
- net Net-(Rsense1-Pad1): track 0.00 -> 48.5 mm, vias 0 -> 1
- net /motor_part/DIAG_1: track 0.00 -> 42.0 mm, vias 0 -> 4
- net Net-(K1-Pad1): track 0.00 -> 31.1 mm
- net Net-(K1-Pad5): track 0.00 -> 20.9 mm
- net VCC: track 0.00 -> 19.0 mm, vias 0 -> 1
- net /motor_part/VCP1: track 0.00 -> 18.6 mm, vias 0 -> 1
- net +3V3: track 0.00 -> 17.7 mm, vias 0 -> 2
- net /motor_part/RCPULSE1: track 0.00 -> 16.5 mm, vias 0 -> 1
- net /motor_part/VBOOT1: track 0.00 -> 16.1 mm, vias 0 -> 1
- net /motor_part/Vref: track 0.00 -> 15.7 mm, vias 0 -> 1
- net +5V: track 0.00 -> 14.6 mm, vias 0 -> 1
- net Net-(K1-Pad3): track 0.00 -> 14.5 mm
- net Net-(K1-Pad10): track 0.00 -> 14.0 mm, vias 0 -> 2
- net Net-(K1-Pad8): track 0.00 -> 12.7 mm, vias 0 -> 2
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Other:
- net class Default: clearance 0.2 -> 0.25; trace_width 0.25 -> 0.5; via_dia 0.6 -> 1.2; via_drill 0.4 -> 0.8
- rule trace_clearance: 0.2 -> 0.25

Commit message: début routage brushless
Parts:
- C2, Cboot1, Cboot2, Cen1, Cen2, Coff1, Coff2, Cp1, Cp2, Cpul1, Cpul2, D1, D2, D3, D4, R1, R2, Rdd1, Rdd2, Ren1, Ren2, Roff1, Roff2, Rp1, Rp2, Rpul1, Rpul2: moved to F.Cu
- moved Rsense2 222.2 mm to (21.3, 81.5), turned to 90 degrees
- moved C2 209.2 mm to (50.8, 57.7), turned to 0 degrees
- moved Cboot2 198.3 mm to (41.9, 61.8), turned to 180 degrees
- moved Rdd2 197.6 mm to (39.4, 81.2), turned to 270 degrees
- moved Roff2 197.3 mm to (31.2, 81.2), turned to 270 degrees
- moved D3 194.5 mm to (39.4, 57.2), turned to 270 degrees
- moved Coff2 193.6 mm to (35.2, 81.2), turned to 270 degrees
- moved U2 192.8 mm to (39.0, 70.7)
- moved Cp2 192.2 mm to (34.4, 59.5), turned to 90 degrees
- moved Rp2 189.7 mm to (36.8, 51.9)
- moved D4 189.5 mm to (44.1, 57.3), turned to 90 degrees
- moved K1 186.2 mm to (99.0, 69.8), turned to 270 degrees
- moved Cpul2 186.0 mm to (43.5, 81.3), turned to 270 degrees
- moved Cen2 182.3 mm to (54.9, 83.4), turned to 0 degrees
- moved Ren2 181.5 mm to (54.9, 78.9), turned to 0 degrees
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Connections:
- C1 pad 1: /motor_part/Vref -> /motor_part/Vref1
- C2 pad 1: /motor_part/Vref -> /motor_part/Vref2
- R1 pad 1: /motor_part/Vref -> /motor_part/Vref1
- R2 pad 2: /motor_part/Vref -> /motor_part/Vref1
- R3 pad 1: /motor_part/Vref -> /motor_part/Vref2
- R4 pad 2: /motor_part/Vref -> /motor_part/Vref2
- U1 pad 13: /motor_part/Vref -> /motor_part/Vref1
- U2 pad 13: /motor_part/Vref -> /motor_part/Vref2
Routing:
- net GND: track 75.4 -> 0.00 mm, vias 1 -> 0
- net Net-(Rsense1-Pad1): track 48.5 -> 0.00 mm, vias 1 -> 0
- net /motor_part/DIAG_1: track 42.0 -> 0.00 mm, vias 4 -> 0
- net Net-(K1-Pad1): track 31.1 -> 0.00 mm
- net Net-(K1-Pad5): track 20.9 -> 0.00 mm
- net VCC: track 19.0 -> 0.00 mm, vias 1 -> 0
- net /motor_part/VCP1: track 18.6 -> 0.00 mm, vias 1 -> 0
- net +3V3: track 17.7 -> 0.00 mm, vias 2 -> 0
- net /motor_part/RCPULSE1: track 16.5 -> 0.00 mm, vias 1 -> 0
- net /motor_part/VBOOT1: track 16.1 -> 0.00 mm, vias 1 -> 0
- net /motor_part/Vref: track 15.7 -> 0.00 mm, vias 1 -> 0
- net +5V: track 14.6 -> 0.00 mm, vias 1 -> 0
- net Net-(K1-Pad3): track 14.5 -> 0.00 mm
- net Net-(K1-Pad10): track 14.0 -> 0.00 mm, vias 2 -> 0
- net Net-(K1-Pad8): track 12.7 -> 0.00 mm, vias 2 -> 0
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