File: driver_moteurs/driver-moteurs.sch (KiCad schematic (older format))
At the start: 16 parts, among them P1 CONN_01X12, P2 CONN_I2C, P3 CONN_SERIAL, P4 CONN_CAN, U1 stm32f303k8t6, U2 MCP2562, Y1 Crystal

Commit message: début routage brushless
Parts:
- added P2: CONN_01X02, symbol CONN_01X02
- added P4: CONN_01X04, symbol CONN_01X04
- added P5: CONN_01X03, symbol CONN_01X03
- gave numbers to parts that had none: 1
- renumbered P2 to P3, P3 to P6, P4 to P8
Connections:
- net at U1.18 (PA8): now also P5.3 (P3)
- net at U1.19 (PA9): now also P5.2 (P2)
- net at U1.20 (PA10): now also P5.1 (P1)
- net at U1.25 (PA15): now also P4.4 (P4)
- net at U1.26 (PB3): now also P4.3 (P3)
- net at U1.27 (PB4): now also P4.2 (P2)
- net at U1.28 (PB5): now also P4.1 (P1)
- net at U1.6 (PA0): now also P2.2 (P2)
- net at U1.7 (PA1): now also P2.1 (P1)
- no-connect marks 13 -> 4
Changed lines of the file:
@@
 LIBS:mcp2562
 LIBS:Propulsion_control
+LIBS:driver-moteurs-cache
 EELAYER 25 0
 EELAYER END
@@
 $EndComp
 $Comp
-L CONN_01X02 P2
+L CONN_01X02 P3
 U 1 1 59F78032
 P 4800 900
-F 0 "P2" H 4800 1050 50  0000 C CNN
+F 0 "P3" H 4800 1050 50  0000 C CNN
 F 1 "CONN_I2C" V 4900 900 50  0000 C CNN
 F 2 "" H 4800 900 50  0000 C CNN
@@
 Wire Wire Line
 	4850 1100 4850 2350
-Wire Wire Line
-	5750 3550 5950 3550
-Wire Wire Line
-	5950 3550 5950 3400
 $Comp
 L +3.3V #PWR010
 U 1 1 59F78312
-P 5950 3400
-F 0 "#PWR010" H 5950 3250 50  0001 C CNN
-F 1 "+3.3V" H 5950 3540 50  0000 C CNN
-F 2 "" H 5950 3400 50  0000 C CNN
-F 3 "" H 5950 3400 50  0000 C CNN
-	1    5950 3400
-	1    0    0    -1
-$EndComp
-NoConn ~ 5750 3250
-NoConn ~ 5750 3350
-NoConn ~ 5750 3450
+P 5800 3650
+F 0 "#PWR010" H 5800 3500 50  0001 C CNN
+F 1 "+3.3V" H 5800 3790 50  0000 C CNN
+F 2 "" H 5800 3650 50  0000 C CNN
+F 3 "" H 5800 3650 50  0000 C CNN
+	1    5800 3650
+	-1   0    0    1
+$EndComp
 NoConn ~ 5750 3050
-NoConn ~ 4950 2350
-NoConn ~ 5050 2350
-NoConn ~ 5150 2350
-NoConn ~ 5250 2350
 Wire Wire Line
 	4050 3550 3450 3550
@@
 	0    -1   -1   0
 $EndComp
-NoConn ~ 4050 3350
-NoConn ~ 4050 3450
 Wire Wire Line
 	4050 3150 3250 3150
@@
 $EndComp
 $Comp
-L CONN_01X02 P3
+L CONN_01X02 P6
 U 1 1 59F790F1
 P 7800 2300
-F 0 "P3" H 7800 2450 50  0000 C CNN
+F 0 "P6" H 7800 2450 50  0000 C CNN
 F 1 "CONN_SERIAL" V 7900 2300 50  0000 C CNN
 F 2 "" H 7800 2300 50  0000 C CNN
@@
 $EndComp
 $Comp
-L CONN_01X02 P4
+L CONN_01X02 P8
 U 1 1 59F798B5
 P 10200 3550
-F 0 "P4" H 10200 3700 50  0000 C CNN
+F 0 "P8" H 10200 3700 50  0000 C CNN
 F 1 "CONN_CAN" V 10300 3550 50  0000 C CNN
 F 2 "" H 10200 3550 50  0000 C CNN
@@
 	8550 5050 8550 5200
 $Comp
-L GND #PWR?
+L GND #PWR018
 U 1 1 59F7A8C5
 P 8550 5200
-F 0 "#PWR?" H 8550 4950 50  0001 C CNN
+F 0 "#PWR018" H 8550 4950 50  0001 C CNN
 F 1 "GND" H 8550 5050 50  0000 C CNN
 F 2 "" H 8550 5200 50  0000 C CNN
@@
 swdio
 $Comp
-L CONN_01X04 P?
+L CONN_01X04 P7
 U 1 1 59F7AD02
 P 8050 4900
-F 0 "P?" H 8050 5150 50  0000 C CNN
+F 0 "P7" H 8050 5150 50  0000 C CNN
 F 1 "CONN_SWDIO" V 8150 4900 50  0000 C CNN
 F 2 "" H 8050 4900 50  0000 C CNN
@@
 Text Label 8550 4950 0    60   ~ 0
 nrst
+Wire Wire Line
+	5750 3550 5800 3550
+Wire Wire Line
+	5800 3550 5800 3650
+$Comp
+L CONN_01X03 P5
+U 1 1 5A047397
+P 6150 4400
+F 0 "P5" H 6150 4600 50  0000 C CNN
+F 1 "CONN_01X03" V 6250 4400 50  0000 C CNN
+F 2 "" H 6150 4400 50  0000 C CNN
+F 3 "" H 6150 4400 50  0000 C CNN
+	1    6150 4400
+	0    1    1    0
+$EndComp
+Wire Wire Line
+	5750 3450 6050 3450
+Wire Wire Line
+	6050 3450 6050 4200
+Wire Wire Line
+	6150 4200 6150 3350
+Wire Wire Line
+	6150 3350 5750 3350
+Wire Wire Line
+	5750 3250 6250 3250
+Wire Wire Line
+	6250 3250 6250 4200
+$Comp
+L CONN_01X04 P4
+U 1 1 5A047644
+P 5100 2050
+F 0 "P4" H 5100 2300 50  0000 C CNN
+F 1 "CONN_01X04" V 5200 2050 50  0000 C CNN
+F 2 "" H 5100 2050 50  0000 C CNN
+F 3 "" H 5100 2050 50  0000 C CNN
+	1    5100 2050
+	0    -1   -1   0
+$EndComp
+Wire Wire Line
+	4950 2250 4950 2350
+Wire Wire Line
+	5050 2250 5050 2350
+Wire Wire Line
+	5150 2250 5150 2350
+Wire Wire Line
+	5250 2250 5250 2350
+$Comp
+L CONN_01X02 P2
+U 1 1 5A04791B
+P 3100 3850
+F 0 "P2" H 3100 4000 50  0000 C CNN
+F 1 "CONN_01X02" V 3200 3850 50  0000 C CNN
+F 2 "" H 3100 3850 50  0000 C CNN
+F 3 "" H 3100 3850 50  0000 C CNN
+	1    3100 3850
+	0    1    1    0
+$EndComp
+Wire Wire Line
+	4050 3350 3050 3350
+Wire Wire Line
+	3050 3350 3050 3650
+Wire Wire Line
+	3150 3650 3150 3450
+Wire Wire Line
+	3150 3450 4050 3450
 $EndSCHEMATC
