File: driver_moteurs/power_part.sch (KiCad schematic (older format))
At the start: 19 parts, among them U3 B_Plug_5mm, U4 LM317_SOT223, U5 LM317_SOT223

Commit message: début routage brushless
Parts:
- removed F1: FUSE, symbol FUSE
- added F1: F_Small, symbol F_Small
Connections:
- net VCC: now also F1.2
- net at U3.1: now also F1.1
Changed lines of the file:
@@
 LIBS:mcp2562
 LIBS:Propulsion_control
+LIBS:driver-moteurs-cache
 EELAYER 25 0
 EELAYER END
@@
 $EndComp
 $Comp
-L FUSE F1
-U 1 1 59F75D3C
-P 3500 2400
-F 0 "F1" H 3600 2450 50  0000 C CNN
-F 1 "FUSE" H 3400 2350 50  0000 C CNN
-F 2 "" H 3500 2400 50  0000 C CNN
-F 3 "" H 3500 2400 50  0000 C CNN
-	1    3500 2400
-	1    0    0    -1
-$EndComp
-$Comp
 L CP C4
 U 1 1 59F75D85
@@
 $EndComp
 $Comp
-L GND #PWR018
+L GND #PWR019
 U 1 1 59F7601E
 P 3850 3250
-F 0 "#PWR018" H 3850 3000 50  0001 C CNN
+F 0 "#PWR019" H 3850 3000 50  0001 C CNN
 F 1 "GND" H 3850 3100 50  0000 C CNN
 F 2 "" H 3850 3250 50  0000 C CNN
@@
 $EndComp
 $Comp
-L VCC #PWR019
+L VCC #PWR020
 U 1 1 59F761AB
 P 4750 2200
-F 0 "#PWR019" H 4750 2050 50  0001 C CNN
+F 0 "#PWR020" H 4750 2050 50  0001 C CNN
 F 1 "VCC" H 4750 2350 50  0000 C CNN
 F 2 "" H 4750 2200 50  0000 C CNN
@@
 $EndComp
 $Comp
-L PWR_FLAG #FLG020
+L PWR_FLAG #FLG021
 U 1 1 59F761CD
 P 4450 2200
-F 0 "#FLG020" H 4450 2295 50  0001 C CNN
+F 0 "#FLG021" H 4450 2295 50  0001 C CNN
 F 1 "PWR_FLAG" H 4450 2380 50  0000 C CNN
 F 2 "" H 4450 2200 50  0000 C CNN
@@
 $EndComp
 $Comp
-L GND #PWR021
+L GND #PWR022
 U 1 1 59F763B8
 P 3000 3200
-F 0 "#PWR021" H 3000 2950 50  0001 C CNN
+F 0 "#PWR022" H 3000 2950 50  0001 C CNN
 F 1 "GND" H 3000 3050 50  0000 C CNN
 F 2 "" H 3000 3200 50  0000 C CNN
@@
 $EndComp
 $Comp
-L GND #PWR022
+L GND #PWR023
 U 1 1 59F763D8
 P 5500 3200
-F 0 "#PWR022" H 5500 2950 50  0001 C CNN
+F 0 "#PWR023" H 5500 2950 50  0001 C CNN
 F 1 "GND" H 5500 3050 50  0000 C CNN
 F 2 "" H 5500 3200 50  0000 C CNN
@@
 $EndComp
 $Comp
-L PWR_FLAG #FLG023
+L PWR_FLAG #FLG024
 U 1 1 59F76416
 P 3250 3200
-F 0 "#FLG023" H 3250 3295 50  0001 C CNN
+F 0 "#FLG024" H 3250 3295 50  0001 C CNN
 F 1 "PWR_FLAG" H 3250 3380 50  0000 C CNN
 F 2 "" H 3250 3200 50  0000 C CNN
@@
 $EndComp
 $Comp
-L VCC #PWR024
+L VCC #PWR025
 U 1 1 59F764CC
 P 7000 2250
-F 0 "#PWR024" H 7000 2100 50  0001 C CNN
+F 0 "#PWR025" H 7000 2100 50  0001 C CNN
 F 1 "VCC" H 7000 2400 50  0000 C CNN
 F 2 "" H 7000 2250 50  0000 C CNN
@@
 $EndComp
 Wire Wire Line
-	3000 2400 3250 2400
-Wire Wire Line
-	3750 2400 4900 2400
+	3000 2400 3400 2400
+Wire Wire Line
+	3600 2400 4900 2400
 Wire Wire Line
 	3850 2400 3850 2700
@@
 Wire Wire Line
 	5500 3200 5500 3050
-Connection ~ 3850 3200
 Wire Wire Line
 	3000 2500 3000 3200
@@
 Connection ~ 7850 3100
 $Comp
-L GND #PWR025
+L GND #PWR026
 U 1 1 59F76711
 P 7850 3700
-F 0 "#PWR025" H 7850 3450 50  0001 C CNN
+F 0 "#PWR026" H 7850 3450 50  0001 C CNN
 F 1 "GND" H 7850 3550 50  0000 C CNN
 F 2 "" H 7850 3700 50  0000 C CNN
@@
 	9300 2900 9300 3150
 $Comp
-L +5V #PWR026
+L +5V #PWR027
 U 1 1 59F76B40
 P 9300 2100
-F 0 "#PWR026" H 9300 1950 50  0001 C CNN
+F 0 "#PWR027" H 9300 1950 50  0001 C CNN
 F 1 "+5V" H 9300 2240 50  0000 C CNN
 F 2 "" H 9300 2100 50  0000 C CNN
@@
 	1    0    0    -1
 $EndComp
-$Comp
-L PWR_FLAG #FLG027
-U 1 1 59F76B6E
-P 9600 2100
-F 0 "#FLG027" H 9600 2195 50  0001 C CNN
-F 1 "PWR_FLAG" H 9600 2280 50  0000 C CNN
-F 2 "" H 9600 2100 50  0000 C CNN
-F 3 "" H 9600 2100 50  0000 C CNN
-	1    9600 2100
-	1    0    0    -1
-$EndComp
-Wire Wire Line
-	9300 2200 9600 2200
-Wire Wire Line
-	9600 2200 9600 2100
 Connection ~ 9300 2200
 $Comp
@@
 $EndComp
 Wire Wire Line
-	3700 4800 5200 4800
-Wire Wire Line
 	4100 4800 4100 5250
 Wire Wire Line
@@
 	4750 5350 4750 5600
 $Comp
-L PWR_FLAG #FLG032
-U 1 1 59F77092
-P 5050 4550
-F 0 "#FLG032" H 5050 4645 50  0001 C CNN
-F 1 "PWR_FLAG" H 5050 4730 50  0000 C CNN
-F 2 "" H 5050 4550 50  0000 C CNN
-F 3 "" H 5050 4550 50  0000 C CNN
-	1    5050 4550
-	1    0    0    -1
-$EndComp
-Wire Wire Line
-	4750 4650 5050 4650
-Wire Wire Line
-	5050 4650 5050 4550
-Connection ~ 4750 4650
-$Comp
-L GND #PWR033
+L GND #PWR032
 U 1 1 59F7709B
 P 4750 5600
-F 0 "#PWR033" H 4750 5350 50  0001 C CNN
+F 0 "#PWR032" H 4750 5350 50  0001 C CNN
 F 1 "GND" H 4750 5450 50  0000 C CNN
 F 2 "" H 4750 5600 50  0000 C CNN
@@
 $EndComp
 $Comp
-L GND #PWR034
+L GND #PWR033
 U 1 1 59F770A1
 P 6050 5650
-F 0 "#PWR034" H 6050 5400 50  0001 C CNN
+F 0 "#PWR033" H 6050 5400 50  0001 C CNN
 F 1 "GND" H 6050 5500 50  0000 C CNN
 F 2 "" H 6050 5650 50  0000 C CNN
@@
 $EndComp
 $Comp
-L +3.3V #PWR035
+L +3.3V #PWR034
 U 1 1 59F7712F
 P 4750 4550
-F 0 "#PWR035" H 4750 4400 50  0001 C CNN
+F 0 "#PWR034" H 4750 4400 50  0001 C CNN
 F 1 "+3.3V" H 4750 4690 50  0000 C CNN
 F 2 "" H 4750 4550 50  0000 C CNN
@@
 Connection ~ 4100 4800
 Connection ~ 8650 2350
+Wire Wire Line
+	3700 4800 5200 4800
+$Comp
+L F_Small F1
+U 1 1 59F7C292
+P 3500 2400
+F 0 "F1" H 3460 2460 50  0000 L CNN
+F 1 "F_Small" H 3380 2340 50  0000 L CNN
+F 2 "" H 3500 2400 50  0000 C CNN
+F 3 "" H 3500 2400 50  0000 C CNN
+	1    3500 2400
+	1    0    0    -1
+$EndComp
 $EndSCHEMATC
