File: Electronique/moteurs_brushless_elec/PCB/uC.sch (KiCad schematic (older format))
At the start: 17 parts, among them J1 CONN_SERIAL, J2 swdio, P1 CONN_I2C, P2 CONN_FREE, P3 CONN_CAN, U3 stm32f303k8t6, U9 MCP2562, Y1 Crystal_8MHz

Commit message: rectification des empreintes
Parts:
- J2: footprint Connectors_Molex:Molex_KK-6410-04_04x2.54mm_Straight -> Pin_Headers:Pin_Header_Angled_1x04_Pitch2.54mm
Changed lines of the file:
@@
 $EndComp
 $Comp
-L GND #PWR027
+L GND #PWR34
 U 1 1 59615D7C
 P 3950 3000
-F 0 "#PWR027" H 3950 2750 50  0001 C CNN
+F 0 "#PWR34" H 3950 2750 50  0001 C CNN
 F 1 "GND" H 3950 2850 50  0000 C CNN
 F 2 "" H 3950 3000 50  0001 C CNN
@@
 F 0 "J2" H 3450 1750 50  0000 C CNN
 F 1 "swdio" V 3550 1500 50  0000 C CNN
-F 2 "Connectors_Molex:Molex_KK-6410-04_04x2.54mm_Straight" H 3450 1500 50  0001 C CNN
+F 2 "Pin_Headers:Pin_Header_Angled_1x04_Pitch2.54mm" H 3450 1500 50  0001 C CNN
 F 3 "" H 3450 1500 50  0001 C CNN
 	1    3450 1500
@@
 nrst
 $Comp
-L GND #PWR028
+L GND #PWR33
 U 1 1 59615FF5
 P 3850 1650
-F 0 "#PWR028" H 3850 1400 50  0001 C CNN
+F 0 "#PWR33" H 3850 1400 50  0001 C CNN
 F 1 "GND" H 3850 1500 50  0000 C CNN
 F 2 "" H 3850 1650 50  0001 C CNN
@@
 	3650 1650 3850 1650
 $Comp
-L GND #PWR029
+L GND #PWR39
 U 1 1 596164DB
 P 5450 2050
-F 0 "#PWR029" H 5450 1800 50  0001 C CNN
+F 0 "#PWR39" H 5450 1800 50  0001 C CNN
 F 1 "GND" H 5450 1900 50  0000 C CNN
 F 2 "" H 5450 2050 50  0001 C CNN
@@
 $EndComp
 $Comp
-L GND #PWR030
+L GND #PWR40
 U 1 1 596164F6
 P 6150 4050
-F 0 "#PWR030" H 6150 3800 50  0001 C CNN
+F 0 "#PWR40" H 6150 3800 50  0001 C CNN
 F 1 "GND" H 6150 3900 50  0000 C CNN
 F 2 "" H 6150 4050 50  0001 C CNN
@@
 	6150 3900 6150 4050
 $Comp
-L +3.3V #PWR031
+L +3.3V #PWR41
 U 1 1 59629D6A
 P 6800 3400
-F 0 "#PWR031" H 6800 3250 50  0001 C CNN
+F 0 "#PWR41" H 6800 3250 50  0001 C CNN
 F 1 "+3.3V" H 6800 3540 50  0000 C CNN
 F 2 "" H 6800 3400 50  0001 C CNN
@@
 $EndComp
 $Comp
-L +3.3V #PWR032
+L +3.3V #PWR36
 U 1 1 59629D85
 P 4750 3100
-F 0 "#PWR032" H 4750 2950 50  0001 C CNN
+F 0 "#PWR36" H 4750 2950 50  0001 C CNN
 F 1 "+3.3V" H 4750 3240 50  0000 C CNN
 F 2 "" H 4750 3100 50  0001 C CNN
@@
 $EndComp
 $Comp
-L +3.3V #PWR033
+L +3.3V #PWR35
 U 1 1 59629D99
 P 4750 2700
-F 0 "#PWR033" H 4750 2550 50  0001 C CNN
+F 0 "#PWR35" H 4750 2550 50  0001 C CNN
 F 1 "+3.3V" H 4750 2840 50  0000 C CNN
 F 2 "" H 4750 2700 50  0001 C CNN
@@
 $EndComp
 $Comp
-L GND #PWR034
+L GND #PWR42
 U 1 1 596A8A12
 P 7900 4300
-F 0 "#PWR034" H 7900 4050 50  0001 C CNN
+F 0 "#PWR42" H 7900 4050 50  0001 C CNN
 F 1 "GND" H 7900 4150 50  0000 C CNN
 F 2 "" H 7900 4300 50  0001 C CNN
@@
 $EndComp
 $Comp
-L +3.3V #PWR035
+L +3.3V #PWR37
 U 1 1 5974E084
 P 4900 1300
-F 0 "#PWR035" H 4900 1150 50  0001 C CNN
+F 0 "#PWR37" H 4900 1150 50  0001 C CNN
 F 1 "+3.3V" H 4900 1440 50  0000 C CNN
 F 2 "" H 4900 1300 50  0001 C CNN
@@
 $EndComp
 $Comp
-L GND #PWR036
+L GND #PWR38
 U 1 1 5974E0A8
 P 4900 2100
-F 0 "#PWR036" H 4900 1850 50  0001 C CNN
+F 0 "#PWR38" H 4900 1850 50  0001 C CNN
 F 1 "GND" H 4900 1950 50  0000 C CNN
 F 2 "" H 4900 2100 50  0001 C CNN
@@
 $EndComp
 $Comp
-L GND #PWR037
+L GND #PWR28
 U 1 1 59C15C7D
 P 2400 2500
-F 0 "#PWR037" H 2400 2250 50  0001 C CNN
+F 0 "#PWR28" H 2400 2250 50  0001 C CNN
 F 1 "GND" H 2400 2350 50  0000 C CNN
 F 2 "" H 2400 2500 50  0000 C CNN
@@
 $EndComp
 $Comp
-L +3.3V #PWR038
+L +3.3V #PWR30
 U 1 1 59C2F346
 P 3300 4500
-F 0 "#PWR038" H 3300 4350 50  0001 C CNN
+F 0 "#PWR30" H 3300 4350 50  0001 C CNN
 F 1 "+3.3V" H 3300 4640 50  0000 C CNN
 F 2 "" H 3300 4500 50  0000 C CNN
@@
 $EndComp
 $Comp
-L +5V #PWR039
+L +5V #PWR32
 U 1 1 59C2F5FE
 P 3700 4500
-F 0 "#PWR039" H 3700 4350 50  0001 C CNN
+F 0 "#PWR32" H 3700 4350 50  0001 C CNN
 F 1 "+5V" H 3700 4640 50  0000 C CNN
 F 2 "" H 3700 4500 50  0000 C CNN
@@
 $EndComp
 $Comp
-L GND #PWR040
+L GND #PWR31
 U 1 1 59C2F720
 P 3500 6100
-F 0 "#PWR040" H 3500 5850 50  0001 C CNN
+F 0 "#PWR31" H 3500 5850 50  0001 C CNN
 F 1 "GND" H 3500 5950 50  0000 C CNN
 F 2 "" H 3500 6100 50  0000 C CNN
@@
 $EndComp
 $Comp
-L GND #PWR041
+L GND #PWR29
 U 1 1 59C2F752
 P 2550 5650
-F 0 "#PWR041" H 2550 5400 50  0001 C CNN
+F 0 "#PWR29" H 2550 5400 50  0001 C CNN
 F 1 "GND" H 2550 5500 50  0000 C CNN
 F 2 "" H 2550 5650 50  0000 C CNN
