File: Electronique/moteurs_brushless_elec/PCB/power_part.sch (KiCad schematic (older format))
At the start: 27 parts, among them J3 FAN, U12 B_Plug_5mm, U4 B_Plug_5mm, U5 LM317_SOT223, U6 LM317_SOT223

Commit message: trous et dim o
Connections:
- net VCC: no longer J3.1 (P1)
- net VDD: now also J3.1 (P1)
Changed lines of the file:
@@
-	1    0    0    -1
-$EndComp
-$Comp
-L VCC #PWR060
-U 1 1 596AA4E5
-P 5500 1850
-F 0 "#PWR060" H 5500 1700 50  0001 C CNN
-F 1 "VCC" H 5500 2000 50  0000 C CNN
-F 2 "" H 5500 1850 50  0001 C CNN
-F 3 "" H 5500 1850 50  0001 C CNN
-	1    5500 1850
 	1    0    0    -1
 $EndComp
 Wire Wire Line
-	5500 1850 5500 1900
+	5500 1750 5500 1900
 Wire Wire Line
 	5500 1900 5600 1900
@@
 Wire Wire Line
 	3550 4000 3550 4150
+$Comp
+L VDD #PWR?
+U 1 1 5A345130
+P 5500 1750
+F 0 "#PWR?" H 5500 1600 50  0001 C CNN
+F 1 "VDD" H 5500 1900 50  0000 C CNN
+F 2 "" H 5500 1750 50  0000 C CNN
+F 3 "" H 5500 1750 50  0000 C CNN
+	1    5500 1750
+	1    0    0    -1
+$EndComp
 $EndSCHEMATC

Commit message: correction
Changed lines of the file:
@@
 $EndDescr
 $Comp
-L VCC #PWR043
+L VCC #PWR042
 U 1 1 5962E5D8
 P 4650 2300
-F 0 "#PWR043" H 4650 2150 50  0001 C CNN
+F 0 "#PWR042" H 4650 2150 50  0001 C CNN
 F 1 "VCC" H 4650 2450 50  0000 C CNN
 F 2 "" H 4650 2300 50  0001 C CNN
@@
 $EndComp
 $Comp
-L +3.3V #PWR044
+L +3.3V #PWR043
 U 1 1 5962E5EC
 P 10450 2450
-F 0 "#PWR044" H 10450 2300 50  0001 C CNN
+F 0 "#PWR043" H 10450 2300 50  0001 C CNN
 F 1 "+3.3V" H 10450 2590 50  0000 C CNN
 F 2 "" H 10450 2450 50  0001 C CNN
@@
 $EndComp
 $Comp
-L GND #PWR045
+L GND #PWR044
 U 1 1 5962E732
 P 3650 2900
-F 0 "#PWR045" H 3650 2650 50  0001 C CNN
+F 0 "#PWR044" H 3650 2650 50  0001 C CNN
 F 1 "GND" H 3650 2750 50  0000 C CNN
 F 2 "" H 3650 2900 50  0001 C CNN
@@
 $EndComp
 $Comp
-L GND #PWR046
+L GND #PWR045
 U 1 1 5962E829
 P 4250 3000
-F 0 "#PWR046" H 4250 2750 50  0001 C CNN
+F 0 "#PWR045" H 4250 2750 50  0001 C CNN
 F 1 "GND" H 4250 2850 50  0000 C CNN
 F 2 "" H 4250 3000 50  0001 C CNN
@@
 	3650 2650 3650 2900
 $Comp
-L PWR_FLAG #FLG047
+L PWR_FLAG #FLG046
 U 1 1 5962EB73
 P 4500 2400
-F 0 "#FLG047" H 4500 2475 50  0001 C CNN
+F 0 "#FLG046" H 4500 2475 50  0001 C CNN
 F 1 "PWR_FLAG" H 4500 2550 50  0000 C CNN
 F 2 "" H 4500 2400 50  0001 C CNN
@@
 $EndComp
 $Comp
-L PWR_FLAG #FLG048
+L PWR_FLAG #FLG047
 U 1 1 5962EBA1
 P 3800 2850
-F 0 "#FLG048" H 3800 2925 50  0001 C CNN
+F 0 "#FLG047" H 3800 2925 50  0001 C CNN
 F 1 "PWR_FLAG" H 3800 3000 50  0000 C CNN
 F 2 "" H 3800 2850 50  0001 C CNN
@@
 Connection ~ 3650 2850
 $Comp
-L +5V #PWR049
+L +5V #PWR048
 U 1 1 5962ECD4
 P 7900 2450
-F 0 "#PWR049" H 7900 2300 50  0001 C CNN
+F 0 "#PWR048" H 7900 2300 50  0001 C CNN
 F 1 "+5V" H 7900 2590 50  0000 C CNN
 F 2 "" H 7900 2450 50  0001 C CNN
@@
 $EndComp
 $Comp
-L VCC #PWR050
+L VCC #PWR049
 U 1 1 5962F11A
 P 6450 2450
-F 0 "#PWR050" H 6450 2300 50  0001 C CNN
+F 0 "#PWR049" H 6450 2300 50  0001 C CNN
 F 1 "VCC" H 6450 2600 50  0000 C CNN
 F 2 "" H 6450 2450 50  0001 C CNN
@@
 $EndComp
 $Comp
-L VCC #PWR051
+L VCC #PWR050
 U 1 1 5962F138
 P 9050 2450
-F 0 "#PWR051" H 9050 2300 50  0001 C CNN
+F 0 "#PWR050" H 9050 2300 50  0001 C CNN
 F 1 "VCC" H 9050 2600 50  0000 C CNN
 F 2 "" H 9050 2450 50  0001 C CNN
@@
 $EndComp
 $Comp
-L GND #PWR052
+L GND #PWR051
 U 1 1 5962F3CB
 P 7000 3600
-F 0 "#PWR052" H 7000 3350 50  0001 C CNN
+F 0 "#PWR051" H 7000 3350 50  0001 C CNN
 F 1 "GND" H 7000 3450 50  0000 C CNN
 F 2 "" H 7000 3600 50  0001 C CNN
@@
 $EndComp
 $Comp
-L GND #PWR053
+L GND #PWR052
 U 1 1 5962F3F1
 P 9650 3600
-F 0 "#PWR053" H 9650 3350 50  0001 C CNN
+F 0 "#PWR052" H 9650 3350 50  0001 C CNN
 F 1 "GND" H 9650 3450 50  0000 C CNN
 F 2 "" H 9650 3600 50  0001 C CNN
@@
 $EndComp
 $Comp
-L GND #PWR054
+L GND #PWR053
 U 1 1 5963063C
 P 5450 3000
-F 0 "#PWR054" H 5450 2750 50  0001 C CNN
+F 0 "#PWR053" H 5450 2750 50  0001 C CNN
 F 1 "GND" H 5450 2850 50  0000 C CNN
 F 2 "" H 5450 3000 50  0001 C CNN
@@
 $EndComp
 $Comp
-L GND #PWR055
+L GND #PWR054
 U 1 1 5963066E
 P 8400 3100
-F 0 "#PWR055" H 8400 2850 50  0001 C CNN
+F 0 "#PWR054" H 8400 2850 50  0001 C CNN
 F 1 "GND" H 8400 2950 50  0000 C CNN
 F 2 "" H 8400 3100 50  0001 C CNN
@@
 $EndComp
 $Comp
-L GND #PWR056
+L GND #PWR055
 U 1 1 596306A0
 P 10850 3100
-F 0 "#PWR056" H 10850 2850 50  0001 C CNN
+F 0 "#PWR055" H 10850 2850 50  0001 C CNN
 F 1 "GND" H 10850 2950 50  0000 C CNN
 F 2 "" H 10850 3100 50  0001 C CNN
@@
 $EndComp
 $Comp
-L GND #PWR057
+L GND #PWR056
 U 1 1 596262B8
 P 7900 3300
-F 0 "#PWR057" H 7900 3050 50  0001 C CNN
+F 0 "#PWR056" H 7900 3050 50  0001 C CNN
 F 1 "GND" H 7900 3150 50  0000 C CNN
 F 2 "" H 7900 3300 50  0001 C CNN
@@
 $EndComp
 $Comp
-L GND #PWR058
+L GND #PWR057
 U 1 1 5962633A
 P 10450 3350
-F 0 "#PWR058" H 10450 3100 50  0001 C CNN
+F 0 "#PWR057" H 10450 3100 50  0001 C CNN
 F 1 "GND" H 10450 3200 50  0000 C CNN
 F 2 "" H 10450 3350 50  0001 C CNN
@@
 $EndComp
 $Comp
-L GND #PWR059
+L GND #PWR058
 U 1 1 596AA4A9
 P 5500 2050
-F 0 "#PWR059" H 5500 1800 50  0001 C CNN
+F 0 "#PWR058" H 5500 1800 50  0001 C CNN
 F 1 "GND" H 5500 1900 50  0000 C CNN
 F 2 "" H 5500 2050 50  0001 C CNN
@@
 $EndComp
 $Comp
-L GND #PWR060
+L GND #PWR059
 U 1 1 5A3446EC
 P 5450 4450
-F 0 "#PWR060" H 5450 4200 50  0001 C CNN
+F 0 "#PWR059" H 5450 4200 50  0001 C CNN
 F 1 "GND" H 5450 4300 50  0000 C CNN
 F 2 "" H 5450 4450 50  0000 C CNN
@@
 $EndComp
 $Comp
-L GND #PWR061
+L GND #PWR060
 U 1 1 5A344736
 P 4600 4550
-F 0 "#PWR061" H 4600 4300 50  0001 C CNN
+F 0 "#PWR060" H 4600 4300 50  0001 C CNN
 F 1 "GND" H 4600 4400 50  0000 C CNN
 F 2 "" H 4600 4550 50  0000 C CNN
@@
 Connection ~ 4850 3900
 $Comp
-L VDD #PWR062
+L VDD #PWR061
 U 1 1 5A345F99
 P 4600 3600
-F 0 "#PWR062" H 4600 3450 50  0001 C CNN
+F 0 "#PWR061" H 4600 3450 50  0001 C CNN
 F 1 "VDD" H 4600 3750 50  0000 C CNN
 F 2 "" H 4600 3600 50  0000 C CNN
@@
 $EndComp
 $Comp
-L PWR_FLAG #FLG063
+L PWR_FLAG #FLG062
 U 1 1 5A345FE3
 P 4450 3750
-F 0 "#FLG063" H 4450 3845 50  0001 C CNN
+F 0 "#FLG062" H 4450 3845 50  0001 C CNN
 F 1 "PWR_FLAG" H 4450 3930 50  0000 C CNN
 F 2 "" H 4450 3750 50  0000 C CNN
@@
 	3350 3900 3650 3900
 $Comp
-L GND #PWR064
+L GND #PWR063
 U 1 1 5A343A85
 P 3550 4150
-F 0 "#PWR064" H 3550 3900 50  0001 C CNN
+F 0 "#PWR063" H 3550 3900 50  0001 C CNN
 F 1 "GND" H 3550 4000 50  0000 C CNN
 F 2 "" H 3550 4150 50  0000 C CNN
@@
 	3550 4000 3550 4150
 $Comp
-L VDD #PWR065
+L VDD #PWR064
 U 1 1 5A345130
 P 5500 1750
-F 0 "#PWR065" H 5500 1600 50  0001 C CNN
+F 0 "#PWR064" H 5500 1600 50  0001 C CNN
 F 1 "VDD" H 5500 1900 50  0000 C CNN
 F 2 "" H 5500 1750 50  0000 C CNN
@@
 	1    0    0    -1
 $EndComp
+Wire Wire Line
+	3650 2850 3800 2850
 $EndSCHEMATC

Commit message: modif moteur axe z
Parts:
- R10, R13: value R -> 470R
- R11: value 33kR -> 370R
- R12: value 56kR -> 220R
- R16, R7: value R -> 2kR
- R8: value 3.3kR -> 820R
- R9: value 10kR -> 270R
Changed lines of the file:
@@
 P 7000 3350
 F 0 "R8" V 7080 3350 50  0000 C CNN
-F 1 "3.3kR" V 7000 3350 50  0000 C CNN
+F 1 "820R" V 7000 3350 50  0000 C CNN
 F 2 "Resistors_SMD:R_1206_HandSoldering" V 6930 3350 50  0001 C CNN
 F 3 "" H 7000 3350 50  0001 C CNN
@@
 P 7350 3150
 F 0 "R9" V 7430 3150 50  0000 C CNN
-F 1 "10kR" V 7350 3150 50  0000 C CNN
+F 1 "270R" V 7350 3150 50  0000 C CNN
 F 2 "Resistors_SMD:R_1206_HandSoldering" V 7280 3150 50  0001 C CNN
 F 3 "" H 7350 3150 50  0001 C CNN
@@
 P 9650 3350
 F 0 "R11" V 9730 3350 50  0000 C CNN
-F 1 "33kR" V 9650 3350 50  0000 C CNN
+F 1 "370R" V 9650 3350 50  0000 C CNN
 F 2 "Resistors_SMD:R_1206_HandSoldering" V 9580 3350 50  0001 C CNN
 F 3 "" H 9650 3350 50  0001 C CNN
@@
 P 10000 3150
 F 0 "R12" V 10080 3150 50  0000 C CNN
-F 1 "56kR" V 10000 3150 50  0000 C CNN
+F 1 "220R" V 10000 3150 50  0000 C CNN
 F 2 "Resistors_SMD:R_1206_HandSoldering" V 9930 3150 50  0001 C CNN
 F 3 "" H 10000 3150 50  0001 C CNN
@@
 P 5200 2550
 F 0 "R7" V 5280 2550 50  0000 C CNN
-F 1 "R" V 5200 2550 50  0000 C CNN
+F 1 "2kR" V 5200 2550 50  0000 C CNN
 F 2 "Resistors_SMD:R_1206_HandSoldering" V 5130 2550 50  0001 C CNN
 F 3 "" H 5200 2550 50  0001 C CNN
@@
 P 8150 2550
 F 0 "R10" V 8230 2550 50  0000 C CNN
-F 1 "R" V 8150 2550 50  0000 C CNN
+F 1 "470R" V 8150 2550 50  0000 C CNN
 F 2 "Resistors_SMD:R_1206_HandSoldering" V 8080 2550 50  0001 C CNN
 F 3 "" H 8150 2550 50  0001 C CNN
@@
 P 10650 2500
 F 0 "R13" V 10730 2500 50  0000 C CNN
-F 1 "R" V 10650 2500 50  0000 C CNN
+F 1 "470R" V 10650 2500 50  0000 C CNN
 F 2 "Resistors_SMD:R_1206_HandSoldering" V 10580 2500 50  0001 C CNN
 F 3 "" H 10650 2500 50  0001 C CNN
@@
 P 5150 3900
 F 0 "R16" V 5230 3900 50  0000 C CNN
-F 1 "R" V 5150 3900 50  0000 C CNN
+F 1 "2kR" V 5150 3900 50  0000 C CNN
 F 2 "Resistors_SMD:R_1206_HandSoldering" V 5080 3900 50  0001 C CNN
 F 3 "" H 5150 3900 50  0000 C CNN
