File: Electronique/moteurs_brushless_elec/PCB/carte_moteurs.kicad_pcb (KiCad board)
At the start: 2 copper layers, 90 x 65 mm, 82 parts, among them J1 CONN_SERIAL, J2 swdio, J3 FAN, K1 Maxon-200142, K2 Maxon-200142, P1 CONN_I2C, P2 CONN_FREE, P3 CONN_CAN, P4 encoder_2, P5 encoder_1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

Commit message: Placement brushless
Parts:
- Cboot2, R12, R9, Rdd2: moved to B.Cu
- Cen2, Cp1, Cp2, Rp1, Rp2, U1, U2, U5, U6, U9: moved to F.Cu
- moved J2 61.6 mm to (138.7, 113.0), turned to 0 degrees
- moved P2 57.0 mm to (138.4, 136.1), turned to 270 degrees
- moved C5 54.0 mm to (112.5, 138.4), turned to 270 degrees
- moved P4 52.2 mm to (138.6, 124.5), turned to 270 degrees
- moved C7 42.1 mm to (56.6, 125.4), turned to 270 degrees
- moved R7 37.4 mm to (60.1, 125.4), turned to 90 degrees
- moved D5 37.0 mm to (140.7, 96.8), turned to 270 degrees
- moved F2 34.9 mm to (100.7, 144.1), turned to 180 degrees
- moved J3 34.8 mm to (69.0, 146.8), turned to 0 degrees
- moved Rp1 34.0 mm to (121.2, 92.7), turned to 0 degrees
- moved U4 32.6 mm to (63.6, 125.1), turned to 0 degrees
- moved D2 30.7 mm to (116.1, 96.8)
- moved R6 30.2 mm to (133.9, 100.1)
- moved Cen2 29.7 mm to (81.5, 101.3), turned to 0 degrees
- moved Cboot1 28.3 mm to (121.4, 98.6), turned to 270 degrees
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Routing:
- net GND: track 466.0 -> 0.00 mm, vias 19 -> 0
- net +3V3: track 178.4 -> 0.00 mm, vias 3 -> 0
- net VCC: track 163.7 -> 0.00 mm
- net +5V: track 156.5 -> 0.00 mm, vias 4 -> 0
- net VDD: track 120.4 -> 0.00 mm
- net Net-(P2-Pad1): track 87.2 -> 0.00 mm
- net Net-(P2-Pad2): track 74.5 -> 0.00 mm
- net /uC/nrst: track 73.3 -> 0.00 mm, vias 3 -> 0
- net /motor_part/DIAG_2: track 65.6 -> 0.00 mm, vias 5 -> 0
- net /motor_part/DIAG_1: track 46.5 -> 0.00 mm, vias 5 -> 0
- net /motor_part/TACHO_1: track 44.7 -> 0.00 mm, vias 1 -> 0
- net /motor_part/TACHO_2: track 44.6 -> 0.00 mm, vias 2 -> 0
- net /uC/I2C_SDA: track 44.0 -> 0.00 mm, vias 1 -> 0
- net Net-(R5-Pad1): track 43.6 -> 0.00 mm, vias 2 -> 0
- net /uC/swclk: track 42.6 -> 0.00 mm
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
Commit message: Routage brushless
Parts:
- moved D5 35.2 mm to (126.7, 129.0), turned to 0 degrees
- moved R6 33.3 mm to (126.7, 132.6)
- moved J3 0.40 mm to (69.0, 146.4)
Routing:
- net GND: track 0.00 -> 558.2 mm, vias 0 -> 11
- net +5V: track 0.00 -> 216.1 mm, vias 0 -> 4
- net +3V3: track 0.00 -> 206.8 mm, vias 0 -> 1
- net VCC: track 0.00 -> 176.8 mm, vias 0 -> 2
- net VDD: track 0.00 -> 101.9 mm
- net /motor_part/TACHO_2: track 0.00 -> 82.4 mm, vias 0 -> 4
- net /motor_part/DIR_2: track 0.00 -> 47.8 mm, vias 0 -> 2
- net /motor_part/DIAG_2: track 0.00 -> 47.2 mm, vias 0 -> 2
- net /motor_part/BRAKE_2: track 0.00 -> 42.2 mm
- net /uC/nrst: track 0.00 -> 42.0 mm, vias 0 -> 1
- net /motor_part/DIAG_1: track 0.00 -> 36.1 mm, vias 0 -> 3
- net /motor_part/BRAKE_1: track 0.00 -> 36.0 mm, vias 0 -> 2
- net Net-(K2-Pad5): track 0.00 -> 34.8 mm, vias 0 -> 1
- net /motor_part/Vref2: track 0.00 -> 32.9 mm, vias 0 -> 1
- net /uC/swclk: track 0.00 -> 32.9 mm
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
Commit message: Textes PCB
Routing:
- net GND: vias 11 -> 12
Other:
- board text added: "Robotronik CDFR 2018"
- board text removed: "Robotronik_CDFR_2018"
Changed lines of the file:
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@@
     (thickness 1.6)
     (drawings 14)
-    (tracks 989)
+    (tracks 990)
     (zones 0)
     (modules 82)
@@
     (46 B.CrtYd user)
     (47 F.CrtYd user)
-    (48 B.Fab user hide)
-    (49 F.Fab user hide)
+    (48 B.Fab user)
+    (49 F.Fab user)
   )
   (setup
-    (last_trace_width 0.5)
+    (last_trace_width 1.2)
     (user_trace_width 0.25)
     (user_trace_width 0.5)
@@
     )
   )
-  (gr_line (start 53 85) (end 143 85) (angle 90) (layer Edge.Cuts) (width 0.15))
-  (gr_line (start 143 150) (end 53 150) (angle 90) (layer Edge.Cuts) (width 0.15))
-  (gr_line (start 143 150) (end 143 85) (angle 90) (layer Edge.Cuts) (width 0.15))
-  (gr_text +3.3V (at 120.65 163.322 90) (layer F.Paste)
+  (gr_text +3.3V (at 92.8624 91.8464) (layer F.SilkS)
     (effects (font (size 1.5 1.5) (thickness 0.3)))
   )
-  (gr_text +5V (at 117.856 162.56 90) (layer F.Paste)
+  (gr_text +5V (at 91.7956 87.2744) (layer F.SilkS)
     (effects (font (size 1.5 1.5) (thickness 0.3)))
   )
-  (gr_text VCC (at 67.4488 137.8592 360) (layer F.Paste)
+  (gr_text "Robotronik CDFR 2018" (at 114.1984 87.7316) (layer F.SilkS)
     (effects (font (size 1.5 1.5) (thickness 0.3)))
   )
-  (gr_text VDD (at 70.8952 132.3496 360) (layer F.Paste)
+  (gr_line (start 53 85) (end 143 85) (angle 90) (layer Edge.Cuts) (width 0.15))
+  (gr_line (start 143 150) (end 53 150) (angle 90) (layer Edge.Cuts) (width 0.15))
+  (gr_line (start 143 150) (end 143 85) (angle 90) (layer Edge.Cuts) (width 0.15))
+  (gr_text VCC (at 67.4488 137.8592) (layer F.Paste)
     (effects (font (size 1.5 1.5) (thickness 0.3)))
   )
-  (gr_line (start 53 85) (end 53 150) (angle 90) (layer Edge.Cuts) (width 0.15))
-  (gr_line (start 53 125) (end 53 85) (angle 90) (layer Edge.Cuts) (width 0.15))
-  (gr_text Robotronik_CDFR_2018 (at 129.36 157.928) (layer F.Cu)
+  (gr_text VDD (at 70.8952 132.3496) (layer F.Paste)
     (effects (font (size 1.5 1.5) (thickness 0.3)))
   )
+  (gr_line (start 53 85) (end 53 150) (angle 90) (layer Edge.Cuts) (width 0.15))
+  (gr_line (start 53 125) (end 53 85) (angle 90) (layer Edge.Cuts) (width 0.15))
   (gr_line (start 110 100) (end 110 120) (layer F.SilkS) (width 0.2))
   (gr_line (start 96 100) (end 110 100) (layer F.SilkS) (width 0.2))
   (gr_line (start 96 120) (end 96 100) (layer F.SilkS) (width 0.2))
   (gr_line (start 110 120) (end 96 120) (layer F.SilkS) (width 0.2))
+  (via (at 123.846 129.032) (size 0.8) (drill 0.3) (layers F.Cu B.Cu) (net 1))
   (segment (start 120.65 121.888) (end 122.904 119.634) (width 1.2) (layer F.Cu) (net 1))
   (segment (start 122.904 119.634) (end 126.208 119.634) (width 1.2) (layer F.Cu) (net 1))
@@
   (segment (start 60.1452 139.3496) (end 60.1452 142.8548) (width 2) (layer B.Cu) (net 1))
   (segment (start 60.1452 142.8548) (end 58 145) (width 2) (layer B.Cu) (net 1))
-  (segment (start 119.823399 130.288976) (end 113.63206 136.480315) (width 0.25) (layer B.Cu) (net 2))
   (segment (start 113.63206 136.480315) (end 112.148529 136.480315) (width 0.25) (layer B.Cu) (net 2))
-  (segment (start 120.273599 128.538599) (end 119.823399 128.988799) (width 0.25) (layer B.Cu) (net 2))
-  (segment (start 128.509401 128.538599) (end 120.273599 128.538599) (width 0.25) (layer B.Cu) (net 2))
-  (segment (start 137.508999 119.539001) (end 128.509401 128.538599) (width 0.25) (layer B.Cu) (net 2))
-  (segment (start 138.684 115.57) (end 137.508999 116.745001) (width 0.25) (layer B.Cu) (net 2))
   (segment (start 119.823399 128.988799) (end 119.823399 130.288976) (width 0.25) (layer B.Cu) (net 2))
+  (segment (start 120.505199 128.306999) (end 119.823399 128.988799) (width 0.25) (layer B.Cu) (net 2))
+  (segment (start 137.508999 119.539001) (end 128.741001 128.306999) (width 0.25) (layer B.Cu) (net 2))
   (segment (start 137.508999 116.745001) (end 137.508999 119.539001) (width 0.25) (layer B.Cu) (net 2))
+  (segment (start 119.823399 130.288976) (end 113.63206 136.480315) (width 0.25) (layer B.Cu) (net 2))
+  (segment (start 138.684 115.57) (end 137.508999 116.745001) (width 0.25) (layer B.Cu) (net 2))
+  (segment (start 128.741001 128.306999) (end 120.505199 128.306999) (width 0.25) (layer B.Cu) (net 2))
   (segment (start 112.148529 136.480315) (end 111.582844 136.480315) (width 0.25) (layer B.Cu) (net 2))
   (segment (start 111.582844 135.91463) (end 111.582844 136.480315) (width 0.5) (layer F.Cu) (net 2))
