File: Electronique/moteurs_brushless_elec/PCB/motor_part.sch (KiCad schematic (older format))
At the start: 36 parts, among them K1 Maxon-200142, K2 Maxon-200142, U1 L6235D, U2 L6235D

Commit message: ajout valeurs
Parts:
- C1, C2: value C -> 10nC
- R1, R3: value R -> 1.2kR
- R2, R4: value R -> 220R
- Rsense1, Rsense2: value 0.03R -> 0.33R
Changed lines of the file:
@@
 P 2350 1850
 F 0 "Rsense1" V 2430 1850 50  0000 C CNN
-F 1 "0.03R" V 2350 1850 50  0000 C CNN
+F 1 "0.33R" V 2350 1850 50  0000 C CNN
 F 2 "Resistors_THT:R_Bare_Metal_Element_L12.4mm_W4.8mm_P11.40mm" V 2280 1850 50  0001 C CNN
 F 3 "" H 2350 1850 50  0001 C CNN
@@
 P 4550 4800
 F 0 "R1" V 4630 4800 50  0000 C CNN
-F 1 "R" V 4550 4800 50  0000 C CNN
+F 1 "1.2kR" V 4550 4800 50  0000 C CNN
 F 2 "Resistors_THT:R_Axial_DIN0207_L6.3mm_D2.5mm_P10.16mm_Horizontal" V 4480 4800 50  0001 C CNN
 F 3 "" H 4550 4800 50  0001 C CNN
@@
 P 5000 5100
 F 0 "R2" V 5080 5100 50  0000 C CNN
-F 1 "R" V 5000 5100 50  0000 C CNN
+F 1 "220R" V 5000 5100 50  0000 C CNN
 F 2 "Resistors_THT:R_Axial_DIN0207_L6.3mm_D2.5mm_P10.16mm_Horizontal" V 4930 5100 50  0001 C CNN
 F 3 "" H 5000 5100 50  0001 C CNN
@@
 P 5250 5100
 F 0 "C1" H 5275 5200 50  0000 L CNN
-F 1 "C" H 5275 5000 50  0000 L CNN
+F 1 "10nC" H 5275 5000 50  0000 L CNN
 F 2 "Capacitors_SMD:C_1206_HandSoldering" H 5288 4950 50  0001 C CNN
 F 3 "" H 5250 5100 50  0001 C CNN
@@
 P 9500 1750
 F 0 "Rsense2" V 9580 1750 50  0000 C CNN
-F 1 "0.03R" V 9500 1750 50  0000 C CNN
+F 1 "0.33R" V 9500 1750 50  0000 C CNN
 F 2 "Resistors_THT:R_Bare_Metal_Element_L12.4mm_W4.8mm_P11.40mm" V 9430 1750 50  0001 C CNN
 F 3 "" H 9500 1750 50  0001 C CNN
@@
 P 11700 4700
 F 0 "R3" V 11780 4700 50  0000 C CNN
-F 1 "R" V 11700 4700 50  0000 C CNN
+F 1 "1.2kR" V 11700 4700 50  0000 C CNN
 F 2 "Resistors_THT:R_Axial_DIN0207_L6.3mm_D2.5mm_P10.16mm_Horizontal" V 11630 4700 50  0001 C CNN
 F 3 "" H 11700 4700 50  0001 C CNN
@@
 P 12150 5000
 F 0 "R4" V 12230 5000 50  0000 C CNN
-F 1 "R" V 12150 5000 50  0000 C CNN
+F 1 "220R" V 12150 5000 50  0000 C CNN
 F 2 "Resistors_THT:R_Axial_DIN0207_L6.3mm_D2.5mm_P10.16mm_Horizontal" V 12080 5000 50  0001 C CNN
 F 3 "" H 12150 5000 50  0001 C CNN
@@
 P 12400 5000
 F 0 "C2" H 12425 5100 50  0000 L CNN
-F 1 "C" H 12425 4900 50  0000 L CNN
+F 1 "10nC" H 12425 4900 50  0000 L CNN
 F 2 "Capacitors_SMD:C_1206_HandSoldering" H 12438 4850 50  0001 C CNN
 F 3 "" H 12400 5000 50  0001 C CNN
