File: Electronique/driver_moteurs/power_part.sch (KiCad schematic (older format))
At the start: 19 parts, among them U3 B_Plug_5mm, U4 LM317_SOT223, U5 LM317_SOT223

Commit message: modif moteur axe z
Parts:
- added C8: CP, symbol CP
- added C9: C, symbol C
- added D6: D, symbol D
- added F2: F_Small, symbol F_Small
- added U9: B_Plug_5mm, symbol B_Plug_5mm
- R10, R7: value R -> 470R
- R6: value R -> 2kR
Connections:
- net labels added: +9V
- wire segments 42 -> 54

Commit message: axe z routage en cours
Parts:
- C4, C8: footprint (none) -> Capacitors_THT:CP_Radial_D8.0mm_P3.50mm
- C5, C6, C7, C9: footprint (none) -> Capacitors_SMD:C_1206_HandSoldering
- D2, D6: footprint (none) -> Diodes_SMD:D_SMA_Handsoldering
- D3, D4, D5: footprint (none) -> Diodes_SMD:D_SMA-SMB_Universal_Handsoldering
- F1, F2: footprint (none) -> Fuse_Holders_and_Fuses:Fuseholder5x20_horiz_SemiClosed_Casing10x25mm
- R10, R4, R5, R6, R7, R8, R9: footprint (none) -> Resistors_SMD:R_1206_HandSoldering
- U3, U9: footprint (none) -> B plug:B plug 5mm
- U4, U5: footprint (none) -> TO_SOT_Packages_SMD:SOT-223-3Lead_TabPin2

Commit message: Correction schéma driver
Parts:
- D3, D4, D5: symbol LED -> LED-RESCUE-driver-moteurs
- U5: footprint TO_SOT_Packages_SMD:SOT-223-3Lead_TabPin2 -> (none)
Connections:
- wire segments 54 -> 52
Changed lines of the file:
@@
 EESchema Schematic File Version 2
+LIBS:driver-moteurs-rescue
 LIBS:power
 LIBS:device
@@
 $EndComp
 $Comp
-L LED D3
+L LED-RESCUE-driver-moteurs D3
 U 1 1 59F75E2C
 P 5500 2850
+AR Path="/59F75E2C" Ref="D3"  Part="1"
+AR Path="/59F75CC2/59F75E2C" Ref="D3"  Part="1"
 F 0 "D3" H 5500 2950 50  0000 C CNN
 F 1 "LED" H 5500 2750 50  0000 C CNN
@@
 $EndComp
 $Comp
-L PWR_FLAG #FLG036
-U 1 1 59F761CD
-P 4450 2200
-F 0 "#FLG036" H 4450 2295 50  0001 C CNN
-F 1 "PWR_FLAG" H 4450 2380 50  0000 C CNN
-F 2 "" H 4450 2200 50  0000 C CNN
-F 3 "" H 4450 2200 50  0000 C CNN
-	1    4450 2200
-	1    0    0    -1
-$EndComp
-$Comp
-L GND #PWR037
+L GND #PWR036
 U 1 1 59F763B8
 P 3000 3200
-F 0 "#PWR037" H 3000 2950 50  0001 C CNN
+F 0 "#PWR036" H 3000 2950 50  0001 C CNN
 F 1 "GND" H 3000 3050 50  0000 C CNN
 F 2 "" H 3000 3200 50  0000 C CNN
@@
 $EndComp
 $Comp
-L GND #PWR038
+L GND #PWR037
 U 1 1 59F763D8
 P 5500 3200
-F 0 "#PWR038" H 5500 2950 50  0001 C CNN
+F 0 "#PWR037" H 5500 2950 50  0001 C CNN
 F 1 "GND" H 5500 3050 50  0000 C CNN
 F 2 "" H 5500 3200 50  0000 C CNN
@@
 $EndComp
 $Comp
-L PWR_FLAG #FLG039
+L PWR_FLAG #FLG038
 U 1 1 59F76416
 P 3250 3200
-F 0 "#FLG039" H 3250 3295 50  0001 C CNN
+F 0 "#FLG038" H 3250 3295 50  0001 C CNN
 F 1 "PWR_FLAG" H 3250 3380 50  0000 C CNN
 F 2 "" H 3250 3200 50  0000 C CNN
@@
 $EndComp
 $Comp
-L LM317_SOT223 U5
-U 1 1 59F76469
-P 7850 2500
-F 0 "U5" H 7850 2800 50  0000 C CNN
-F 1 "LM317_SOT223" H 7900 2250 50  0000 L CNN
-F 2 "TO_SOT_Packages_SMD:SOT-223-3Lead_TabPin2" H 7850 2500 50  0001 C CNN
-F 3 "" H 7850 2500 50  0000 C CNN
-	1    7850 2500
-	1    0    0    -1
-$EndComp
-$Comp
-L VCC #PWR040
+L VCC #PWR039
 U 1 1 59F764CC
 P 7000 2250
-F 0 "#PWR040" H 7000 2100 50  0001 C CNN
+F 0 "#PWR039" H 7000 2100 50  0001 C CNN
 F 1 "VCC" H 7000 2400 50  0000 C CNN
 F 2 "" H 7000 2250 50  0000 C CNN
@@
 Connection ~ 4750 2400
 Wire Wire Line
-	4450 2200 4450 2250
-Wire Wire Line
-	4450 2250 4750 2250
-Connection ~ 4750 2250
-Wire Wire Line
 	5200 2400 5500 2400
 Wire Wire Line
@@
 Connection ~ 3000 3000
 Wire Wire Line
-	7450 2350 7000 2350
-Wire Wire Line
 	7000 2350 7000 2250
 Wire Wire Line
 	8650 3100 7850 3100
-Wire Wire Line
-	7850 2850 7850 3250
 Connection ~ 7850 3100
 $Comp
-L GND #PWR041
+L GND #PWR040
 U 1 1 59F76711
 P 7850 3700
-F 0 "#PWR041" H 7850 3450 50  0001 C CNN
+F 0 "#PWR040" H 7850 3450 50  0001 C CNN
 F 1 "GND" H 7850 3550 50  0000 C CNN
 F 2 "" H 7850 3700 50  0000 C CNN
@@
 $EndComp
 $Comp
-L LED D5
+L LED-RESCUE-driver-moteurs D5
 U 1 1 59F7690E
 P 10600 2750
+AR Path="/59F7690E" Ref="D5"  Part="1"
+AR Path="/59F75CC2/59F7690E" Ref="D5"  Part="1"
 F 0 "D5" H 10600 2850 50  0000 C CNN
 F 1 "LED" H 10600 2650 50  0000 C CNN
@@
 $EndComp
 Wire Wire Line
-	8250 2350 9750 2350
-Wire Wire Line
 	8650 2350 8650 2800
 Connection ~ 9300 2350
@@
 	9300 2900 9300 3150
 $Comp
-L +5V #PWR042
+L +5V #PWR041
 U 1 1 59F76B40
 P 9300 2100
-F 0 "#PWR042" H 9300 1950 50  0001 C CNN
+F 0 "#PWR041" H 9300 1950 50  0001 C CNN
 F 1 "+5V" H 9300 2240 50  0000 C CNN
 F 2 "" H 9300 2100 50  0000 C CNN
@@
 $EndComp
 $Comp
-L GND #PWR043
+L GND #PWR042
 U 1 1 59F76BEF
 P 9300 3150
-F 0 "#PWR043" H 9300 2900 50  0001 C CNN
+F 0 "#PWR042" H 9300 2900 50  0001 C CNN
 F 1 "GND" H 9300 3000 50  0000 C CNN
 F 2 "" H 9300 3150 50  0000 C CNN
@@
 $EndComp
 $Comp
-L GND #PWR044
+L GND #PWR043
 U 1 1 59F76C21
 P 10600 3200
-F 0 "#PWR044" H 10600 2950 50  0001 C CNN
+F 0 "#PWR043" H 10600 2950 50  0001 C CNN
 F 1 "GND" H 10600 3050 50  0000 C CNN
 F 2 "" H 10600 3200 50  0000 C CNN
@@
 $EndComp
 $Comp
-L VCC #PWR045
+L VCC #PWR044
 U 1 1 59F77053
 P 2450 4700
-F 0 "#PWR045" H 2450 4550 50  0001 C CNN
+F 0 "#PWR044" H 2450 4550 50  0001 C CNN
 F 1 "VCC" H 2450 4850 50  0000 C CNN
 F 2 "" H 2450 4700 50  0000 C CNN
@@
 Connection ~ 3300 5550
 $Comp
-L GND #PWR046
+L GND #PWR045
 U 1 1 59F7706A
 P 3300 6150
-F 0 "#PWR046" H 3300 5900 50  0001 C CNN
+F 0 "#PWR045" H 3300 5900 50  0001 C CNN
 F 1 "GND" H 3300 6000 50  0000 C CNN
 F 2 "" H 3300 6150 50  0000 C CNN
@@
 $EndComp
 $Comp
-L LED D4
+L LED-RESCUE-driver-moteurs D4
 U 1 1 59F7707D
 P 6050 5200
+AR Path="/59F7707D" Ref="D4"  Part="1"
+AR Path="/59F75CC2/59F7707D" Ref="D4"  Part="1"
 F 0 "D4" H 6050 5300 50  0000 C CNN
 F 1 "LED" H 6050 5100 50  0000 C CNN
@@
 	4750 5350 4750 5600
 $Comp
-L GND #PWR047
+L GND #PWR046
 U 1 1 59F7709B
 P 4750 5600
-F 0 "#PWR047" H 4750 5350 50  0001 C CNN
+F 0 "#PWR046" H 4750 5350 50  0001 C CNN
 F 1 "GND" H 4750 5450 50  0000 C CNN
 F 2 "" H 4750 5600 50  0000 C CNN
@@
 $EndComp
 $Comp
-L GND #PWR048
+L GND #PWR047
 U 1 1 59F770A1
 P 6050 5650
-F 0 "#PWR048" H 6050 5400 50  0001 C CNN
+F 0 "#PWR047" H 6050 5400 50  0001 C CNN
 F 1 "GND" H 6050 5500 50  0000 C CNN
 F 2 "" H 6050 5650 50  0000 C CNN
@@
 $EndComp
 $Comp
-L +3.3V #PWR049
+L +3.3V #PWR048
 U 1 1 59F7712F
 P 4750 4550
-F 0 "#PWR049" H 4750 4400 50  0001 C CNN
+F 0 "#PWR048" H 4750 4400 50  0001 C CNN
 F 1 "+3.3V" H 4750 4690 50  0000 C CNN
 F 2 "" H 4750 4550 50  0000 C CNN
@@
 $EndComp
 $Comp
-L GND #PWR050
+L GND #PWR049
 U 1 1 5A3E7A0F
 P 7300 5350
-F 0 "#PWR050" H 7300 5100 50  0001 C CNN
+F 0 "#PWR049" H 7300 5100 50  0001 C CNN
 F 1 "GND" H 7300 5200 50  0000 C CNN
 F 2 "" H 7300 5350 50  0000 C CNN
@@
 $EndComp
 $Comp
-L +9V #PWR051
+L +9V #PWR050
 U 1 1 5A3E7A4B
 P 8550 4700
-F 0 "#PWR051" H 8550 4550 50  0001 C CNN
+F 0 "#PWR050" H 8550 4550 50  0001 C CNN
 F 1 "+9V" H 8550 4840 50  0000 C CNN
 F 2 "" H 8550 4700 50  0000 C CNN
@@
 Connection ~ 8550 4800
 $Comp
-L GND #PWR052
+L GND #PWR051
 U 1 1 5A3E7EEF
 P 8350 5600
-F 0 "#PWR052" H 8350 5350 50  0001 C CNN
+F 0 "#PWR051" H 8350 5350 50  0001 C CNN
 F 1 "GND" H 8350 5450 50  0000 C CNN
 F 2 "" H 8350 5600 50  0000 C CNN
@@
 Wire Wire Line
 	7300 4900 7200 4900
+$Comp
+L LM317_SOT223 U5
+U 1 1 5A4AB301
+P 7850 2500
+F 0 "U5" H 7850 2800 50  0000 C CNN
+F 1 "LM317_SOT223" H 7900 2250 50  0000 L CNN
+F 2 "" H 7850 2500 50  0000 C CNN
+F 3 "" H 7850 2500 50  0000 C CNN
+	1    7850 2500
+	1    0    0    -1
+$EndComp
+Wire Wire Line
+	7000 2350 7450 2350
+Wire Wire Line
+	8250 2350 9750 2350
+Wire Wire Line
+	7850 2850 7850 3250
 $EndSCHEMATC

Commit message: Correction PCB driver moteurs
Parts:
- U5: footprint (none) -> TO_SOT_Packages_SMD:SOT-223-3_TabPin2
Connections:
- net VCC renamed VDD
Changed lines of the file:
@@
-$EndComp
-$Comp
-L VCC #PWR035
-U 1 1 59F761AB
-P 4750 2200
-F 0 "#PWR035" H 4750 2050 50  0001 C CNN
-F 1 "VCC" H 4750 2350 50  0000 C CNN
-F 2 "" H 4750 2200 50  0000 C CNN
-F 3 "" H 4750 2200 50  0000 C CNN
-	1    4750 2200
-	1    0    0    -1
 $EndComp
 $Comp
@@
 	1    3250 3200
 	-1   0    0    1
-$EndComp
-$Comp
-L VCC #PWR039
-U 1 1 59F764CC
-P 7000 2250
-F 0 "#PWR039" H 7000 2100 50  0001 C CNN
-F 1 "VCC" H 7000 2400 50  0000 C CNN
-F 2 "" H 7000 2250 50  0000 C CNN
-F 3 "" H 7000 2250 50  0000 C CNN
-	1    7000 2250
-	1    0    0    -1
 $EndComp
 $Comp
@@
 $EndComp
 $Comp
-L VCC #PWR044
-U 1 1 59F77053
-P 2450 4700
-F 0 "#PWR044" H 2450 4550 50  0001 C CNN
-F 1 "VCC" H 2450 4850 50  0000 C CNN
-F 2 "" H 2450 4700 50  0000 C CNN
-F 3 "" H 2450 4700 50  0000 C CNN
-	1    2450 4700
-	1    0    0    -1
-$EndComp
-$Comp
 L R R4
 U 1 1 59F77059
@@
 F 0 "U5" H 7850 2800 50  0000 C CNN
 F 1 "LM317_SOT223" H 7900 2250 50  0000 L CNN
-F 2 "" H 7850 2500 50  0000 C CNN
+F 2 "TO_SOT_Packages_SMD:SOT-223-3_TabPin2" H 7850 2500 50  0001 C CNN
 F 3 "" H 7850 2500 50  0000 C CNN
 	1    7850 2500
@@
 Wire Wire Line
 	7850 2850 7850 3250
+$Comp
+L VDD #PWR?
+U 1 1 5A4B034E
+P 4750 2200
+F 0 "#PWR?" H 4750 2050 50  0001 C CNN
+F 1 "VDD" H 4750 2350 50  0000 C CNN
+F 2 "" H 4750 2200 50  0001 C CNN
+F 3 "" H 4750 2200 50  0001 C CNN
+	1    4750 2200
+	1    0    0    -1
+$EndComp
+$Comp
+L VDD #PWR?
+U 1 1 5A4B043B
+P 7000 2250
+F 0 "#PWR?" H 7000 2100 50  0001 C CNN
+F 1 "VDD" H 7000 2400 50  0000 C CNN
+F 2 "" H 7000 2250 50  0001 C CNN
+F 3 "" H 7000 2250 50  0001 C CNN
+	1    7000 2250
+	1    0    0    -1
+$EndComp
+$Comp
+L VDD #PWR?
+U 1 1 5A4B05B8
+P 2450 4700
+F 0 "#PWR?" H 2450 4550 50  0001 C CNN
+F 1 "VDD" H 2450 4850 50  0000 C CNN
+F 2 "" H 2450 4700 50  0001 C CNN
+F 3 "" H 2450 4700 50  0001 C CNN
+	1    2450 4700
+	1    0    0    -1
+$EndComp
 $EndSCHEMATC

Commit message: valeurs de resistance manquantes
Parts:
- R4: value R -> 390R
- R5: value R -> 220R
- R8: value R -> 820R
- R9: value R -> 270R
Changed lines of the file:
@@
 P 7850 3400
 F 0 "R8" V 7930 3400 50  0000 C CNN
-F 1 "R" V 7850 3400 50  0000 C CNN
+F 1 "820R" V 7850 3400 50  0000 C CNN
 F 2 "Resistors_SMD:R_1206_HandSoldering" V 7780 3400 50  0001 C CNN
 F 3 "" H 7850 3400 50  0000 C CNN
@@
 P 8650 2950
 F 0 "R9" V 8730 2950 50  0000 C CNN
-F 1 "R" V 8650 2950 50  0000 C CNN
+F 1 "270R" V 8650 2950 50  0000 C CNN
 F 2 "Resistors_SMD:R_1206_HandSoldering" V 8580 2950 50  0001 C CNN
 F 3 "" H 8650 2950 50  0000 C CNN
@@
 P 3300 5850
 F 0 "R4" V 3380 5850 50  0000 C CNN
-F 1 "R" V 3300 5850 50  0000 C CNN
+F 1 "390R" V 3300 5850 50  0000 C CNN
 F 2 "Resistors_SMD:R_1206_HandSoldering" V 3230 5850 50  0001 C CNN
 F 3 "" H 3300 5850 50  0000 C CNN
@@
 P 4100 5400
 F 0 "R5" V 4180 5400 50  0000 C CNN
-F 1 "R" V 4100 5400 50  0000 C CNN
+F 1 "220R" V 4100 5400 50  0000 C CNN
 F 2 "Resistors_SMD:R_1206_HandSoldering" V 4030 5400 50  0001 C CNN
 F 3 "" H 4100 5400 50  0000 C CNN
