File: Electronique/Central/central.kicad_pcb (KiCad board)
At the start: 2 copper layers, 2 parts, among them U1 Nucleo-64, U2 APE8865U5-28-HF-3

Commit message: led!
Parts:
- added F1: FUSE, Fuse_Holders_and_Fuses:Fuseholder5x20_horiz_SemiClosed_Casing10x25mm, F.Cu at (54.6, 91.9)
- added F2: FUSE, Fuse_Holders_and_Fuses:Fuseholder5x20_horiz_SemiClosed_Casing10x25mm, F.Cu at (57.2, 119.2)
- added P2: CONN_Speaker, Connectors_Molex:Molex_KK-6410-02_02x2.54mm_Straight, F.Cu at (37.2, 25.4)
- added P3: CONN_jack, Pin_Headers:Pin_Header_Straight_1x02_Pitch2.54mm, F.Cu at (17.4, 25.2)
- added U3: I2C_repeater, Housings_SOIC:SOIC-8_3.9x4.9mm_Pitch1.27mm, F.Cu at (137.3, 55.8)
- added U4: TDA8541, Housings_SOIC:SOIC-8_3.9x4.9mm_Pitch1.27mm, F.Cu at (26.1, 25.1)
- added U5: B_Plug_5mm, dsn2596:B plug 5mm, F.Cu at (44.2, 101.8)
- added U6: B_Plug_5mm, dsn2596:B plug 5mm, F.Cu at (42.8, 122.1)
- added U7: DSN2596, dsn2596:DSN2596, F.Cu at (113.3, 100.3)
- added U8: DSN2596, dsn2596:DSN2596, F.Cu at (113.3, 127.3)
Connections:
- U1 pad 32: (no net) -> +3V3
- U1 pad 37: (no net) -> +5V
- U1 pad 66: (no net) -> I2C_TOF_SDA
- U1 pad 67: (no net) -> I2C_TOF_EN
- U1 pad 68: (no net) -> I2C_TOF_SCL
- U2 pad 2: (no net) -> GND
- U2 pad 5: (no net) -> +2.8V
