File: Electronique/Central/central.kicad_pcb (KiCad board)
At the start: 2 copper layers, 182 x 90 mm, 58 parts, among them P1 CONN_02X03, P10 CONN_Selec, P11 CONN_01X02, P12 CONN_01X02, P13 CONN_01X02, P14 CONN_01X02, P15 CONN_01X02, P2 CONN_Speaker, P3 CONN_jack, P4 CONN_jacky_led, P5 CONN_LED, P6 CONN_02X03, P7 CONN_02X03, P8 CONN_02X03, P9 CONN_jack_start, Q1 IRF540N, U1 Nucleo-64, U10 trou-d3mm, U11 trou-d3mm, U12 trou-d3mm, U13 trou-d3mm, U14 trou-d3mm, U15 trou-d3mm, U2 APE8865U5-28-HF-3, U3 I2C_repeater, U4 TDA8541, U5 B_Plug_5mm, U6 B_Plug_5mm, U7 DSN2596, U8 DSN2596, U9 MC34152

Commit message: pdf export and corrections
Routing:
- net Net-(P1-Pad4): track 434.8 -> 440.0 mm, vias 4 -> 5
- net GND: track 826.4 -> 831.2 mm
- net Net-(D4-Pad2): track 102.4 -> 103.7 mm, vias 1 -> 2
Other:
- net class Default: trace_width 0.5 -> 1
- board text added: "Robotronik_CDFR_2018 Central"
Changed lines of the file:
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@@
-(kicad_pcb (version 4) (host pcbnew 4.0.7)
+(kicad_pcb (version 4) (host pcbnew 4.0.2+dfsg1-stable)
   (general
     (links 128)
     (no_connects 0)
-    (area 63.949999 67.949999 246.050001 158.050001)
+    (area 49.899999 49.899999 260.100001 168.100001)
     (thickness 1.6)
-    (drawings 37)
-    (tracks 572)
+    (drawings 38)
+    (tracks 580)
     (zones 0)
     (modules 58)
@@
     (visible_elements FFFFEF7F)
     (pcbplotparams
-      (layerselection 0x00030_80000001)
+      (layerselection 0x00000_80000000)
       (usegerberextensions false)
       (excludeedgelayer true)
@@
       (padsonsilk false)
       (subtractmaskfromsilk false)
-      (outputformat 1)
+      (outputformat 4)
       (mirror false)
-      (drillshape 1)
+      (drillshape 2)
       (scaleselection 1)
       (outputdirectory ""))
@@
   (net_class Default "This is the default net class."
     (clearance 0.2)
-    (trace_width 0.5)
+    (trace_width 1)
     (via_dia 1.2)
     (via_drill 0.8)
@@
       (net 2 GND))
   )
+  (gr_text "Robotronik_CDFR_2018\nCentral" (at 150 76) (layer F.Cu)
+    (effects (font (size 1.5 1.5) (thickness 0.3)))
+  )
   (gr_circle (center 94 143) (end 94 133) (layer F.Paste) (width 0.2))
   (gr_circle (center 216 143) (end 215.4 133) (layer Edge.Cuts) (width 0.1))
@@
   (segment (start 157.119999 143.314999) (end 157.119999 144.685001) (width 0.5) (layer F.Cu) (net 1))
   (segment (start 157.119999 144.685001) (end 157.384998 144.95) (width 0.5) (layer F.Cu) (net 1))
+  (segment (start 219 70) (end 236 70) (width 1) (layer B.Cu) (net 2))
+  (segment (start 236 70) (end 240 74) (width 1) (layer B.Cu) (net 2))
+  (segment (start 214.3 77) (end 214.3 74.7) (width 1) (layer B.Cu) (net 2))
+  (segment (start 214.3 74.7) (end 219 70) (width 1) (layer B.Cu) (net 2))
   (segment (start 174 134.095) (end 177.3 134.095) (width 1) (layer F.Cu) (net 2))
   (segment (start 160.4 146) (end 162.095 146) (width 0.5) (layer B.Cu) (net 2))
@@
   (segment (start 162 134) (end 159 134) (width 1) (layer B.Cu) (net 2))
   (segment (start 156 134) (end 159 134) (width 1) (layer B.Cu) (net 2))
-  (segment (start 240 74) (end 217 74) (width 1) (layer B.Cu) (net 2))
-  (segment (start 217 74) (end 214.3 76.7) (width 1) (layer B.Cu) (net 2))
   (segment (start 214.3 76.7) (end 214.3 77) (width 1) (layer B.Cu) (net 2))
   (segment (start 202.5 122) (end 202.5 124.08) (width 1) (layer B.Cu) (net 2))
@@
   (segment (start 185.872927 75.46) (end 198.727208 75.46) (width 1) (layer B.Cu) (net 9))
   (segment (start 161.880001 107.180001) (end 182.509988 86.550014) (width 1) (layer B.Cu) (net 9))
+  (segment (start 205 76) (end 205.54 75.46) (width 1) (layer B.Cu) (net 10))
+  (segment (start 205.54 75.46) (end 208 75.46) (width 1) (layer B.Cu) (net 10))
+  (segment (start 204 76) (end 205 76) (width 1) (layer B.Cu) (net 10))
+  (segment (start 202.587207 79.600001) (end 202.587207 77.412793) (width 1) (layer F.Cu) (net 10))
+  (segment (start 202.587207 77.412793) (end 204 76) (width 1) (layer F.Cu) (net 10))
+  (via (at 204 76) (size 1.2) (drill 0.8) (layers F.Cu B.Cu) (net 10))
   (segment (start 194 77) (end 196.600001 79.600001) (width 1) (layer F.Cu) (net 10))
   (segment (start 196.600001 79.600001) (end 202.587207 79.600001) (width 1) (layer F.Cu) (net 10))
-  (segment (start 202.587207 79.600001) (end 206.727208 75.46) (width 1) (layer F.Cu) (net 10))
-  (segment (start 206.727208 75.46) (end 208 75.46) (width 1) (layer F.Cu) (net 10))
   (segment (start 183.709999 87.069999) (end 183.709999 79.319999) (width 1) (layer B.Cu) (net 10))
   (segment (start 160.259998 110.52) (end 183.709999 87.069999) (width 1) (layer B.Cu) (net 10))
@@
   (segment (start 89.78 70.84) (end 91.86863 70.84) (width 1) (layer B.Cu) (net 15))
   (segment (start 91.86863 70.84) (end 93 70.84) (width 1) (layer B.Cu) (net 15))
+  (segment (start 221 72) (end 219.38 73.62) (width 1) (layer B.Cu) (net 16))
+  (segment (start 219.38 73.62) (end 219.38 77) (width 1) (layer B.Cu) (net 16))
+  (segment (start 228.700001 73.700001) (end 227 72) (width 1) (layer F.Cu) (net 16))
+  (segment (start 227 72) (end 221 72) (width 1) (layer F.Cu) (net 16))
+  (via (at 221 72) (size 1.2) (drill 0.8) (layers F.Cu B.Cu) (net 16))
+  (segment (start 228.700001 110.792269) (end 228.700001 73.700001) (width 1) (layer F.Cu) (net 16))
   (segment (start 93.2 78.284004) (end 93.6 77.884004) (width 1) (layer B.Cu) (net 16))
   (segment (start 73.4 141.6) (end 72.299999 140.499999) (width 1) (layer F.Cu) (net 16))
@@
   (segment (start 229.319246 137.832226) (end 229.319246 138.680754) (width 1) (layer F.Cu) (net 16))
   (segment (start 229.319246 115.826976) (end 229.319246 137.832226) (width 1) (layer F.Cu) (net 16))
-  (segment (start 228.260002 74.7) (end 228.700001 75.139999) (width 1) (layer F.Cu) (net 16))
-  (segment (start 219.38 76.7) (end 221.38 74.7) (width 1) (layer F.Cu) (net 16))
   (segment (start 219.38 77) (end 219.38 76.7) (width 1) (layer F.Cu) (net 16))
-  (segment (start 221.38 74.7) (end 228.260002 74.7) (width 1) (layer F.Cu) (net 16))
   (via (at 229.319246 138.680754) (size 1.2) (drill 0.8) (layers F.Cu B.Cu) (net 16))
   (segment (start 227.29999 112.19228) (end 227.29999 113.80772) (width 1) (layer F.Cu) (net 16))
-  (segment (start 228.700001 75.139999) (end 228.700001 110.792269) (width 1) (layer F.Cu) (net 16))
   (segment (start 228.700001 110.792269) (end 227.29999 112.19228) (width 1) (layer F.Cu) (net 16))
   (segment (start 227.29999 113.80772) (end 229.319246 115.826976) (width 1) (layer F.Cu) (net 16))
@@
     (connect_pads (clearance 0.508))
     (min_thickness 0.254)
-    (fill (arc_segments 16) (thermal_gap 0.508) (thermal_bridge_width 0.508))
+    (fill yes (arc_segments 16) (thermal_gap 0.508) (thermal_bridge_width 0.508))
     (polygon
       (pts
@@
     (connect_pads (clearance 0.508))
     (min_thickness 0.254)
-    (fill (arc_segments 16) (thermal_gap 0.508) (thermal_bridge_width 0.508))
+    (fill yes (arc_segments 16) (thermal_gap 0.508) (thermal_bridge_width 0.508))
     (polygon
       (pts
@@
       )
     )
+  )
+  (zone (net 2) (net_name GND) (layer F.Cu) (hatch edge 0.508)
+    (connect_pads (clearance 1))
+    (min_thickness 0.254)
+    (fill yes (arc_segments 16) (thermal_gap 0.508) (thermal_bridge_width 0.508))
+    (polygon
+      (pts
+        (xy 64 158) (xy 246 158) (xy 246 68) (xy 64 68)
+      )
+    )
+  )
+  (zone (net 2) (net_name GND) (layer B.Cu) (hatch edge 0.508)
+    (connect_pads (clearance 1))
+    (min_thickness 0.254)
+    (fill yes (arc_segments 16) (thermal_gap 0.508) (thermal_bridge_width 0.508))
+    (polygon
+      (pts
+        (xy 64 158) (xy 246 158) (xy 246 68) (xy 64 68)
+      )
+    )
