File: Electronique/Central/central.kicad_pcb (KiCad board)
At the start: 2 copper layers, 182 x 90 mm, 58 parts, among them P1 CONN_02X03, P10 CONN_Selec, P11 CONN_01X02, P12 CONN_01X02, P13 CONN_01X02, P14 CONN_01X02, P15 CONN_01X02, P2 CONN_Speaker, P3 CONN_jack, P4 CONN_jacky_led, P5 CONN_LED, P6 CONN_02X03, P7 CONN_02X03, P8 CONN_02X03, P9 CONN_jack_start, Q1 IRF540N, U1 Nucleo-64, U10 trou-d3mm, U11 trou-d3mm, U12 trou-d3mm, U13 trou-d3mm, U14 trou-d3mm, U15 trou-d3mm, U2 APE8865U5-28-HF-3, U3 I2C_repeater, U4 TDA8541, U5 B_Plug_5mm, U6 B_Plug_5mm, U7 DSN2596, U8 DSN2596, U9 MC34152

Commit message: PCB Central
Parts:
- removed U15: trou-d3mm, Mounting_Holes:MountingHole_3.2mm_M3_Pad
- moved R13 33.4 mm to (97.0, 120.0), turned to 180 degrees
- moved R12 33.0 mm to (210.6, 156.0), turned to 180 degrees
- moved R8 28.3 mm to (213.0, 156.0), turned to 0 degrees
- moved R9 26.2 mm to (97.0, 123.0), turned to 180 degrees
- moved U14 25.6 mm to (88.0, 130.0)
- moved P4 17.0 mm to (225.0, 124.0)
- moved P5 17.0 mm to (225.0, 130.0)
- moved P7 16.6 mm to (235.0, 132.0)
- moved U9 15.0 mm to (219.0, 129.0)
- moved Q1 14.0 mm to (205.0, 125.0)
- moved P12 5.89 mm to (70.0, 121.2)
- moved D1 5.00 mm to (229.0, 82.0)
- moved D3 5.00 mm to (195.0, 78.0)
- moved D4 5.00 mm to (203.0, 78.0)
- moved P6 5.00 mm to (222.0, 77.0)
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Routing:
- net Net-(P1-Pad4): track 440.0 -> 298.9 mm, vias 5 -> 4
- net GND: track 831.2 -> 729.6 mm
- net Net-(P1-Pad2): track 368.7 -> 315.9 mm, vias 5 -> 6
- net Net-(P7-Pad1): track 12.0 -> 62.8 mm
- net Net-(P7-Pad3): track 7.34 -> 54.7 mm, vias 0 -> 1
- net +5V: track 194.5 -> 158.6 mm, vias 4 -> 1
- net Net-(P5-Pad2): track 26.5 -> 0.00 mm
- net Net-(P8-Pad3): track 9.00 -> 23.5 mm
- net BATT: track 90.6 -> 79.0 mm
- net Net-(P8-Pad1): track 11.5 -> 22.7 mm
- net Net-(P4-Pad1): track 9.02 -> 0.00 mm
- net +2.8V: track 427.3 -> 420.7 mm, vias 3 -> 2
- net Net-(D3-Pad2): track 91.2 -> 85.2 mm
- net Net-(C3-Pad1): track 31.9 -> 27.4 mm
- net /Pince_TX: track 62.1 -> 58.7 mm
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Other:
- board size 182 x 90 mm -> 175 x 90 mm

Commit message: pcb modif
Routing:
- net GND: track 729.6 -> 770.6 mm, vias 6 -> 8
- net Net-(P5-Pad2): track 0.00 -> 21.3 mm
- net Net-(P4-Pad1): track 0.00 -> 7.02 mm
- net +2.8V: track 420.7 -> 424.1 mm
Other:
- net class Default: trace_width 1 -> 2
Changed lines of the file:
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@@
-(kicad_pcb (version 4) (host pcbnew 4.0.7)
+(kicad_pcb (version 4) (host pcbnew 4.0.2+dfsg1-stable)
   (general
     (links 127)
-    (no_connects 10)
-    (area 63.949999 67.949999 239.050001 158.050001)
+    (no_connects 0)
+    (area 49.899999 49.899999 260.100001 168.100001)
     (thickness 1.6)
     (drawings 41)
-    (tracks 565)
+    (tracks 583)
     (zones 0)
     (modules 57)
@@
   )
   (setup
-    (last_trace_width 1)
+    (last_trace_width 2)
     (user_trace_width 0.5)
     (user_trace_width 1)
@@
     (visible_elements FFFFEF7F)
     (pcbplotparams
-      (layerselection 0x00000_80000000)
+      (layerselection 0x00000_00000001)
       (usegerberextensions false)
       (excludeedgelayer true)
@@
       (subtractmaskfromsilk false)
       (outputformat 4)
-      (mirror false)
+      (mirror true)
       (drillshape 2)
       (scaleselection 1)
@@
   (net_class Default "This is the default net class."
     (clearance 0.2)
-    (trace_width 1)
+    (trace_width 2)
     (via_dia 1.2)
     (via_drill 0.8)
@@
   (gr_line (start 84 134) (end 50 134) (layer Margin) (width 0.2))
   (gr_line (start 84 168) (end 84 134) (layer Margin) (width 0.2))
-  (gr_text "Robotronik_CDFR_2018\nCentral" (at 150 76) (layer F.Cu)
+  (gr_text "Robotronik_CDFR_2018\nCentral" (at 147.32 73.66) (layer F.Cu)
     (effects (font (size 1.5 1.5) (thickness 0.3)))
   )
@@
   (segment (start 157.119999 143.314999) (end 157.119999 144.685001) (width 0.5) (layer F.Cu) (net 1))
   (segment (start 157.119999 144.685001) (end 157.384998 144.95) (width 0.5) (layer F.Cu) (net 1))
+  (segment (start 215.5 101) (end 211.5 101) (width 2) (layer B.Cu) (net 2))
+  (segment (start 211.5 101) (end 199.5 113) (width 2) (layer B.Cu) (net 2))
+  (segment (start 221 106.5) (end 215.5 101) (width 2) (layer F.Cu) (net 2))
+  (via (at 215.5 101) (size 1.2) (drill 0.8) (layers F.Cu B.Cu) (net 2))
+  (segment (start 232 109.5) (end 224 109.5) (width 2) (layer B.Cu) (net 2))
+  (via (at 221 106.5) (size 1.2) (drill 0.8) (layers F.Cu B.Cu) (net 2))
+  (segment (start 224 109.5) (end 221 106.5) (width 2) (layer B.Cu) (net 2))
   (segment (start 187.75 102.9) (end 188.714001 101.935999) (width 1) (layer B.Cu) (net 2))
   (segment (start 199.5 111.86863) (end 199.5 113) (width 1) (layer B.Cu) (net 2))
@@
   (segment (start 68.442 103.636) (end 68.442 109.942) (width 2) (layer B.Cu) (net 2))
   (segment (start 68.442 109.942) (end 74 115.5) (width 2) (layer B.Cu) (net 2))
+  (segment (start 235 121.84) (end 234.7 121.84) (width 0.5) (layer B.Cu) (net 3))
+  (segment (start 234.7 121.84) (end 229.749999 126.790001) (width 0.5) (layer B.Cu) (net 3))
+  (segment (start 229.749999 126.790001) (end 229.749999 128.304001) (width 0.5) (layer B.Cu) (net 3))
+  (segment (start 229.749999 128.304001) (end 226.554 131.5) (width 0.5) (layer B.Cu) (net 3))
+  (segment (start 204.6 132.543516) (end 204.6 150) (width 0.5) (layer B.Cu) (net 3))
+  (segment (start 226.554 131.5) (end 205.643516 131.5) (width 0.5) (layer B.Cu) (net 3))
+  (segment (start 205.643516 131.5) (end 204.6 132.543516) (width 0.5) (layer B.Cu) (net 3))
+  (segment (start 204.6 150) (end 210.6 156) (width 0.5) (layer B.Cu) (net 3))
   (segment (start 229.4 121.8) (end 234.96 121.8) (width 1) (layer B.Cu) (net 3))
   (segment (start 234.96 121.8) (end 235 121.84) (width 1) (layer B.Cu) (net 3))
@@
   (segment (start 212 104.4) (end 229.4 121.8) (width 1) (layer F.Cu) (net 3))
   (via (at 229.4 121.8) (size 1.2) (drill 0.8) (layers F.Cu B.Cu) (net 3))
-  (segment (start 234.7 121.84) (end 235 121.84) (width 0.5) (layer B.Cu) (net 3))
-  (segment (start 229.749999 126.790001) (end 234.7 121.84) (width 0.5) (layer B.Cu) (net 3))
-  (segment (start 229.749999 128.304001) (end 229.749999 126.790001) (width 0.5) (layer B.Cu) (net 3))
-  (segment (start 226.603999 131.450001) (end 229.749999 128.304001) (width 0.5) (layer B.Cu) (net 3))
-  (segment (start 211.560034 131.450001) (end 226.603999 131.450001) (width 0.5) (layer B.Cu) (net 3))
-  (segment (start 210.6 156) (end 204.6 150) (width 0.5) (layer B.Cu) (net 3))
-  (segment (start 204.6 138.410035) (end 211.560034 131.450001) (width 0.5) (layer B.Cu) (net 3))
-  (segment (start 204.6 150) (end 204.6 138.410035) (width 0.5) (layer B.Cu) (net 3))
   (segment (start 153 145) (end 153 145.848528) (width 1) (layer F.Cu) (net 3))
   (segment (start 153 145.848528) (end 164.651473 157.500001) (width 1) (layer F.Cu) (net 3))
@@
   (segment (start 185 142) (end 185 140.205) (width 1) (layer F.Cu) (net 18))
   (segment (start 185 140.205) (end 182.7 137.905) (width 1) (layer F.Cu) (net 18))
+  (segment (start 219 126.46) (end 219.4 126.46) (width 0.5) (layer B.Cu) (net 19))
+  (segment (start 219.4 126.46) (end 221.86 124) (width 0.5) (layer B.Cu) (net 19))
+  (segment (start 221.86 124) (end 225 124) (width 0.5) (layer B.Cu) (net 19))
+  (segment (start 205 125) (end 206.77 125) (width 0.5) (layer B.Cu) (net 20))
+  (segment (start 206.77 125) (end 209.519999 127.749999) (width 0.5) (layer B.Cu) (net 20))
+  (segment (start 209.519999 127.749999) (end 222.910001 127.749999) (width 0.5) (layer B.Cu) (net 20))
+  (segment (start 222.910001 127.749999) (end 223.2 127.46) (width 0.5) (layer B.Cu) (net 20))
+  (segment (start 223.2 127.46) (end 225 127.46) (width 0.5) (layer B.Cu) (net 20))
   (segment (start 222 77) (end 222 82.84) (width 1) (layer B.Cu) (net 21))
   (segment (start 222 82.84) (end 222.16 83) (width 1) (layer B.Cu) (net 21))
@@
   (segment (start 215.084167 79.00001) (end 216.92 77.164177) (width 1) (layer B.Cu) (net 22))
   (segment (start 216.92 77.164177) (end 216.92 77) (width 1) (layer B.Cu) (net 22))
+  (segment (start 212.5 132.5) (end 232.7 132.5) (width 0.5) (layer B.Cu) (net 23))
+  (segment (start 232.7 132.5) (end 233.2 132) (width 0.5) (layer B.Cu) (net 23))
   (segment (start 233.2 132) (end 235 132) (width 0.5) (layer B.Cu) (net 23))
-  (segment (start 205.4 138.6) (end 211.849988 132.150012) (width 0.5) (layer B.Cu) (net 23))
-  (segment (start 211.849988 132.150012) (end 233.049988 132.150012) (width 0.5) (layer B.Cu) (net 23))
-  (segment (start 233.049988 132.150012) (end 233.2 132) (width 0.5) (layer B.Cu) (net 23))
-  (segment (start 205.4 148) (end 205.4 138.6) (width 0.5) (layer B.Cu) (net 23))
-  (segment (start 211.2 153.8) (end 205.4 148) (width 0.5) (layer B.Cu) (net 23))
-  (segment (start 220.96 153.8) (end 211.2 153.8) (width 0.5) (layer B.Cu) (net 23))
+  (segment (start 211.65 133.35) (end 212.5 132.5) (width 0.5) (layer B.Cu) (net 23))
+  (segment (start 210.82 133.35) (end 211.65 133.35) (width 0.5) (layer B.Cu) (net 23))
+  (segment (start 205.57 138.6) (end 210.82 133.35) (width 0.5) (layer B.Cu) (net 23))
+  (segment (start 205.4 138.6) (end 205.57 138.6) (width 0.5) (layer B.Cu) (net 23))
   (segment (start 223.16 156) (end 220.96 153.8) (width 0.5) (layer B.Cu) (net 23))
+  (segment (start 220.96 153.8) (end 211.2 153.8) (width 0.5) (layer B.Cu) (net 23))
+  (segment (start 211.2 153.8) (end 205.4 148) (width 0.5) (layer B.Cu) (net 23))
+  (segment (start 205.4 148) (end 205.4 138.6) (width 0.5) (layer B.Cu) (net 23))
   (segment (start 205.2 137.4) (end 205.2 151.24) (width 0.5) (layer F.Cu) (net 24))
   (segment (start 205.2 151.24) (end 200.44 156) (width 0.5) (layer F.Cu) (net 24))
@@
     (connect_pads (clearance 0.508))
     (min_thickness 0.254)
-    (fill (arc_segments 16) (thermal_gap 0.508) (thermal_bridge_width 0.508))
+    (fill yes (arc_segments 16) (thermal_gap 0.508) (thermal_bridge_width 0.508))
     (polygon
       (pts
@@
     (connect_pads (clearance 0.508))
     (min_thickness 0.254)
-    (fill (arc_segments 16) (thermal_gap 0.508) (thermal_bridge_width 0.508))
+    (fill yes (arc_segments 16) (thermal_gap 0.508) (thermal_bridge_width 0.508))
     (polygon
       (pts

Commit message: ready to route
Parts:
- added Q2: Q_NMOS_DGS, TO_SOT_Packages_SMD:SOT-323_SC-70_Handsoldering, F.Cu at (102.5, 182.5)
- added Q3: Q_NMOS_DGS, TO_SOT_Packages_SMD:SOT-323_SC-70_Handsoldering, F.Cu at (107.0, 188.5)
- added R15: 3.3kR, Resistors_THT:R_Axial_DIN0207_L6.3mm_D2.5mm_P10.16mm_Horizontal, F.Cu at (166.0, 185.0)
- added R16: 470R, Resistors_THT:R_Axial_DIN0207_L6.3mm_D2.5mm_P10.16mm_Horizontal, F.Cu at (115.5, 181.5)
- added R17: 330R, Resistors_THT:R_Axial_DIN0207_L6.3mm_D2.5mm_P10.16mm_Horizontal, F.Cu at (104.0, 177.5)
- added R18: 270R, Resistors_THT:R_Axial_DIN0207_L6.3mm_D2.5mm_P10.16mm_Horizontal, F.Cu at (94.5, 170.0)
- added R19: 20kR, Resistors_THT:R_Axial_DIN0207_L6.3mm_D2.5mm_P10.16mm_Horizontal, F.Cu at (116.0, 192.5)
- added R21: 20kR, Resistors_THT:R_Axial_DIN0207_L6.3mm_D2.5mm_P10.16mm_Horizontal, F.Cu at (145.5, 206.5)
- added U15: trou-d3mm, Mounting_Holes:MountingHole_3.2mm_M3_Pad, F.Cu at (127.5, 206.5)
- C3: value 47uCP -> 1uC
- C4: value 1uC -> 390nC
- C5: value C -> 10uC; footprint Capacitors_THT:C_Rect_L7.0mm_W2.5mm_P5.00mm -> Capacitors_THT:CP_Radial_D8.0mm_P3.50mm
- C6: value CP -> C; footprint Capacitors_THT:CP_Radial_D8.0mm_P3.50mm -> Capacitors_THT:C_Rect_L7.0mm_W2.5mm_P5.00mm
- R5: value 11kR -> 500R
- R6: value 56kR -> 500R
- U2: value APE8865U5-28-HF-3 -> LM317_SOT223; footprint TO_SOT_Packages_SMD:SOT-23-5_HandSoldering -> TO_SOT_Packages_SMD:SOT-223-3Lead_TabPin2
- U3: value I2C_repeater -> LM317_SOT223; footprint Housings_SOIC:SOIC-8_3.9x4.9mm_Pitch1.27mm -> TO_SOT_Packages_SMD:SOT-223-3Lead_TabPin2
- U4: value TDA8541 -> TDA6205
- moved U3 116.8 mm to (180.0, 218.5), turned to 0 degrees
- moved U2 87.1 mm to (204.5, 217.0), turned to 0 degrees
- moved C6 83.1 mm to (200.5, 205.0)
- moved U4 74.7 mm to (112.5, 168.0)
- moved C5 60.8 mm to (168.5, 199.5), turned to 0 degrees
- moved R5 57.3 mm to (133.0, 184.0)
- moved R6 57.1 mm to (150.5, 187.5), turned to 0 degrees
- moved C4 56.4 mm to (187.0, 205.0)
- moved C3 43.1 mm to (186.5, 173.0)
Connections:
- C5 pad 1: +5V -> /Power/Rasp_power
- R5 pad 1: Net-(R5-Pad1) -> Net-(D4-Pad2)
- R5 pad 2: Net-(C4-Pad1) -> Net-(R5-Pad2)
- R6 pad 1: Net-(P2-Pad2) -> Net-(D3-Pad2)
- R6 pad 2: Net-(R5-Pad1) -> Net-(R6-Pad2)
- U1 pad 1: Net-(U1-Pad1) -> (no net)
- U1 pad 11: Net-(U1-Pad11) -> (no net)
- U1 pad 12: Net-(U1-Pad12) -> (no net)
- U1 pad 13: Net-(U1-Pad13) -> (no net)
- U1 pad 14: Net-(U1-Pad14) -> (no net)
- U1 pad 15: Net-(U1-Pad15) -> (no net)
- U1 pad 16: Net-(U1-Pad16) -> (no net)
- U1 pad 18: Net-(U1-Pad18) -> (no net)
- U1 pad 19: Net-(U1-Pad19) -> (no net)
- U1 pad 2: Net-(U1-Pad2) -> (no net)
- U1 pad 20: Net-(U1-Pad20) -> (no net)
- U1 pad 21: Net-(U1-Pad21) -> (no net)
- U1 pad 22: Net-(U1-Pad22) -> (no net)
- U1 pad 23: Net-(U1-Pad23) -> (no net)
- U1 pad 24: Net-(U1-Pad24) -> (no net)
- U1 pad 25: Net-(U1-Pad25) -> (no net)
- U1 pad 26: Net-(U1-Pad26) -> (no net)
- U1 pad 27: Net-(U1-Pad27) -> (no net)
- U1 pad 28: Net-(U1-Pad28) -> (no net)
- U1 pad 3: Net-(U1-Pad3) -> (no net)
- U1 pad 31: Net-(U1-Pad31) -> (no net)
- U1 pad 33: Net-(U1-Pad33) -> (no net)
- U1 pad 34: Net-(U1-Pad34) -> (no net)
- U1 pad 35: Net-(U1-Pad35) -> (no net)
- U1 pad 38: Net-(U1-Pad38) -> (no net)
- U1 pad 39: Net-(U1-Pad39) -> (no net)
- U1 pad 4: Net-(U1-Pad4) -> (no net)
- U1 pad 40: Net-(U1-Pad40) -> (no net)
- U1 pad 41: Net-(U1-Pad41) -> (no net)
- U1 pad 42: Net-(U1-Pad42) -> (no net)
- U1 pad 43: Net-(U1-Pad43) -> (no net)
- U1 pad 45: Net-(U1-Pad45) -> (no net)
- U1 pad 46: Net-(U1-Pad46) -> (no net)
- U1 pad 47: Net-(U1-Pad47) -> (no net)
- U1 pad 48: Net-(U1-Pad48) -> (no net)
- U1 pad 49: Net-(U1-Pad49) -> (no net)
- U1 pad 5: Net-(U1-Pad5) -> (no net)
- U1 pad 51: Net-(U1-Pad51) -> (no net)
- U1 pad 52: Net-(U1-Pad52) -> (no net)
- U1 pad 55: Net-(U1-Pad55) -> (no net)
- U1 pad 56: Net-(U1-Pad56) -> (no net)
- U1 pad 57: Net-(U1-Pad57) -> (no net)
- U1 pad 6: Net-(U1-Pad6) -> (no net)
- U1 pad 60: Net-(U1-Pad60) -> (no net)
- U1 pad 64: Net-(U1-Pad64) -> (no net)
- U1 pad 65: Net-(U1-Pad65) -> (no net)
- U1 pad 67: I2C_TOF_EN -> (no net)
- U1 pad 7: Net-(U1-Pad7) -> (no net)
- U1 pad 70: Net-(U1-Pad70) -> (no net)
- U1 pad 72: Net-(D3-Pad2) -> Net-(R6-Pad2)
- U1 pad 73: Net-(D4-Pad2) -> Net-(R5-Pad2)
- U1 pad 74: Net-(U1-Pad74) -> (no net)
- U1 pad 76: Net-(U1-Pad76) -> (no net)
- U1 pad 77: Net-(U1-Pad77) -> (no net)
- U1 pad 78: Net-(U1-Pad78) -> (no net)
- U1 pad 79: Net-(U1-Pad79) -> (no net)
- U1 pad 8: Net-(U1-Pad8) -> (no net)
- U1 pad 80: Net-(U1-Pad80) -> (no net)
- U1 pad 81: Net-(U1-Pad81) -> (no net)
- U1 pad 82: Net-(U1-Pad82) -> (no net)
- U1 pad 83: Net-(U1-Pad83) -> (no net)
- U1 pad 84: Net-(U1-Pad84) -> (no net)
- U2 pad 1: +5V -> Net-(R15-Pad1)
- U2 pad 2: GND -> +9V
- U2 pad 3: +5V -> BATT
- U3 pad 1: +3V3 -> Net-(R17-Pad1)
- U3 pad 2: I2C_TOF_SCL -> +2.8V
- U3 pad 3: I2C_TOF_SDA -> +5V
- U4 pad 4: Net-(R5-Pad1) -> Net-(R19-Pad1)
- U9 pad 1: Net-(U9-Pad1) -> (no net)
- U9 pad 5: Net-(U9-Pad5) -> (no net)
- U9 pad 6: BATT -> +9V
- U9 pad 8: Net-(U9-Pad8) -> (no net)
Routing:
- net (no net): track 0.00 -> 79.4 mm, vias 0 -> 2
- net Net-(R5-Pad2): track 0.00 -> 38.9 mm
- net Net-(D4-Pad2): track 102.4 -> 63.5 mm
- net I2C_TOF_EN: track 31.9 -> 0.00 mm, vias 1 -> 0
- net Net-(C3-Pad1): track 27.4 -> 0.00 mm, vias 1 -> 0
- net +9V: track 0.00 -> 8.86 mm
- net BATT: track 79.0 -> 70.1 mm
- net Net-(R5-Pad1): track 8.18 -> 0.00 mm
- net Net-(C4-Pad1): track 6.82 -> 0.00 mm
- net Net-(P2-Pad2): track 19.2 -> 14.2 mm
- net Net-(D3-Pad2): track 85.2 -> 84.1 mm
- net Net-(R6-Pad2): track 0.00 -> 1.13 mm

Commit message: RagePCB
Parts:
- moved P8 25.0 mm to (94.0, 130.0)
- moved U14 17.0 mm to (71.0, 129.0)
- moved P1 4.12 mm to (90.0, 73.0)
- moved U11 1.41 mm to (71.0, 73.0)
- moved U13 1.41 mm to (234.0, 73.0)
Routing:
- net GND: track 770.6 -> 0.00 mm, vias 8 -> 0
- net +2.8V: track 424.1 -> 0.00 mm, vias 2 -> 0
- net Net-(P1-Pad2): track 315.9 -> 0.00 mm, vias 6 -> 0
- net Net-(P1-Pad4): track 298.9 -> 0.00 mm, vias 4 -> 0
- net +5V: track 158.6 -> 0.00 mm, vias 1 -> 0
- net I2C_Free_SDA: track 97.1 -> 0.00 mm
- net Net-(D3-Pad2): track 84.1 -> 0.00 mm
- net (no net): track 79.4 -> 0.00 mm, vias 2 -> 0
- net BATT: track 70.1 -> 0.00 mm, vias 1 -> 0
- net +3V3: track 66.9 -> 0.00 mm, vias 2 -> 0
- net Net-(D4-Pad2): track 63.5 -> 0.00 mm, vias 2 -> 0
- net Net-(P7-Pad1): track 62.8 -> 0.00 mm
- net /Pince_RX: track 58.7 -> 0.00 mm, vias 2 -> 0
- net /Pince_TX: track 58.7 -> 0.00 mm, vias 2 -> 0
- net Net-(D2-Pad1): track 55.6 -> 0.00 mm, vias 1 -> 0
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- removed copper zone on B.Cu, net GND
- removed copper zone on F.Cu, net GND
Other:
- board size 175 x 90 mm -> 173 x 90 mm

Commit message: smd resistor
Parts:
- R1, R10, R11, R12, R13, R14, R15, R16, R17, R18, R19, R2, R21, R3, R4, R5, R6, R7, R8, R9: footprint Resistors_THT:R_Axial_DIN0207_L6.3mm_D2.5mm_P10.16mm_Horizontal -> Resistors_SMD:R_1206_HandSoldering
- moved R8 20.7 mm to (202.0, 173.5)
