File: Electronique/Central/Power.sch (KiCad schematic (older format))
At the start: 3 parts, among them U2 APE8865U5-28-HF-3

Commit message: led!
Parts:
- added D1, D2: D, symbol D
- added F1, F2: FUSE, Fuse_Holders_and_Fuses:Fuseholder5x20_horiz_SemiClosed_Casing10x25mm, symbol FUSE
- added U5, U6: B_Plug_5mm, dsn2596:B plug 5mm, symbol B_Plug_5mm
- added U7, U8: DSN2596, dsn2596:DSN2596, symbol DSN2596
Connections:
- net +5V: now also U7.4 (OUT+)
- net GND: now also D1.2 (A), D2.2 (A), U5.2, U6.2, U7.2 (IN-), U7.3 (OUT-), U8.2 (IN-), U8.3 (OUT-)
- new net: D2.1 (K), F2.2, U8.1 (IN+)
- new net: F1.1, U5.1
- new net: F2.1, U6.1
- new net +5V_Rasp: U8.4 (OUT+)
- new net BATT: D1.1 (K), F1.2, U7.1 (IN+)
Other:
- moved on the sheet: C1, C2, U2

Commit message: go routage
Parts:
- added C7: CP, Capacitors_THT:CP_Radial_D8.0mm_P3.50mm, symbol CP
- added P11: CONN_01X02, Connectors_Molex:Molex_KK-6410-02_02x2.54mm_Straight, symbol CONN_01X02
- C1, C2: footprint (none) -> Capacitors_THT:C_Rect_L7.0mm_W2.5mm_P5.00mm
- D1, D2: footprint (none) -> Diodes_SMD:D_SMA_Handsoldering
Connections:
- net +5V: now also C7.1
- net GND: now also C7.2, P11.2 (P2)
- net +5V_Rasp renamed Rasp_power
- net Rasp_power: now also P11.1 (P1)
Other:
- note added: "Non polarisé de plus grande valeur possible"
Changed lines of the file:
@@
 LIBS:2
 LIBS:dsn2596
+LIBS:raspberry_pi_3
 LIBS:central-cache
 EELAYER 25 0
@@
 $EndComp
 $Comp
-L +5V #PWR15
+L +5V #PWR025
 U 1 1 5A6CA927
 P 7100 1650
-F 0 "#PWR15" H 7100 1500 50  0001 C CNN
+F 0 "#PWR025" H 7100 1500 50  0001 C CNN
 F 1 "+5V" H 7100 1790 50  0000 C CNN
 F 2 "" H 7100 1650 50  0000 C CNN
@@
 Connection ~ 7800 1950
 $Comp
-L GND #PWR17
+L GND #PWR026
 U 1 1 5A6CA964
 P 8450 2450
-F 0 "#PWR17" H 8450 2200 50  0001 C CNN
+F 0 "#PWR026" H 8450 2200 50  0001 C CNN
 F 1 "GND" H 8450 2300 50  0000 C CNN
 F 2 "" H 8450 2450 50  0000 C CNN
@@
 F 0 "C1" H 7425 2300 50  0000 L CNN
 F 1 "1uC" H 7425 2100 50  0000 L CNN
-F 2 "" H 7438 2050 50  0001 C CNN
+F 2 "Capacitors_THT:C_Rect_L7.0mm_W2.5mm_P5.00mm" H 7438 2050 50  0001 C CNN
 F 3 "" H 7400 2200 50  0000 C CNN
 	1    7400 2200
@@
 F 0 "C2" H 9125 2350 50  0000 L CNN
 F 1 "1uC" H 9125 2150 50  0000 L CNN
-F 2 "" H 9138 2100 50  0001 C CNN
+F 2 "Capacitors_THT:C_Rect_L7.0mm_W2.5mm_P5.00mm" H 9138 2100 50  0001 C CNN
 F 3 "" H 9100 2250 50  0000 C CNN
 	1    9100 2250
@@
 $EndComp
 $Comp
-L GND #PWR16
+L GND #PWR027
 U 1 1 5A6CB546
 P 7400 2550
-F 0 "#PWR16" H 7400 2300 50  0001 C CNN
+F 0 "#PWR027" H 7400 2300 50  0001 C CNN
 F 1 "GND" H 7400 2400 50  0000 C CNN
 F 2 "" H 7400 2550 50  0000 C CNN
@@
 $EndComp
 $Comp
-L GND #PWR18
+L GND #PWR028
 U 1 1 5A6CB560
 P 9100 2550
-F 0 "#PWR18" H 9100 2300 50  0001 C CNN
+F 0 "#PWR028" H 9100 2300 50  0001 C CNN
 F 1 "GND" H 9100 2400 50  0000 C CNN
 F 2 "" H 9100 2550 50  0000 C CNN
@@
 F 0 "D1" H 2500 1950 50  0000 C CNN
 F 1 "D" H 2500 1750 50  0000 C CNN
-F 2 "" H 2500 1850 50  0001 C CNN
+F 2 "Diodes_SMD:D_SMA_Handsoldering" H 2500 1850 50  0001 C CNN
 F 3 "" H 2500 1850 50  0000 C CNN
 	1    2500 1850
@@
 F 0 "D2" H 2500 2750 50  0000 C CNN
 F 1 "D" H 2500 2550 50  0000 C CNN
-F 2 "" H 2500 2650 50  0001 C CNN
+F 2 "Diodes_SMD:D_SMA_Handsoldering" H 2500 2650 50  0001 C CNN
 F 3 "" H 2500 2650 50  0000 C CNN
 	1    2500 2650
@@
 	1250 2300 1850 2300
 $Comp
-L GND #PWR6
+L GND #PWR029
 U 1 1 5A74E256
 P 1550 1750
-F 0 "#PWR6" H 1550 1500 50  0001 C CNN
+F 0 "#PWR029" H 1550 1500 50  0001 C CNN
 F 1 "GND" H 1550 1600 50  0000 C CNN
 F 2 "" H 1550 1750 50  0000 C CNN
@@
 $EndComp
 $Comp
-L GND #PWR7
+L GND #PWR030
 U 1 1 5A74E280
 P 1550 2500
-F 0 "#PWR7" H 1550 2250 50  0001 C CNN
+F 0 "#PWR030" H 1550 2250 50  0001 C CNN
 F 1 "GND" H 1550 2350 50  0000 C CNN
 F 2 "" H 1550 2500 50  0000 C CNN
@@
 	2500 2300 2500 2500
 $Comp
-L GND #PWR8
+L GND #PWR031
 U 1 1 5A74E3F6
 P 2500 2050
-F 0 "#PWR8" H 2500 1800 50  0001 C CNN
+F 0 "#PWR031" H 2500 1800 50  0001 C CNN
 F 1 "GND" H 2500 1900 50  0000 C CNN
 F 2 "" H 2500 2050 50  0000 C CNN
@@
 $EndComp
 $Comp
-L GND #PWR9
+L GND #PWR032
 U 1 1 5A74E420
 P 2500 2850
-F 0 "#PWR9" H 2500 2600 50  0001 C CNN
+F 0 "#PWR032" H 2500 2600 50  0001 C CNN
 F 1 "GND" H 2500 2700 50  0000 C CNN
 F 2 "" H 2500 2850 50  0000 C CNN
@@
 Connection ~ 2500 2300
 $Comp
-L GND #PWR10
+L GND #PWR033
 U 1 1 5A74E67A
 P 3400 1850
-F 0 "#PWR10" H 3400 1600 50  0001 C CNN
+F 0 "#PWR033" H 3400 1600 50  0001 C CNN
 F 1 "GND" H 3400 1700 50  0000 C CNN
 F 2 "" H 3400 1850 50  0000 C CNN
@@
 $EndComp
 $Comp
-L GND #PWR11
+L GND #PWR034
 U 1 1 5A74E804
 P 3400 2600
-F 0 "#PWR11" H 3400 2350 50  0001 C CNN
+F 0 "#PWR034" H 3400 2350 50  0001 C CNN
 F 1 "GND" H 3400 2450 50  0000 C CNN
 F 2 "" H 3400 2600 50  0000 C CNN
@@
 	3400 2500 3500 2500
 $Comp
-L GND #PWR12
+L GND #PWR035
 U 1 1 5A74EC12
 P 4700 1850
-F 0 "#PWR12" H 4700 1600 50  0001 C CNN
+F 0 "#PWR035" H 4700 1600 50  0001 C CNN
 F 1 "GND" H 4700 1700 50  0000 C CNN
 F 2 "" H 4700 1850 50  0000 C CNN
@@
 $EndComp
 $Comp
-L GND #PWR13
+L GND #PWR036
 U 1 1 5A74ED5A
 P 4700 2600
-F 0 "#PWR13" H 4700 2350 50  0001 C CNN
+F 0 "#PWR036" H 4700 2350 50  0001 C CNN
 F 1 "GND" H 4700 2450 50  0000 C CNN
 F 2 "" H 4700 2600 50  0000 C CNN
@@
 	4700 2500 4700 2600
 $Comp
-L +5V #PWR14
+L +5V #PWR037
 U 1 1 5A74F2CA
 P 5000 1500
-F 0 "#PWR14" H 5000 1350 50  0001 C CNN
+F 0 "#PWR037" H 5000 1350 50  0001 C CNN
 F 1 "+5V" H 5000 1640 50  0000 C CNN
 F 2 "" H 5000 1500 50  0000 C CNN
@@
 $EndComp
 Wire Wire Line
-	4600 1550 5000 1550
+	4600 1550 5700 1550
 Wire Wire Line
 	5000 1550 5000 1500
 $Comp
-L PWR_FLAG #FLG1
+L PWR_FLAG #FLG038
 U 1 1 5A74F572
 P 1500 1400
-F 0 "#FLG1" H 1500 1495 50  0001 C CNN
+F 0 "#FLG038" H 1500 1495 50  0001 C CNN
 F 1 "PWR_FLAG" H 1500 1580 50  0000 C CNN
 F 2 "" H 1500 1400 50  0000 C CNN
@@
 $EndComp
 $Comp
-L PWR_FLAG #FLG2
+L PWR_FLAG #FLG039
 U 1 1 5A74F59C
 P 1600 2200
-F 0 "#FLG2" H 1600 2295 50  0001 C CNN
+F 0 "#FLG039" H 1600 2295 50  0001 C CNN
 F 1 "PWR_FLAG" H 1600 2380 50  0000 C CNN
 F 2 "" H 1600 2200 50  0000 C CNN
@@
 $EndComp
 $Comp
-L PWR_FLAG #FLG3
+L PWR_FLAG #FLG040
 U 1 1 5A74F5C6
 P 1600 2450
-F 0 "#FLG3" H 1600 2545 50  0001 C CNN
+F 0 "#FLG040" H 1600 2545 50  0001 C CNN
 F 1 "PWR_FLAG" H 1600 2630 50  0000 C CNN
 F 2 "" H 1600 2450 50  0000 C CNN
@@
 	1600 2450 1550 2450
 Connection ~ 1550 2450
-Text GLabel 5200 2150 1    60   Input ~ 0
-+5V_Rasp
 Wire Wire Line
 	4600 2300 5200 2300
-Wire Wire Line
-	5200 2300 5200 2150
 Wire Wire Line
 	1250 1550 1850 1550
@@
 	2700 1350 2700 1550
 Connection ~ 2700 1550
+$Comp
+L CP C7
+U 1 1 5A77C1B0
+P 5700 1750
+F 0 "C7" H 5725 1850 50  0000 L CNN
+F 1 "CP" H 5725 1650 50  0000 L CNN
+F 2 "Capacitors_THT:CP_Radial_D8.0mm_P3.50mm" H 5738 1600 50  0001 C CNN
+F 3 "" H 5700 1750 50  0000 C CNN
+	1    5700 1750
+	1    0    0    -1
+$EndComp
+$Comp
+L GND #PWR041
+U 1 1 5A77C1FF
+P 5700 2000
+F 0 "#PWR041" H 5700 1750 50  0001 C CNN
+F 1 "GND" H 5700 1850 50  0000 C CNN
+F 2 "" H 5700 2000 50  0000 C CNN
+F 3 "" H 5700 2000 50  0000 C CNN
+	1    5700 2000
+	1    0    0    -1
+$EndComp
+Wire Wire Line
+	5700 1550 5700 1600
+Connection ~ 5000 1550
+Wire Wire Line
+	5700 1900 5700 2000
+Text Notes 7500 1300 0    60   ~ 0
+Non polarisé de plus grande valeur possible
+$Comp
+L CONN_01X02 P11
+U 1 1 5A782930
+P 5550 2550
+F 0 "P11" H 5550 2700 50  0000 C CNN
+F 1 "CONN_01X02" V 5650 2550 50  0000 C CNN
+F 2 "Connectors_Molex:Molex_KK-6410-02_02x2.54mm_Straight" H 5550 2550 50  0001 C CNN
+F 3 "" H 5550 2550 50  0000 C CNN
+	1    5550 2550
+	1    0    0    -1
+$EndComp
+Wire Wire Line
+	5200 2500 5350 2500
+$Comp
+L GND #PWR042
+U 1 1 5A782A30
+P 5250 2700
+F 0 "#PWR042" H 5250 2450 50  0001 C CNN
+F 1 "GND" H 5250 2550 50  0000 C CNN
+F 2 "" H 5250 2700 50  0000 C CNN
+F 3 "" H 5250 2700 50  0000 C CNN
+	1    5250 2700
+	1    0    0    -1
+$EndComp
+Wire Wire Line
+	5250 2700 5250 2600
+Wire Wire Line
+	5250 2600 5350 2600
+Wire Wire Line
+	5200 2300 5200 2500
+Text Label 5050 2300 0    60   ~ 0
+Rasp_power
 $EndSCHEMATC

Commit message: Routage PCB central
Parts:
- U2: symbol APE8865U5-28-HF-3 -> APE8865U5-28-HF-3-RESCUE-central
Changed lines of the file:
@@
 EESchema Schematic File Version 2
+LIBS:central-rescue
 LIBS:power
 LIBS:device
@@
 $EndDescr
 $Comp
-L APE8865U5-28-HF-3 U2
+L APE8865U5-28-HF-3-RESCUE-central U2
 U 1 1 5A6CA894
 P 8450 2000
+AR Path="/5A6CA894" Ref="U2"  Part="1"
+AR Path="/5A6CA888/5A6CA894" Ref="U2"  Part="1"
 F 0 "U2" H 8150 2250 50  0000 C CNN
 F 1 "APE8865U5-28-HF-3" H 8450 2200 50  0000 C CNN
@@
 $EndComp
 $Comp
-L +5V #PWR025
+L +5V #PWR023
 U 1 1 5A6CA927
 P 7100 1650
-F 0 "#PWR025" H 7100 1500 50  0001 C CNN
+F 0 "#PWR023" H 7100 1500 50  0001 C CNN
 F 1 "+5V" H 7100 1790 50  0000 C CNN
 F 2 "" H 7100 1650 50  0000 C CNN
@@
 Connection ~ 7800 1950
 $Comp
-L GND #PWR026
+L GND #PWR024
 U 1 1 5A6CA964
 P 8450 2450
-F 0 "#PWR026" H 8450 2200 50  0001 C CNN
+F 0 "#PWR024" H 8450 2200 50  0001 C CNN
 F 1 "GND" H 8450 2300 50  0000 C CNN
 F 2 "" H 8450 2450 50  0000 C CNN
@@
 $EndComp
 $Comp
-L GND #PWR027
+L GND #PWR025
 U 1 1 5A6CB546
 P 7400 2550
-F 0 "#PWR027" H 7400 2300 50  0001 C CNN
+F 0 "#PWR025" H 7400 2300 50  0001 C CNN
 F 1 "GND" H 7400 2400 50  0000 C CNN
 F 2 "" H 7400 2550 50  0000 C CNN
@@
 $EndComp
 $Comp
-L GND #PWR028
+L GND #PWR026
 U 1 1 5A6CB560
 P 9100 2550
-F 0 "#PWR028" H 9100 2300 50  0001 C CNN
+F 0 "#PWR026" H 9100 2300 50  0001 C CNN
 F 1 "GND" H 9100 2400 50  0000 C CNN
 F 2 "" H 9100 2550 50  0000 C CNN
@@
 	1250 2300 1850 2300
 $Comp
-L GND #PWR029
+L GND #PWR027
 U 1 1 5A74E256
 P 1550 1750
-F 0 "#PWR029" H 1550 1500 50  0001 C CNN
+F 0 "#PWR027" H 1550 1500 50  0001 C CNN
 F 1 "GND" H 1550 1600 50  0000 C CNN
 F 2 "" H 1550 1750 50  0000 C CNN
@@
 $EndComp
 $Comp
-L GND #PWR030
+L GND #PWR028
 U 1 1 5A74E280
 P 1550 2500
-F 0 "#PWR030" H 1550 2250 50  0001 C CNN
+F 0 "#PWR028" H 1550 2250 50  0001 C CNN
 F 1 "GND" H 1550 2350 50  0000 C CNN
 F 2 "" H 1550 2500 50  0000 C CNN
@@
 	2500 2300 2500 2500
 $Comp
-L GND #PWR031
+L GND #PWR029
 U 1 1 5A74E3F6
 P 2500 2050
-F 0 "#PWR031" H 2500 1800 50  0001 C CNN
+F 0 "#PWR029" H 2500 1800 50  0001 C CNN
 F 1 "GND" H 2500 1900 50  0000 C CNN
 F 2 "" H 2500 2050 50  0000 C CNN
@@
 $EndComp
 $Comp
-L GND #PWR032
+L GND #PWR030
 U 1 1 5A74E420
 P 2500 2850
-F 0 "#PWR032" H 2500 2600 50  0001 C CNN
+F 0 "#PWR030" H 2500 2600 50  0001 C CNN
 F 1 "GND" H 2500 2700 50  0000 C CNN
 F 2 "" H 2500 2850 50  0000 C CNN
@@
 Connection ~ 2500 2300
 $Comp
-L GND #PWR033
+L GND #PWR031
 U 1 1 5A74E67A
 P 3400 1850
-F 0 "#PWR033" H 3400 1600 50  0001 C CNN
+F 0 "#PWR031" H 3400 1600 50  0001 C CNN
 F 1 "GND" H 3400 1700 50  0000 C CNN
 F 2 "" H 3400 1850 50  0000 C CNN
@@
 $EndComp
 $Comp
-L GND #PWR034
+L GND #PWR032
 U 1 1 5A74E804
 P 3400 2600
-F 0 "#PWR034" H 3400 2350 50  0001 C CNN
+F 0 "#PWR032" H 3400 2350 50  0001 C CNN
 F 1 "GND" H 3400 2450 50  0000 C CNN
 F 2 "" H 3400 2600 50  0000 C CNN
@@
 	3400 2500 3500 2500
 $Comp
-L GND #PWR035
+L GND #PWR033
 U 1 1 5A74EC12
 P 4700 1850
-F 0 "#PWR035" H 4700 1600 50  0001 C CNN
+F 0 "#PWR033" H 4700 1600 50  0001 C CNN
 F 1 "GND" H 4700 1700 50  0000 C CNN
 F 2 "" H 4700 1850 50  0000 C CNN
@@
 $EndComp
 $Comp
-L GND #PWR036
+L GND #PWR034
 U 1 1 5A74ED5A
 P 4700 2600
-F 0 "#PWR036" H 4700 2350 50  0001 C CNN
+F 0 "#PWR034" H 4700 2350 50  0001 C CNN
 F 1 "GND" H 4700 2450 50  0000 C CNN
 F 2 "" H 4700 2600 50  0000 C CNN
@@
 	4700 2500 4700 2600
 $Comp
-L +5V #PWR037
+L +5V #PWR035
 U 1 1 5A74F2CA
 P 5000 1500
-F 0 "#PWR037" H 5000 1350 50  0001 C CNN
+F 0 "#PWR035" H 5000 1350 50  0001 C CNN
 F 1 "+5V" H 5000 1640 50  0000 C CNN
 F 2 "" H 5000 1500 50  0000 C CNN
@@
 	5000 1550 5000 1500
 $Comp
-L PWR_FLAG #FLG038
+L PWR_FLAG #FLG036
 U 1 1 5A74F572
 P 1500 1400
-F 0 "#FLG038" H 1500 1495 50  0001 C CNN
+F 0 "#FLG036" H 1500 1495 50  0001 C CNN
 F 1 "PWR_FLAG" H 1500 1580 50  0000 C CNN
 F 2 "" H 1500 1400 50  0000 C CNN
@@
 $EndComp
 $Comp
-L PWR_FLAG #FLG039
+L PWR_FLAG #FLG037
 U 1 1 5A74F59C
 P 1600 2200
-F 0 "#FLG039" H 1600 2295 50  0001 C CNN
+F 0 "#FLG037" H 1600 2295 50  0001 C CNN
 F 1 "PWR_FLAG" H 1600 2380 50  0000 C CNN
 F 2 "" H 1600 2200 50  0000 C CNN
@@
 $EndComp
 $Comp
-L PWR_FLAG #FLG040
+L PWR_FLAG #FLG038
 U 1 1 5A74F5C6
 P 1600 2450
-F 0 "#FLG040" H 1600 2545 50  0001 C CNN
+F 0 "#FLG038" H 1600 2545 50  0001 C CNN
 F 1 "PWR_FLAG" H 1600 2630 50  0000 C CNN
 F 2 "" H 1600 2450 50  0000 C CNN
@@
 $EndComp
 $Comp
-L GND #PWR041
+L GND #PWR039
 U 1 1 5A77C1FF
 P 5700 2000
-F 0 "#PWR041" H 5700 1750 50  0001 C CNN
+F 0 "#PWR039" H 5700 1750 50  0001 C CNN
 F 1 "GND" H 5700 1850 50  0000 C CNN
 F 2 "" H 5700 2000 50  0000 C CNN
@@
 	5200 2500 5350 2500
 $Comp
-L GND #PWR042
+L GND #PWR040
 U 1 1 5A782A30
 P 5250 2700
-F 0 "#PWR042" H 5250 2450 50  0001 C CNN
+F 0 "#PWR040" H 5250 2450 50  0001 C CNN
 F 1 "GND" H 5250 2550 50  0000 C CNN
 F 2 "" H 5250 2700 50  0000 C CNN
