File: Electronique/Central/Power.sch (KiCad schematic (older format))
At the start: 19 parts, among them P11 CONN_01X02, U2 LM317_SOT223, U3 LM317_SOT223, U5 B_Plug_5mm, U6 B_Plug_5mm, U7 DSN2596, U8 DSN2596

Commit message: ready to route
Parts:
- C5: footprint (none) -> Capacitors_THT:CP_Radial_D8.0mm_P3.50mm
- R15, R16, R17, R18: footprint (none) -> Resistors_THT:R_Axial_DIN0207_L6.3mm_D2.5mm_P10.16mm_Horizontal
- U2, U3: footprint (none) -> TO_SOT_Packages_SMD:SOT-223-3Lead_TabPin2
Changed lines of the file:
@@
 F 0 "U3" H 8150 2400 50  0000 C CNN
 F 1 "LM317_SOT223" H 8200 1850 50  0000 L CNN
-F 2 "" H 8150 2100 50  0000 C CNN
+F 2 "TO_SOT_Packages_SMD:SOT-223-3Lead_TabPin2" H 8150 2100 50  0001 C CNN
 F 3 "" H 8150 2100 50  0000 C CNN
 	1    8150 2100
@@
 F 0 "R18" V 8880 2350 50  0000 C CNN
 F 1 "270R" V 8800 2350 50  0000 C CNN
-F 2 "" V 8730 2350 50  0000 C CNN
+F 2 "Resistors_THT:R_Axial_DIN0207_L6.3mm_D2.5mm_P10.16mm_Horizontal" V 8730 2350 50  0001 C CNN
 F 3 "" H 8800 2350 50  0000 C CNN
 	1    8800 2350
@@
 F 0 "R17" V 8230 2850 50  0000 C CNN
 F 1 "330R" V 8150 2850 50  0000 C CNN
-F 2 "" V 8080 2850 50  0000 C CNN
+F 2 "Resistors_THT:R_Axial_DIN0207_L6.3mm_D2.5mm_P10.16mm_Horizontal" V 8080 2850 50  0001 C CNN
 F 3 "" H 8150 2850 50  0000 C CNN
 	1    8150 2850
@@
 F 0 "U2" H 6900 4450 50  0000 C CNN
 F 1 "LM317_SOT223" H 6950 3900 50  0000 L CNN
-F 2 "" H 6900 4150 50  0000 C CNN
+F 2 "TO_SOT_Packages_SMD:SOT-223-3Lead_TabPin2" H 6900 4150 50  0001 C CNN
 F 3 "" H 6900 4150 50  0000 C CNN
 	1    6900 4150
@@
 F 0 "R16" V 7730 4300 50  0000 C CNN
 F 1 "470R" V 7650 4300 50  0000 C CNN
-F 2 "" V 7580 4300 50  0000 C CNN
+F 2 "Resistors_THT:R_Axial_DIN0207_L6.3mm_D2.5mm_P10.16mm_Horizontal" V 7580 4300 50  0001 C CNN
 F 3 "" H 7650 4300 50  0000 C CNN
 	1    7650 4300
@@
 F 0 "R15" V 6980 4800 50  0000 C CNN
 F 1 "3.3kR" V 6900 4800 50  0000 C CNN
-F 2 "" V 6830 4800 50  0000 C CNN
+F 2 "Resistors_THT:R_Axial_DIN0207_L6.3mm_D2.5mm_P10.16mm_Horizontal" V 6830 4800 50  0001 C CNN
 F 3 "" H 6900 4800 50  0000 C CNN
 	1    6900 4800
@@
 F 0 "C5" H 4975 3050 50  0000 L CNN
 F 1 "10uC" H 4975 2850 50  0000 L CNN
-F 2 "" H 4988 2800 50  0000 C CNN
+F 2 "Capacitors_THT:CP_Radial_D8.0mm_P3.50mm" H 4988 2800 50  0001 C CNN
 F 3 "" H 4950 2950 50  0000 C CNN
 	1    4950 2950

Commit message: smd resistor
Parts:
- R15, R16, R17, R18: footprint Resistors_THT:R_Axial_DIN0207_L6.3mm_D2.5mm_P10.16mm_Horizontal -> Resistors_SMD:R_1206_HandSoldering
Changed lines of the file:
@@
 $EndDescr
 $Comp
-L +5V #PWR34
+L +5V #PWR022
 U 1 1 5A6CA927
 P 7100 1650
-F 0 "#PWR34" H 7100 1500 50  0001 C CNN
+F 0 "#PWR022" H 7100 1500 50  0001 C CNN
 F 1 "+5V" H 7100 1790 50  0000 C CNN
 F 2 "" H 7100 1650 50  0000 C CNN
@@
 $EndComp
 $Comp
-L GND #PWR35
+L GND #PWR023
 U 1 1 5A6CB546
 P 7400 2550
-F 0 "#PWR35" H 7400 2300 50  0001 C CNN
+F 0 "#PWR023" H 7400 2300 50  0001 C CNN
 F 1 "GND" H 7400 2400 50  0000 C CNN
 F 2 "" H 7400 2550 50  0000 C CNN
@@
 $EndComp
 $Comp
-L GND #PWR38
+L GND #PWR024
 U 1 1 5A6CB560
 P 9100 2550
-F 0 "#PWR38" H 9100 2300 50  0001 C CNN
+F 0 "#PWR024" H 9100 2300 50  0001 C CNN
 F 1 "GND" H 9100 2400 50  0000 C CNN
 F 2 "" H 9100 2550 50  0000 C CNN
@@
 	1250 2300 1850 2300
 $Comp
-L GND #PWR21
+L GND #PWR025
 U 1 1 5A74E256
 P 1550 1750
-F 0 "#PWR21" H 1550 1500 50  0001 C CNN
+F 0 "#PWR025" H 1550 1500 50  0001 C CNN
 F 1 "GND" H 1550 1600 50  0000 C CNN
 F 2 "" H 1550 1750 50  0000 C CNN
@@
 $EndComp
 $Comp
-L GND #PWR22
+L GND #PWR026
 U 1 1 5A74E280
 P 1550 2500
-F 0 "#PWR22" H 1550 2250 50  0001 C CNN
+F 0 "#PWR026" H 1550 2250 50  0001 C CNN
 F 1 "GND" H 1550 2350 50  0000 C CNN
 F 2 "" H 1550 2500 50  0000 C CNN
@@
 	2500 2300 2500 2500
 $Comp
-L GND #PWR23
+L GND #PWR027
 U 1 1 5A74E3F6
 P 2500 2050
-F 0 "#PWR23" H 2500 1800 50  0001 C CNN
+F 0 "#PWR027" H 2500 1800 50  0001 C CNN
 F 1 "GND" H 2500 1900 50  0000 C CNN
 F 2 "" H 2500 2050 50  0000 C CNN
@@
 $EndComp
 $Comp
-L GND #PWR24
+L GND #PWR028
 U 1 1 5A74E420
 P 2500 2850
-F 0 "#PWR24" H 2500 2600 50  0001 C CNN
+F 0 "#PWR028" H 2500 2600 50  0001 C CNN
 F 1 "GND" H 2500 2700 50  0000 C CNN
 F 2 "" H 2500 2850 50  0000 C CNN
@@
 Connection ~ 2500 2300
 $Comp
-L GND #PWR25
+L GND #PWR029
 U 1 1 5A74E67A
 P 3400 1850
-F 0 "#PWR25" H 3400 1600 50  0001 C CNN
+F 0 "#PWR029" H 3400 1600 50  0001 C CNN
 F 1 "GND" H 3400 1700 50  0000 C CNN
 F 2 "" H 3400 1850 50  0000 C CNN
@@
 $EndComp
 $Comp
-L GND #PWR26
+L GND #PWR030
 U 1 1 5A74E804
 P 3400 2600
-F 0 "#PWR26" H 3400 2350 50  0001 C CNN
+F 0 "#PWR030" H 3400 2350 50  0001 C CNN
 F 1 "GND" H 3400 2450 50  0000 C CNN
 F 2 "" H 3400 2600 50  0000 C CNN
@@
 	3400 2500 3500 2500
 $Comp
-L GND #PWR27
+L GND #PWR031
 U 1 1 5A74EC12
 P 4700 1850
-F 0 "#PWR27" H 4700 1600 50  0001 C CNN
+F 0 "#PWR031" H 4700 1600 50  0001 C CNN
 F 1 "GND" H 4700 1700 50  0000 C CNN
 F 2 "" H 4700 1850 50  0000 C CNN
@@
 $EndComp
 $Comp
-L GND #PWR28
+L GND #PWR032
 U 1 1 5A74ED5A
 P 4700 2600
-F 0 "#PWR28" H 4700 2350 50  0001 C CNN
+F 0 "#PWR032" H 4700 2350 50  0001 C CNN
 F 1 "GND" H 4700 2450 50  0000 C CNN
 F 2 "" H 4700 2600 50  0000 C CNN
@@
 	4700 2500 4700 2600
 $Comp
-L +5V #PWR30
+L +5V #PWR033
 U 1 1 5A74F2CA
 P 5000 1500
-F 0 "#PWR30" H 5000 1350 50  0001 C CNN
+F 0 "#PWR033" H 5000 1350 50  0001 C CNN
 F 1 "+5V" H 5000 1640 50  0000 C CNN
 F 2 "" H 5000 1500 50  0000 C CNN
@@
 	5000 1550 5000 1500
 $Comp
-L PWR_FLAG #FLG2
+L PWR_FLAG #FLG034
 U 1 1 5A74F572
 P 1500 1400
-F 0 "#FLG2" H 1500 1495 50  0001 C CNN
+F 0 "#FLG034" H 1500 1495 50  0001 C CNN
 F 1 "PWR_FLAG" H 1500 1580 50  0000 C CNN
 F 2 "" H 1500 1400 50  0000 C CNN
@@
 $EndComp
 $Comp
-L PWR_FLAG #FLG3
+L PWR_FLAG #FLG035
 U 1 1 5A74F59C
 P 1600 2200
-F 0 "#FLG3" H 1600 2295 50  0001 C CNN
+F 0 "#FLG035" H 1600 2295 50  0001 C CNN
 F 1 "PWR_FLAG" H 1600 2380 50  0000 C CNN
 F 2 "" H 1600 2200 50  0000 C CNN
@@
 $EndComp
 $Comp
-L PWR_FLAG #FLG4
+L PWR_FLAG #FLG036
 U 1 1 5A74F5C6
 P 1600 2450
-F 0 "#FLG4" H 1600 2545 50  0001 C CNN
+F 0 "#FLG036" H 1600 2545 50  0001 C CNN
 F 1 "PWR_FLAG" H 1600 2630 50  0000 C CNN
 F 2 "" H 1600 2450 50  0000 C CNN
@@
 $EndComp
 $Comp
-L GND #PWR32
+L GND #PWR037
 U 1 1 5A77C1FF
 P 5700 2000
-F 0 "#PWR32" H 5700 1750 50  0001 C CNN
+F 0 "#PWR037" H 5700 1750 50  0001 C CNN
 F 1 "GND" H 5700 1850 50  0000 C CNN
 F 2 "" H 5700 2000 50  0000 C CNN
@@
 	5200 2500 5350 2500
 $Comp
-L GND #PWR31
+L GND #PWR038
 U 1 1 5A782A30
 P 5250 2700
-F 0 "#PWR31" H 5250 2450 50  0001 C CNN
+F 0 "#PWR038" H 5250 2450 50  0001 C CNN
 F 1 "GND" H 5250 2550 50  0000 C CNN
 F 2 "" H 5250 2700 50  0000 C CNN
@@
 F 0 "R18" V 8880 2350 50  0000 C CNN
 F 1 "270R" V 8800 2350 50  0000 C CNN
-F 2 "Resistors_THT:R_Axial_DIN0207_L6.3mm_D2.5mm_P10.16mm_Horizontal" V 8730 2350 50  0001 C CNN
+F 2 "Resistors_SMD:R_1206_HandSoldering" V 8730 2350 50  0001 C CNN
 F 3 "" H 8800 2350 50  0000 C CNN
 	1    8800 2350
@@
 F 0 "R17" V 8230 2850 50  0000 C CNN
 F 1 "330R" V 8150 2850 50  0000 C CNN
-F 2 "Resistors_THT:R_Axial_DIN0207_L6.3mm_D2.5mm_P10.16mm_Horizontal" V 8080 2850 50  0001 C CNN
+F 2 "Resistors_SMD:R_1206_HandSoldering" V 8080 2850 50  0001 C CNN
 F 3 "" H 8150 2850 50  0000 C CNN
 	1    8150 2850
@@
 $EndComp
 $Comp
-L GND #PWR37
+L GND #PWR039
 U 1 1 5ABD58D3
 P 8150 3250
-F 0 "#PWR37" H 8150 3000 50  0001 C CNN
+F 0 "#PWR039" H 8150 3000 50  0001 C CNN
 F 1 "GND" H 8150 3100 50  0000 C CNN
 F 2 "" H 8150 3250 50  0000 C CNN
@@
 	5950 4000 6500 4000
 $Comp
-L +9V #PWR36
+L +9V #PWR040
 U 1 1 5ABD83E3
 P 7900 4000
-F 0 "#PWR36" H 7900 3850 50  0001 C CNN
+F 0 "#PWR040" H 7900 3850 50  0001 C CNN
 F 1 "+9V" H 7900 4140 50  0000 C CNN
 F 2 "" H 7900 4000 50  0000 C CNN
@@
 $EndComp
 $Comp
-L GND #PWR33
+L GND #PWR041
 U 1 1 5ABD8417
 P 6900 5000
-F 0 "#PWR33" H 6900 4750 50  0001 C CNN
+F 0 "#PWR041" H 6900 4750 50  0001 C CNN
 F 1 "GND" H 6900 4850 50  0000 C CNN
 F 2 "" H 6900 5000 50  0000 C CNN
@@
 F 0 "R16" V 7730 4300 50  0000 C CNN
 F 1 "470R" V 7650 4300 50  0000 C CNN
-F 2 "Resistors_THT:R_Axial_DIN0207_L6.3mm_D2.5mm_P10.16mm_Horizontal" V 7580 4300 50  0001 C CNN
+F 2 "Resistors_SMD:R_1206_HandSoldering" V 7580 4300 50  0001 C CNN
 F 3 "" H 7650 4300 50  0000 C CNN
 	1    7650 4300
@@
 F 0 "R15" V 6980 4800 50  0000 C CNN
 F 1 "3.3kR" V 6900 4800 50  0000 C CNN
-F 2 "Resistors_THT:R_Axial_DIN0207_L6.3mm_D2.5mm_P10.16mm_Horizontal" V 6830 4800 50  0001 C CNN
+F 2 "Resistors_SMD:R_1206_HandSoldering" V 6830 4800 50  0001 C CNN
 F 3 "" H 6900 4800 50  0000 C CNN
 	1    6900 4800
@@
 $EndComp
 $Comp
-L GND #PWR29
+L GND #PWR042
 U 1 1 5ABE142E
 P 4950 3150
-F 0 "#PWR29" H 4950 2900 50  0001 C CNN
+F 0 "#PWR042" H 4950 2900 50  0001 C CNN
 F 1 "GND" H 4950 3000 50  0000 C CNN
 F 2 "" H 4950 3150 50  0000 C CNN
