File: Electronique/Central/_autosave-central.kicad_pcb (KiCad board)
At the start: 2 copper layers, 175 x 90 mm, 57 parts, among them P1 CONN_02X03, P10 CONN_Selec, P11 CONN_01X02, P12 CONN_01X02, P13 CONN_01X02, P14 CONN_01X02, P15 CONN_01X02, P2 CONN_Speaker, P3 CONN_jack, P4 CONN_jacky_led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

Commit message: PCB Central
Routing:
- net GND: track 729.6 -> 829.5 mm, vias 6 -> 7
- net Net-(P1-Pad4): track 219.3 -> 298.9 mm, vias 3 -> 4
- net +2.8V: track 369.0 -> 422.7 mm, vias 1 -> 2
- net Net-(P5-Pad2): track 0.00 -> 26.3 mm, vias 0 -> 2
- net Net-(P4-Pad1): track 0.00 -> 7.02 mm
- net BATT: track 79.0 -> 82.6 mm
- net Net-(P1-Pad2): track 315.0 -> 318.4 mm
- net Net-(D4-Pad2): track 104.0 -> 102.4 mm
