File: Electronique/Central/Audio.sch (KiCad schematic (older format))
At the start: 9 parts, among them P2 CONN_Speaker, P3 CONN_jack, U4 TDA8541

Commit message: go routage
Parts:
- C3, C6: footprint (none) -> Capacitors_THT:CP_Radial_D8.0mm_P3.50mm
- C4, C5: footprint (none) -> Capacitors_THT:C_Rect_L7.0mm_W2.5mm_P5.00mm
- R5, R6: footprint (none) -> Resistors_THT:R_Axial_DIN0207_L6.3mm_D2.5mm_P10.16mm_Horizontal
Changed lines of the file:
@@
 LIBS:2
 LIBS:dsn2596
+LIBS:raspberry_pi_3
 LIBS:central-cache
 EELAYER 25 0
@@
 $EndComp
 $Comp
-L GND #PWR23
+L GND #PWR043
 U 1 1 5A74B1CD
 P 7100 3300
-F 0 "#PWR23" H 7100 3050 50  0001 C CNN
+F 0 "#PWR043" H 7100 3050 50  0001 C CNN
 F 1 "GND" H 7100 3150 50  0000 C CNN
 F 2 "" H 7100 3300 50  0000 C CNN
@@
 $EndComp
 $Comp
-L +5V #PWR22
+L +5V #PWR044
 U 1 1 5A74B2FA
 P 6950 3400
-F 0 "#PWR22" H 6950 3250 50  0001 C CNN
+F 0 "#PWR044" H 6950 3250 50  0001 C CNN
 F 1 "+5V" H 6950 3540 50  0000 C CNN
 F 2 "" H 6950 3400 50  0000 C CNN
@@
 	7600 3500 6700 3500
 $Comp
-L GND #PWR20
+L GND #PWR045
 U 1 1 5A74B53B
 P 5250 3050
-F 0 "#PWR20" H 5250 2800 50  0001 C CNN
+F 0 "#PWR045" H 5250 2800 50  0001 C CNN
 F 1 "GND" H 5250 2900 50  0000 C CNN
 F 2 "" H 5250 3050 50  0000 C CNN
@@
 F 0 "C3" H 4875 3600 50  0000 L CNN
 F 1 "47uCP" H 4875 3400 50  0000 L CNN
-F 2 "" H 4888 3350 50  0001 C CNN
+F 2 "Capacitors_THT:CP_Radial_D8.0mm_P3.50mm" H 4888 3350 50  0001 C CNN
 F 3 "" H 4850 3500 50  0000 C CNN
 	1    4850 3500
@@
 Connection ~ 5200 3300
 $Comp
-L GND #PWR19
+L GND #PWR046
 U 1 1 5A74B7C7
 P 4850 3800
-F 0 "#PWR19" H 4850 3550 50  0001 C CNN
+F 0 "#PWR046" H 4850 3550 50  0001 C CNN
 F 1 "GND" H 4850 3650 50  0000 C CNN
 F 2 "" H 4850 3800 50  0000 C CNN
@@
 F 0 "R6" V 6430 3900 50  0000 C CNN
 F 1 "56kR" V 6350 3900 50  0000 C CNN
-F 2 "" V 6280 3900 50  0001 C CNN
+F 2 "Resistors_THT:R_Axial_DIN0207_L6.3mm_D2.5mm_P10.16mm_Horizontal" V 6280 3900 50  0001 C CNN
 F 3 "" H 6350 3900 50  0000 C CNN
 	1    6350 3900
@@
 F 0 "R5" V 5380 4200 50  0000 C CNN
 F 1 "11kR" V 5300 4200 50  0000 C CNN
-F 2 "" V 5230 4200 50  0001 C CNN
+F 2 "Resistors_THT:R_Axial_DIN0207_L6.3mm_D2.5mm_P10.16mm_Horizontal" V 5230 4200 50  0001 C CNN
 F 3 "" H 5300 4200 50  0000 C CNN
 	1    5300 4200
@@
 F 0 "C4" H 5325 4650 50  0000 L CNN
 F 1 "1uC" H 5325 4450 50  0000 L CNN
-F 2 "" H 5338 4400 50  0001 C CNN
+F 2 "Capacitors_THT:C_Rect_L7.0mm_W2.5mm_P5.00mm" H 5338 4400 50  0001 C CNN
 F 3 "" H 5300 4550 50  0000 C CNN
 	1    5300 4550
@@
 $EndComp
 $Comp
-L GND #PWR21
+L GND #PWR047
 U 1 1 5A74BFFC
 P 5400 4950
-F 0 "#PWR21" H 5400 4700 50  0001 C CNN
+F 0 "#PWR047" H 5400 4700 50  0001 C CNN
 F 1 "GND" H 5400 4800 50  0000 C CNN
 F 2 "" H 5400 4950 50  0000 C CNN
@@
 F 0 "C5" H 8825 3650 50  0000 L CNN
 F 1 "C" H 8825 3450 50  0000 L CNN
-F 2 "" H 8838 3400 50  0000 C CNN
+F 2 "Capacitors_THT:C_Rect_L7.0mm_W2.5mm_P5.00mm" H 8838 3400 50  0001 C CNN
 F 3 "" H 8800 3550 50  0000 C CNN
 	1    8800 3550
@@
 F 0 "C6" H 9125 3650 50  0000 L CNN
 F 1 "CP" H 9125 3450 50  0000 L CNN
-F 2 "" H 9138 3400 50  0000 C CNN
+F 2 "Capacitors_THT:CP_Radial_D8.0mm_P3.50mm" H 9138 3400 50  0001 C CNN
 F 3 "" H 9100 3550 50  0000 C CNN
 	1    9100 3550
@@
 $EndComp
 $Comp
-L GND #PWR25
+L GND #PWR048
 U 1 1 5A752015
 P 8800 3800
-F 0 "#PWR25" H 8800 3550 50  0001 C CNN
+F 0 "#PWR048" H 8800 3550 50  0001 C CNN
 F 1 "GND" H 8800 3650 50  0000 C CNN
 F 2 "" H 8800 3800 50  0000 C CNN
@@
 $EndComp
 $Comp
-L GND #PWR26
+L GND #PWR049
 U 1 1 5A75203B
 P 9100 3800
-F 0 "#PWR26" H 9100 3550 50  0001 C CNN
+F 0 "#PWR049" H 9100 3550 50  0001 C CNN
 F 1 "GND" H 9100 3650 50  0000 C CNN
 F 2 "" H 9100 3800 50  0000 C CNN
@@
 $EndComp
 $Comp
-L +5V #PWR24
+L +5V #PWR050
 U 1 1 5A752061
 P 8800 3300
-F 0 "#PWR24" H 8800 3150 50  0001 C CNN
+F 0 "#PWR050" H 8800 3150 50  0001 C CNN
 F 1 "+5V" H 8800 3440 50  0000 C CNN
 F 2 "" H 8800 3300 50  0000 C CNN

Commit message: schéma ok
Parts:
- removed C3: 47uCP, Capacitors_THT:CP_Radial_D8.0mm_P3.50mm, symbol CP
- removed C5: C, Capacitors_THT:C_Rect_L7.0mm_W2.5mm_P5.00mm, symbol C
- removed C6: CP, Capacitors_THT:CP_Radial_D8.0mm_P3.50mm, symbol CP
- removed R5: 11kR, Resistors_THT:R_Axial_DIN0207_L6.3mm_D2.5mm_P10.16mm_Horizontal, symbol R
- removed R6: 56kR, Resistors_THT:R_Axial_DIN0207_L6.3mm_D2.5mm_P10.16mm_Horizontal, symbol R
- removed U4: TDA8541, Housings_SOIC:SOIC-8_3.9x4.9mm_Pitch1.27mm, symbol TDA8541
- added C3: 1uC, symbol C
- added R19, R21: 20kR, symbol R
- added R20: 10kR, symbol R
- added U4: TDA6205, symbol TDA6205
- C4: value 1uC -> 390nC; footprint Capacitors_THT:C_Rect_L7.0mm_W2.5mm_P5.00mm -> (none)
Connections:
- wire segments 26 -> 22
Other:
- note added: "FIXED!"
- note added: "G=2*R21/R19"
- note added: "LM4991"
- note removed: "gain=2*R6/R5"
- moved on the sheet: P2, P3

Commit message: schéma ajout découplage
Parts:
- added C6: C, symbol C
Connections:
- wire segments 22 -> 24
Changed lines of the file:
@@
 $EndComp
 $Comp
-L GND #PWR043
+L GND #PWR41
 U 1 1 5A74BFFC
 P 4550 4950
-F 0 "#PWR043" H 4550 4700 50  0001 C CNN
+F 0 "#PWR41" H 4550 4700 50  0001 C CNN
 F 1 "GND" H 4550 4800 50  0000 C CNN
 F 2 "" H 4550 4950 50  0000 C CNN
@@
 	7600 3350 7850 3350
 $Comp
-L +5V #PWR044
+L +5V #PWR44
 U 1 1 5ABDF94E
 P 7050 3450
-F 0 "#PWR044" H 7050 3300 50  0001 C CNN
+F 0 "#PWR44" H 7050 3300 50  0001 C CNN
 F 1 "+5V" H 7050 3590 50  0000 C CNN
 F 2 "" H 7050 3450 50  0000 C CNN
@@
 $EndComp
 $Comp
-L GND #PWR045
+L GND #PWR43
 U 1 1 5ABDF968
 P 7050 3200
-F 0 "#PWR045" H 7050 2950 50  0001 C CNN
+F 0 "#PWR43" H 7050 2950 50  0001 C CNN
 F 1 "GND" H 7050 3050 50  0000 C CNN
 F 2 "" H 7050 3200 50  0000 C CNN
@@
 Connection ~ 4650 3200
 $Comp
-L GND #PWR046
+L GND #PWR39
 U 1 1 5ABE0104
 P 3850 3200
-F 0 "#PWR046" H 3850 2950 50  0001 C CNN
+F 0 "#PWR39" H 3850 2950 50  0001 C CNN
 F 1 "GND" H 3850 3050 50  0000 C CNN
 F 2 "" H 3850 3200 50  0000 C CNN
@@
 $EndComp
 $Comp
-L GND #PWR047
+L GND #PWR40
 U 1 1 5ABE0358
 P 4100 3000
-F 0 "#PWR047" H 4100 2750 50  0001 C CNN
+F 0 "#PWR40" H 4100 2750 50  0001 C CNN
 F 1 "GND" H 4100 2850 50  0000 C CNN
 F 2 "" H 4100 3000 50  0000 C CNN
@@
 Text Notes 6650 2400 0    60   ~ 0
 FIXED!
+$Comp
+L C C6
+U 1 1 5ABE2F92
+P 7000 3700
+F 0 "C6" H 7025 3800 50  0000 L CNN
+F 1 "C" H 7025 3600 50  0000 L CNN
+F 2 "" H 7038 3550 50  0000 C CNN
+F 3 "" H 7000 3700 50  0000 C CNN
+	1    7000 3700
+	1    0    0    -1
+$EndComp
+$Comp
+L GND #PWR42
+U 1 1 5ABE2FF1
+P 7000 3950
+F 0 "#PWR42" H 7000 3700 50  0001 C CNN
+F 1 "GND" H 7000 3800 50  0000 C CNN
+F 2 "" H 7000 3950 50  0000 C CNN
+F 3 "" H 7000 3950 50  0000 C CNN
+	1    7000 3950
+	1    0    0    -1
+$EndComp
+Wire Wire Line
+	7000 3550 7000 3450
+Connection ~ 7000 3450
+Wire Wire Line
+	7000 3950 7000 3850
 $EndSCHEMATC

Commit message: ready to route
Parts:
- removed R20: 10kR, symbol R
- C3: footprint (none) -> Capacitors_THT:CP_Radial_D8.0mm_P3.50mm
- C4, C6: footprint (none) -> Capacitors_THT:C_Rect_L7.0mm_W2.5mm_P5.00mm
- R19, R21: footprint (none) -> Resistors_THT:R_Axial_DIN0207_L6.3mm_D2.5mm_P10.16mm_Horizontal
- U4: footprint (none) -> Housings_SOIC:SOIC-8_3.9x4.9mm_Pitch1.27mm
Connections:
- wire segments 24 -> 23
Changed lines of the file:
@@
 F 0 "U4" H 5900 3350 60  0000 C CNN
 F 1 "TDA6205" H 5900 3500 60  0000 C CNN
-F 2 "" H 5500 3350 60  0000 C CNN
+F 2 "Housings_SOIC:SOIC-8_3.9x4.9mm_Pitch1.27mm" H 5500 3350 60  0001 C CNN
 F 3 "" H 5500 3350 60  0000 C CNN
 	1    5500 3350
@@
 F 0 "C4" H 4475 4600 50  0000 L CNN
 F 1 "390nC" H 4475 4400 50  0000 L CNN
-F 2 "" H 4488 4350 50  0000 C CNN
+F 2 "Capacitors_THT:C_Rect_L7.0mm_W2.5mm_P5.00mm" H 4488 4350 50  0001 C CNN
 F 3 "" H 4450 4500 50  0000 C CNN
 	1    4450 4500
@@
 F 0 "R19" V 4530 4050 50  0000 C CNN
 F 1 "20kR" V 4450 4050 50  0000 C CNN
-F 2 "" V 4380 4050 50  0000 C CNN
+F 2 "Resistors_THT:R_Axial_DIN0207_L6.3mm_D2.5mm_P10.16mm_Horizontal" V 4380 4050 50  0001 C CNN
 F 3 "" H 4450 4050 50  0000 C CNN
 	1    4450 4050
@@
 F 0 "C3" H 4225 3300 50  0000 L CNN
 F 1 "1uC" H 4225 3100 50  0000 L CNN
-F 2 "" H 4238 3050 50  0000 C CNN
+F 2 "Capacitors_THT:CP_Radial_D8.0mm_P3.50mm" H 4238 3050 50  0001 C CNN
 F 3 "" H 4200 3200 50  0000 C CNN
 	1    4200 3200
@@
 	3850 3200 4050 3200
 $Comp
-L R R20
-U 1 1 5ABE02F3
-P 4500 3000
-F 0 "R20" V 4580 3000 50  0000 C CNN
-F 1 "10kR" V 4500 3000 50  0000 C CNN
-F 2 "" V 4430 3000 50  0000 C CNN
-F 3 "" H 4500 3000 50  0000 C CNN
-	1    4500 3000
-	0    1    1    0
-$EndComp
-$Comp
 L GND #PWR40
 U 1 1 5ABE0358
@@
 $EndComp
 Wire Wire Line
-	4100 3000 4350 3000
-Wire Wire Line
-	4650 3000 5050 3000
+	4100 3000 5050 3000
 $Comp
 L R R21
@@
 F 0 "R21" V 6080 4100 50  0000 C CNN
 F 1 "20kR" V 6000 4100 50  0000 C CNN
-F 2 "" V 5930 4100 50  0000 C CNN
+F 2 "Resistors_THT:R_Axial_DIN0207_L6.3mm_D2.5mm_P10.16mm_Horizontal" V 5930 4100 50  0001 C CNN
 F 3 "" H 6000 4100 50  0000 C CNN
 	1    6000 4100
@@
 F 0 "C6" H 7025 3800 50  0000 L CNN
 F 1 "C" H 7025 3600 50  0000 L CNN
-F 2 "" H 7038 3550 50  0000 C CNN
+F 2 "Capacitors_THT:C_Rect_L7.0mm_W2.5mm_P5.00mm" H 7038 3550 50  0001 C CNN
 F 3 "" H 7000 3700 50  0000 C CNN
 	1    7000 3700

Commit message: smd resistor
Parts:
- R19, R21: footprint Resistors_THT:R_Axial_DIN0207_L6.3mm_D2.5mm_P10.16mm_Horizontal -> Resistors_SMD:R_1206_HandSoldering
Changed lines of the file:
@@
 $EndComp
 $Comp
-L GND #PWR41
+L GND #PWR043
 U 1 1 5A74BFFC
 P 4550 4950
-F 0 "#PWR41" H 4550 4700 50  0001 C CNN
+F 0 "#PWR043" H 4550 4700 50  0001 C CNN
 F 1 "GND" H 4550 4800 50  0000 C CNN
 F 2 "" H 4550 4950 50  0000 C CNN
@@
 	7600 3350 7850 3350
 $Comp
-L +5V #PWR44
+L +5V #PWR044
 U 1 1 5ABDF94E
 P 7050 3450
-F 0 "#PWR44" H 7050 3300 50  0001 C CNN
+F 0 "#PWR044" H 7050 3300 50  0001 C CNN
 F 1 "+5V" H 7050 3590 50  0000 C CNN
 F 2 "" H 7050 3450 50  0000 C CNN
@@
 $EndComp
 $Comp
-L GND #PWR43
+L GND #PWR045
 U 1 1 5ABDF968
 P 7050 3200
-F 0 "#PWR43" H 7050 2950 50  0001 C CNN
+F 0 "#PWR045" H 7050 2950 50  0001 C CNN
 F 1 "GND" H 7050 3050 50  0000 C CNN
 F 2 "" H 7050 3200 50  0000 C CNN
@@
 F 0 "R19" V 4530 4050 50  0000 C CNN
 F 1 "20kR" V 4450 4050 50  0000 C CNN
-F 2 "Resistors_THT:R_Axial_DIN0207_L6.3mm_D2.5mm_P10.16mm_Horizontal" V 4380 4050 50  0001 C CNN
+F 2 "Resistors_SMD:R_1206_HandSoldering" V 4380 4050 50  0001 C CNN
 F 3 "" H 4450 4050 50  0000 C CNN
 	1    4450 4050
@@
 Connection ~ 4650 3200
 $Comp
-L GND #PWR39
+L GND #PWR046
 U 1 1 5ABE0104
 P 3850 3200
-F 0 "#PWR39" H 3850 2950 50  0001 C CNN
+F 0 "#PWR046" H 3850 2950 50  0001 C CNN
 F 1 "GND" H 3850 3050 50  0000 C CNN
 F 2 "" H 3850 3200 50  0000 C CNN
@@
 	3850 3200 4050 3200
 $Comp
-L GND #PWR40
+L GND #PWR047
 U 1 1 5ABE0358
 P 4100 3000
-F 0 "#PWR40" H 4100 2750 50  0001 C CNN
+F 0 "#PWR047" H 4100 2750 50  0001 C CNN
 F 1 "GND" H 4100 2850 50  0000 C CNN
 F 2 "" H 4100 3000 50  0000 C CNN
@@
 F 0 "R21" V 6080 4100 50  0000 C CNN
 F 1 "20kR" V 6000 4100 50  0000 C CNN
-F 2 "Resistors_THT:R_Axial_DIN0207_L6.3mm_D2.5mm_P10.16mm_Horizontal" V 5930 4100 50  0001 C CNN
+F 2 "Resistors_SMD:R_1206_HandSoldering" V 5930 4100 50  0001 C CNN
 F 3 "" H 6000 4100 50  0000 C CNN
 	1    6000 4100
@@
 $EndComp
 $Comp
-L GND #PWR42
+L GND #PWR048
 U 1 1 5ABE2FF1
 P 7000 3950
-F 0 "#PWR42" H 7000 3700 50  0001 C CNN
+F 0 "#PWR048" H 7000 3700 50  0001 C CNN
 F 1 "GND" H 7000 3800 50  0000 C CNN
 F 2 "" H 7000 3950 50  0000 C CNN
