File: Electronique/Central/LED.sch (KiCad schematic (older format))
At the start: 4 parts

Commit message: go routage
Parts:
- P4, P5: renamed from P?; footprint (none) -> Connectors_Molex:Molex_KK-6410-02_02x2.54mm_Straight
- Q1: renamed from Q?; footprint TO-220 -> Power_Integrations:TO-220
- U9: renamed from U?; footprint (none) -> Housings_DIP:DIP-8_W7.62mm_LongPads
Changed lines of the file:
@@
 LIBS:2
 LIBS:dsn2596
+LIBS:raspberry_pi_3
 LIBS:central-cache
 EELAYER 25 0
@@
 $EndDescr
 $Comp
-L IRF540N Q?
+L IRF540N Q1
 U 1 1 5A76719A
 P 6200 3550
-F 0 "Q?" H 6450 3625 50  0000 L CNN
+F 0 "Q1" H 6450 3625 50  0000 L CNN
 F 1 "IRF540N" H 6450 3550 50  0000 L CNN
-F 2 "TO-220" H 6450 3475 50  0000 L CIN
+F 2 "Power_Integrations:TO-220" H 6450 3475 50  0000 L CIN
 F 3 "" H 6200 3550 50  0000 L CNN
 	1    6200 3550
@@
 Jacky tuning
 $Comp
-L MC34152 U?
+L MC34152 U9
 U 1 1 5A767332
 P 4600 3900
-F 0 "U?" H 4600 4000 60  0000 C CNN
+F 0 "U9" H 4600 4000 60  0000 C CNN
 F 1 "MC34152" H 4650 4150 60  0000 C CNN
-F 2 "" H 4600 3900 60  0000 C CNN
+F 2 "Housings_DIP:DIP-8_W7.62mm_LongPads" H 4600 3900 60  0001 C CNN
 F 3 "" H 4600 3900 60  0000 C CNN
 	1    4600 3900
@@
 NoConn ~ 5350 3800
 $Comp
-L GND #PWR?
+L GND #PWR051
 U 1 1 5A767FBA
 P 3900 3800
-F 0 "#PWR?" H 3900 3550 50  0001 C CNN
+F 0 "#PWR051" H 3900 3550 50  0001 C CNN
 F 1 "GND" H 3900 3650 50  0000 C CNN
 F 2 "" H 3900 3800 50  0000 C CNN
@@
 $EndComp
 $Comp
-L GND #PWR?
+L GND #PWR052
 U 1 1 5A767FD6
 P 3900 3700
-F 0 "#PWR?" H 3900 3450 50  0001 C CNN
+F 0 "#PWR052" H 3900 3450 50  0001 C CNN
 F 1 "GND" H 3900 3550 50  0000 C CNN
 F 2 "" H 3900 3700 50  0000 C CNN
@@
 	5350 3600 6000 3600
 $Comp
-L CONN_01X02 P?
+L CONN_01X02 P4
 U 1 1 5A76819E
 P 3250 3950
-F 0 "P?" H 3250 4100 50  0000 C CNN
+F 0 "P4" H 3250 4100 50  0000 C CNN
 F 1 "CONN_jacky_led" V 3350 3950 50  0000 C CNN
-F 2 "" H 3250 3950 50  0000 C CNN
+F 2 "Connectors_Molex:Molex_KK-6410-02_02x2.54mm_Straight" H 3250 3950 50  0001 C CNN
 F 3 "" H 3250 3950 50  0000 C CNN
 	1    3250 3950
@@
 	3300 3600 4000 3600
 $Comp
-L GND #PWR?
+L GND #PWR053
 U 1 1 5A768319
 P 3000 3700
-F 0 "#PWR?" H 3000 3450 50  0001 C CNN
+F 0 "#PWR053" H 3000 3450 50  0001 C CNN
 F 1 "GND" H 3000 3550 50  0000 C CNN
 F 2 "" H 3000 3700 50  0000 C CNN
@@
 	3200 3700 3200 3750
 $Comp
-L GND #PWR?
+L GND #PWR054
 U 1 1 5A7685B8
 P 6300 3900
-F 0 "#PWR?" H 6300 3650 50  0001 C CNN
+F 0 "#PWR054" H 6300 3650 50  0001 C CNN
 F 1 "GND" H 6300 3750 50  0000 C CNN
 F 2 "" H 6300 3900 50  0000 C CNN
@@
 	6300 3750 6300 3900
 $Comp
-L CONN_01X02 P?
+L CONN_01X02 P5
 U 1 1 5A76883C
 P 6600 3050
-F 0 "P?" H 6600 3200 50  0000 C CNN
+F 0 "P5" H 6600 3200 50  0000 C CNN
 F 1 "CONN_LED" V 6700 3050 50  0000 C CNN
-F 2 "" H 6600 3050 50  0000 C CNN
+F 2 "Connectors_Molex:Molex_KK-6410-02_02x2.54mm_Straight" H 6600 3050 50  0001 C CNN
 F 3 "" H 6600 3050 50  0000 C CNN
 	1    6600 3050
@@
 $EndComp
 $Comp
-L +5V #PWR?
+L +5V #PWR055
 U 1 1 5A768873
 P 6300 2850
-F 0 "#PWR?" H 6300 2700 50  0001 C CNN
+F 0 "#PWR055" H 6300 2700 50  0001 C CNN
 F 1 "+5V" H 6300 2990 50  0000 C CNN
 F 2 "" H 6300 2850 50  0000 C CNN

Commit message: Routage PCB central
Parts:
- Q1: symbol IRF540N -> IRF540N-RESCUE-central
Changed lines of the file:
@@
 EESchema Schematic File Version 2
+LIBS:central-rescue
 LIBS:power
 LIBS:device
@@
 $EndDescr
 $Comp
-L IRF540N Q1
+L IRF540N-RESCUE-central Q1
 U 1 1 5A76719A
 P 6200 3550
@@
 NoConn ~ 5350 3800
 $Comp
-L GND #PWR051
+L GND #PWR049
 U 1 1 5A767FBA
 P 3900 3800
-F 0 "#PWR051" H 3900 3550 50  0001 C CNN
+F 0 "#PWR049" H 3900 3550 50  0001 C CNN
 F 1 "GND" H 3900 3650 50  0000 C CNN
 F 2 "" H 3900 3800 50  0000 C CNN
@@
 $EndComp
 $Comp
-L GND #PWR052
+L GND #PWR050
 U 1 1 5A767FD6
 P 3900 3700
-F 0 "#PWR052" H 3900 3450 50  0001 C CNN
+F 0 "#PWR050" H 3900 3450 50  0001 C CNN
 F 1 "GND" H 3900 3550 50  0000 C CNN
 F 2 "" H 3900 3700 50  0000 C CNN
@@
 	3300 3600 4000 3600
 $Comp
-L GND #PWR053
+L GND #PWR051
 U 1 1 5A768319
 P 3000 3700
-F 0 "#PWR053" H 3000 3450 50  0001 C CNN
+F 0 "#PWR051" H 3000 3450 50  0001 C CNN
 F 1 "GND" H 3000 3550 50  0000 C CNN
 F 2 "" H 3000 3700 50  0000 C CNN
@@
 	3200 3700 3200 3750
 $Comp
-L GND #PWR054
+L GND #PWR052
 U 1 1 5A7685B8
 P 6300 3900
-F 0 "#PWR054" H 6300 3650 50  0001 C CNN
+F 0 "#PWR052" H 6300 3650 50  0001 C CNN
 F 1 "GND" H 6300 3750 50  0000 C CNN
 F 2 "" H 6300 3900 50  0000 C CNN
@@
 $EndComp
 $Comp
-L +5V #PWR055
+L +5V #PWR053
 U 1 1 5A768873
 P 6300 2850
-F 0 "#PWR055" H 6300 2700 50  0001 C CNN
+F 0 "#PWR053" H 6300 2700 50  0001 C CNN
 F 1 "+5V" H 6300 2990 50  0000 C CNN
 F 2 "" H 6300 2850 50  0000 C CNN

Commit message: schéma ok
Connections:
- net labels added: +9V
- net labels removed: BATT
Changed lines of the file:
@@
 	1    0    0    -1
 $EndComp
-Text GLabel 5550 3700 2    60   Input ~ 0
-BATT
 NoConn ~ 5350 3500
 NoConn ~ 4000 3500
 NoConn ~ 5350 3800
 $Comp
-L GND #PWR049
+L GND #PWR048
 U 1 1 5A767FBA
 P 3900 3800
-F 0 "#PWR049" H 3900 3550 50  0001 C CNN
+F 0 "#PWR048" H 3900 3550 50  0001 C CNN
 F 1 "GND" H 3900 3650 50  0000 C CNN
 F 2 "" H 3900 3800 50  0000 C CNN
@@
 $EndComp
 $Comp
-L GND #PWR050
+L GND #PWR049
 U 1 1 5A767FD6
 P 3900 3700
-F 0 "#PWR050" H 3900 3450 50  0001 C CNN
+F 0 "#PWR049" H 3900 3450 50  0001 C CNN
 F 1 "GND" H 3900 3550 50  0000 C CNN
 F 2 "" H 3900 3700 50  0000 C CNN
@@
 Wire Wire Line
 	3900 3800 4000 3800
-Wire Wire Line
-	5350 3700 5550 3700
 Wire Wire Line
 	5350 3600 6000 3600
@@
 	3300 3600 4000 3600
 $Comp
-L GND #PWR051
+L GND #PWR050
 U 1 1 5A768319
 P 3000 3700
-F 0 "#PWR051" H 3000 3450 50  0001 C CNN
+F 0 "#PWR050" H 3000 3450 50  0001 C CNN
 F 1 "GND" H 3000 3550 50  0000 C CNN
 F 2 "" H 3000 3700 50  0000 C CNN
@@
 	3200 3700 3200 3750
 $Comp
-L GND #PWR052
+L GND #PWR051
 U 1 1 5A7685B8
 P 6300 3900
-F 0 "#PWR052" H 6300 3650 50  0001 C CNN
+F 0 "#PWR051" H 6300 3650 50  0001 C CNN
 F 1 "GND" H 6300 3750 50  0000 C CNN
 F 2 "" H 6300 3900 50  0000 C CNN
@@
 $EndComp
 $Comp
-L +5V #PWR053
+L +5V #PWR052
 U 1 1 5A768873
 P 6300 2850
-F 0 "#PWR053" H 6300 2700 50  0001 C CNN
+F 0 "#PWR052" H 6300 2700 50  0001 C CNN
 F 1 "+5V" H 6300 2990 50  0000 C CNN
 F 2 "" H 6300 2850 50  0000 C CNN
@@
 Wire Wire Line
 	6300 3100 6300 3350
+$Comp
+L +9V #PWR053
+U 1 1 5ABD7B5A
+P 5550 3700
+F 0 "#PWR053" H 5550 3550 50  0001 C CNN
+F 1 "+9V" H 5550 3840 50  0000 C CNN
+F 2 "" H 5550 3700 50  0000 C CNN
+F 3 "" H 5550 3700 50  0000 C CNN
+	1    5550 3700
+	0    1    1    0
+$EndComp
+Wire Wire Line
+	5350 3700 5550 3700
 $EndSCHEMATC
