File: Electronique/Central/central.sch (KiCad schematic (older format))
At the start: 7 parts, among them P1 CONN_TOF_04, U1 Nucleo-64, U3 I2C_repeater

Commit message: led!
Parts:
- gave numbers to parts that had none: 4
Connections:
- wire segments 34 -> 41
- no-connect marks 12 -> 22
Changed lines of the file:
@@
 LIBS:valves
 LIBS:Nucleo_64
+LIBS:2
+LIBS:dsn2596
+LIBS:central-cache
 EELAYER 25 0
 EELAYER END
 $Descr A2 16535 23386 portrait
 encoding utf-8
-Sheet 1 2
+Sheet 1 4
 Title ""
 Date ""
@@
 I2C_TOF_SCL
 $Comp
-L +5V #PWR01
+L +5V #PWR1
 U 1 1 5A6CAF8E
 P 3250 10750
-F 0 "#PWR01" H 3250 10600 50  0001 C CNN
+F 0 "#PWR1" H 3250 10600 50  0001 C CNN
 F 1 "+5V" H 3250 10890 50  0000 C CNN
 F 2 "" H 3250 10750 50  0000 C CNN
@@
 NoConn ~ 4750 12650
 $Comp
-L +3.3V #PWR02
+L +3.3V #PWR2
 U 1 1 5A6CB32D
 P 4250 11800
-F 0 "#PWR02" H 4250 11650 50  0001 C CNN
+F 0 "#PWR2" H 4250 11650 50  0001 C CNN
 F 1 "+3.3V" H 4250 11940 50  0000 C CNN
 F 2 "" H 4250 11800 50  0000 C CNN
@@
 	13300 11850 13900 11850
 $Comp
-L GND #PWR03
+L GND #PWR4
 U 1 1 5A6CC583
 P 14500 12200
-F 0 "#PWR03" H 14500 11950 50  0001 C CNN
+F 0 "#PWR4" H 14500 11950 50  0001 C CNN
 F 1 "GND" H 14500 12050 50  0000 C CNN
 F 2 "" H 14500 12200 50  0000 C CNN
@@
 $EndComp
 $Comp
-L +3.3V #PWR04
+L +3.3V #PWR3
 U 1 1 5A6CC59B
 P 14300 10800
-F 0 "#PWR04" H 14300 10650 50  0001 C CNN
+F 0 "#PWR3" H 14300 10650 50  0001 C CNN
 F 1 "+3.3V" H 14300 10940 50  0000 C CNN
 F 2 "" H 14300 10800 50  0000 C CNN
@@
 	15350 11550 15650 11550
 $Comp
-L GND #PWR05
+L GND #PWR5
 U 1 1 5A6CC78A
 P 15250 11800
-F 0 "#PWR05" H 15250 11550 50  0001 C CNN
+F 0 "#PWR5" H 15250 11550 50  0001 C CNN
 F 1 "GND" H 15250 11650 50  0000 C CNN
 F 2 "" H 15250 11800 50  0000 C CNN
@@
 	15650 12150 15650 11750
 $Comp
-L R R?
+L R R2
 U 1 1 5A6CC90A
 P 13650 11150
-F 0 "R?" V 13730 11150 50  0000 C CNN
+F 0 "R2" V 13730 11150 50  0000 C CNN
 F 1 "10kR" V 13650 11150 50  0000 C CNN
-F 2 "" V 13580 11150 50  0000 C CNN
+F 2 "" V 13580 11150 50  0001 C CNN
 F 3 "" H 13650 11150 50  0000 C CNN
 	1    13650 11150
@@
 $EndComp
 $Comp
-L R R?
+L R R1
 U 1 1 5A6CC927
 P 13500 11400
-F 0 "R?" V 13580 11400 50  0000 C CNN
+F 0 "R1" V 13580 11400 50  0000 C CNN
 F 1 "10kR" V 13500 11400 50  0000 C CNN
-F 2 "" V 13430 11400 50  0000 C CNN
+F 2 "" V 13430 11400 50  0001 C CNN
 F 3 "" H 13500 11400 50  0000 C CNN
 	1    13500 11400
@@
 $EndComp
 $Comp
-L R R?
+L R R3
 U 1 1 5A6CC988
 P 15250 11150
-F 0 "R?" V 15330 11150 50  0000 C CNN
+F 0 "R3" V 15330 11150 50  0000 C CNN
 F 1 "10kR" V 15250 11150 50  0000 C CNN
-F 2 "" V 15180 11150 50  0000 C CNN
+F 2 "" V 15180 11150 50  0001 C CNN
 F 3 "" H 15250 11150 50  0000 C CNN
 	1    15250 11150
@@
 $EndComp
 $Comp
-L R R?
+L R R4
 U 1 1 5A6CC9AD
 P 15500 11350
-F 0 "R?" V 15580 11350 50  0000 C CNN
+F 0 "R4" V 15580 11350 50  0000 C CNN
 F 1 "10kR" V 15500 11350 50  0000 C CNN
-F 2 "" V 15430 11350 50  0000 C CNN
+F 2 "" V 15430 11350 50  0001 C CNN
 F 3 "" H 15500 11350 50  0000 C CNN
 	1    15500 11350
@@
 Wire Wire Line
 	11850 12850 12050 12850
+$Sheet
+S 10600 1350 3650 1450
+U 5A74AF92
+F0 "Audio" 60
+F1 "Audio.sch" 60
+$EndSheet
+NoConn ~ 4750 9250
+NoConn ~ 4750 6850
+NoConn ~ 4750 7050
+NoConn ~ 4750 6650
+NoConn ~ 4750 5850
+NoConn ~ 5300 4750
+NoConn ~ 5500 4750
+NoConn ~ 11300 4750
+NoConn ~ 11500 4750
+$Comp
+L +3.3V #PWR?
+U 1 1 5A7641EB
+P 4400 6450
+F 0 "#PWR?" H 4400 6300 50  0001 C CNN
+F 1 "+3.3V" H 4400 6590 50  0000 C CNN
+F 2 "" H 4400 6450 50  0000 C CNN
+F 3 "" H 4400 6450 50  0000 C CNN
+	1    4400 6450
+	0    -1   -1   0
+$EndComp
+Wire Wire Line
+	4400 6450 4750 6450
+$Comp
+L GND #PWR?
+U 1 1 5A764D00
+P 4550 11050
+F 0 "#PWR?" H 4550 10800 50  0001 C CNN
+F 1 "GND" H 4550 10900 50  0000 C CNN
+F 2 "" H 4550 11050 50  0000 C CNN
+F 3 "" H 4550 11050 50  0000 C CNN
+	1    4550 11050
+	0    1    1    0
+$EndComp
+Wire Wire Line
+	4550 11050 4750 11050
+$Comp
+L GND #PWR?
+U 1 1 5A7650C8
+P 4500 12250
+F 0 "#PWR?" H 4500 12000 50  0001 C CNN
+F 1 "GND" H 4500 12100 50  0000 C CNN
+F 2 "" H 4500 12250 50  0000 C CNN
+F 3 "" H 4500 12250 50  0000 C CNN
+	1    4500 12250
+	0    1    1    0
+$EndComp
+$Comp
+L GND #PWR?
+U 1 1 5A7650EA
+P 4500 12450
+F 0 "#PWR?" H 4500 12200 50  0001 C CNN
+F 1 "GND" H 4500 12300 50  0000 C CNN
+F 2 "" H 4500 12450 50  0000 C CNN
+F 3 "" H 4500 12450 50  0000 C CNN
+	1    4500 12450
+	0    1    1    0
+$EndComp
+Wire Wire Line
+	4500 12250 4750 12250
+Wire Wire Line
+	4500 12450 4750 12450
+$Comp
+L GND #PWR?
+U 1 1 5A765594
+P 12100 11050
+F 0 "#PWR?" H 12100 10800 50  0001 C CNN
+F 1 "GND" H 12100 10900 50  0000 C CNN
+F 2 "" H 12100 11050 50  0000 C CNN
+F 3 "" H 12100 11050 50  0000 C CNN
+	1    12100 11050
+	0    -1   -1   0
+$EndComp
+Wire Wire Line
+	11850 11050 12100 11050
+NoConn ~ 11850 10850
+$Comp
+L GND #PWR?
+U 1 1 5A765CB2
+P 11950 9050
+F 0 "#PWR?" H 11950 8800 50  0001 C CNN
+F 1 "GND" H 11950 8900 50  0000 C CNN
+F 2 "" H 11950 9050 50  0000 C CNN
+F 3 "" H 11950 9050 50  0000 C CNN
+	1    11950 9050
+	0    -1   -1   0
+$EndComp
+Wire Wire Line
+	11850 9050 11950 9050
+$Comp
+L GND #PWR?
+U 1 1 5A766182
+P 11950 7850
+F 0 "#PWR?" H 11950 7600 50  0001 C CNN
+F 1 "GND" H 11950 7700 50  0000 C CNN
+F 2 "" H 11950 7850 50  0000 C CNN
+F 3 "" H 11950 7850 50  0000 C CNN
+	1    11950 7850
+	0    -1   -1   0
+$EndComp
+Wire Wire Line
+	11850 7850 11950 7850
+$Sheet
+S 10600 3050 3650 750
+U 5A76717C
+F0 "LED" 60
+F1 "LED.sch" 60
+$EndSheet
 $EndSCHEMATC

Commit message: go routage
Parts:
- removed P1: CONN_TOF_04, symbol CONN_01X04
- added D3: LED_Red, LEDs:LED_D5.0mm, symbol LED
- added D4: LED_Green, LEDs:LED_D5.0mm, symbol LED
- added P1, P6, P7, P8: CONN_02X03, Connectors_Molex:Molex_KK-6410-06_06x2.54mm_Straight, symbol CONN_02X03
- added P10: CONN_Selec, Connectors_Molex:Molex_KK-6410-02_02x2.54mm_Straight, symbol CONN_01X02
- added P12, P13, P14, P15: CONN_01X02, Connectors_Molex:Molex_KK-6410-02_02x2.54mm_Straight, symbol CONN_01X02
- added P9: CONN_jack_start, Connectors_Molex:Molex_KK-6410-02_02x2.54mm_Straight, symbol CONN_01X02
- added R10, R11, R12, R13, R14, R7, R8, R9: 47kR, Resistors_THT:R_Axial_DIN0207_L6.3mm_D2.5mm_P10.16mm_Horizontal, symbol R
- added U10, U11, U12, U13: trou-d3mm, Mounting_Holes:MountingHole_3.2mm_M3_Pad, symbol trou-d3mm
- added U14: Raspberry_pi_3, Raspberry_pi_3:Raspberry_pi_3, symbol Raspberry_pi_3
- R1, R2, R3, R4: footprint (none) -> Resistors_THT:R_Axial_DIN0207_L6.3mm_D2.5mm_P10.16mm_Horizontal
Connections:
- net labels added: I2C_Free_SCL, I2C_Free_SDA, Pince_RX, Pince_TX, Position_RX, Position_TX, RASP_RX, RASP_TX
- wire segments 41 -> 121
- no-connect marks 22 -> 59
Other:
- moved on the sheet: R1, R2, R3, R4, U3

Commit message: Routage PCB central
Parts:
- removed U14: Raspberry_pi_3, Raspberry_pi_3:Raspberry_pi_3, symbol Raspberry_pi_3
- added U14, U15: trou-d3mm, Mounting_Holes:MountingHole_3.2mm_M3_Pad, symbol trou-d3mm
- D3, D4: symbol LED -> LED-RESCUE-central
Connections:
- net GND: now also U14.1, U15.1
Changed lines of the file:
@@
 EESchema Schematic File Version 2
+LIBS:central-rescue
 LIBS:power
 LIBS:device
@@
 	4500 8050 4750 8050
 $Comp
-L LED D4
+L LED-RESCUE-central D4
 U 1 1 5A77434B
 P 12750 11450
@@
 $EndComp
 $Comp
-L LED D3
+L LED-RESCUE-central D3
 U 1 1 5A774398
 P 12400 11650
@@
 	14000 14750 14350 14750
 $Comp
-L Raspberry_pi_3 U14
-U 1 1 5A79217C
-P 10850 17350
-F 0 "U14" H 10850 17350 60  0000 C CNN
-F 1 "Raspberry_pi_3" H 10850 17500 60  0000 C CNN
-F 2 "Raspberry_pi_3:Raspberry_pi_3" H 10850 17350 60  0001 C CNN
-F 3 "" H 10850 17350 60  0000 C CNN
-	1    10850 17350
-	1    0    0    -1
-$EndComp
-$Comp
 L trou-d3mm U12
 U 1 1 5A79256F
@@
 	10850 18350 11300 18350
 Wire Wire Line
-	11300 17850 11300 19450
+	11300 17850 11300 20350
 Connection ~ 11300 17850
 Wire Wire Line
@@
 Connection ~ 11300 18900
 $Comp
-L GND #PWR023
-U 1 1 5A7662FE
-P 11450 17500
-F 0 "#PWR023" H 11450 17250 50  0001 C CNN
-F 1 "GND" H 11450 17350 50  0000 C CNN
-F 2 "" H 11450 17500 50  0000 C CNN
-F 3 "" H 11450 17500 50  0000 C CNN
-	1    11450 17500
-	1    0    0    -1
-$EndComp
-$Comp
-L GND #PWR024
-U 1 1 5A766350
-P 10150 17550
-F 0 "#PWR024" H 10150 17300 50  0001 C CNN
-F 1 "GND" H 10150 17400 50  0000 C CNN
-F 2 "" H 10150 17550 50  0000 C CNN
-F 3 "" H 10150 17550 50  0000 C CNN
-	1    10150 17550
-	1    0    0    -1
-$EndComp
-Wire Wire Line
-	11400 17100 11450 17100
-Wire Wire Line
-	11450 17100 11450 17500
-Wire Wire Line
-	11400 17450 11450 17450
-Connection ~ 11450 17450
-Wire Wire Line
-	10300 17100 10150 17100
-Wire Wire Line
-	10150 17100 10150 17550
-Wire Wire Line
-	10300 17450 10150 17450
-Connection ~ 10150 17450
+L trou-d3mm U14
+U 1 1 5A79FA80
+P 10600 19900
+F 0 "U14" H 10600 19900 60  0000 C CNN
+F 1 "trou-d3mm" H 10650 20000 60  0000 C CNN
+F 2 "Mounting_Holes:MountingHole_3.2mm_M3_Pad" H 10600 19900 60  0001 C CNN
+F 3 "" H 10600 19900 60  0001 C CNN
+	1    10600 19900
+	1    0    0    -1
+$EndComp
+$Comp
+L trou-d3mm U15
+U 1 1 5A79FB0F
+P 10600 20350
+F 0 "U15" H 10600 20350 60  0000 C CNN
+F 1 "trou-d3mm" H 10650 20450 60  0000 C CNN
+F 2 "Mounting_Holes:MountingHole_3.2mm_M3_Pad" H 10600 20350 60  0001 C CNN
+F 3 "" H 10600 20350 60  0001 C CNN
+	1    10600 20350
+	1    0    0    -1
+$EndComp
+Wire Wire Line
+	11300 19900 10950 19900
+Connection ~ 11300 19450
+Wire Wire Line
+	11300 20350 10950 20350
+Connection ~ 11300 19900
 $EndSCHEMATC

Commit message: i2c converter reference
Other:
- note added: "PCA9515"
Changed lines of the file:
@@
 	11300 20350 10950 20350
 Connection ~ 11300 19900
+Text Notes 3700 17450 0    60   ~ 0
+PCA9515
 $EndSCHEMATC

Commit message: schéma ok
Parts:
- removed U3: I2C_repeater, Housings_SOIC:SOIC-8_3.9x4.9mm_Pitch1.27mm, symbol I2C_repeater
- added Q2, Q3: Q_NMOS_DGS, symbol Q_NMOS_DGS
- added R5, R6: 500R, symbol R
Connections:
- net labels removed: I2C_TOF_EN
- wire segments 117 -> 119
- no-connect marks 59 -> 60
Other:
- note added: "FIXED!"
- note added: "Use BSS138"
- note removed: "PCA9515"
- moved on the sheet: D3, R1, R2

Commit message: ready to route
Parts:
- Q2, Q3: footprint (none) -> TO_SOT_Packages_SMD:SOT-323_SC-70_Handsoldering
- R5, R6: footprint (none) -> Resistors_THT:R_Axial_DIN0207_L6.3mm_D2.5mm_P10.16mm_Horizontal
Changed lines of the file:
@@
 F 0 "R5" V 12280 11450 50  0000 C CNN
 F 1 "500R" V 12200 11450 50  0000 C CNN
-F 2 "" V 12130 11450 50  0000 C CNN
+F 2 "Resistors_THT:R_Axial_DIN0207_L6.3mm_D2.5mm_P10.16mm_Horizontal" V 12130 11450 50  0001 C CNN
 F 3 "" H 12200 11450 50  0000 C CNN
 	1    12200 11450
@@
 F 0 "R6" V 12280 11650 50  0000 C CNN
 F 1 "500R" V 12200 11650 50  0000 C CNN
-F 2 "" V 12130 11650 50  0000 C CNN
+F 2 "Resistors_THT:R_Axial_DIN0207_L6.3mm_D2.5mm_P10.16mm_Horizontal" V 12130 11650 50  0001 C CNN
 F 3 "" H 12200 11650 50  0000 C CNN
 	1    12200 11650
@@
 F 0 "Q2" H 4000 18200 50  0000 R CNN
 F 1 "Q_NMOS_DGS" H 4350 18100 50  0000 R CNN
-F 2 "" H 3900 18250 50  0000 C CNN
+F 2 "TO_SOT_Packages_SMD:SOT-323_SC-70_Handsoldering" H 3900 18250 50  0001 C CNN
 F 3 "" H 3700 18150 50  0000 C CNN
 	1    3700 18150
@@
 F 0 "Q3" H 4450 18400 50  0000 R CNN
 F 1 "Q_NMOS_DGS" H 4800 18300 50  0000 R CNN
-F 2 "" H 4350 18450 50  0000 C CNN
+F 2 "TO_SOT_Packages_SMD:SOT-323_SC-70_Handsoldering" H 4350 18450 50  0001 C CNN
 F 3 "" H 4150 18350 50  0000 C CNN
 	1    4150 18350

Commit message: smd resistor
Parts:
- R1, R10, R11, R12, R13, R14, R2, R3, R4, R5, R6, R7, R8, R9: footprint Resistors_THT:R_Axial_DIN0207_L6.3mm_D2.5mm_P10.16mm_Horizontal -> Resistors_SMD:R_1206_HandSoldering
Changed lines of the file:
@@
 I2C_TOF_SCL
 $Comp
-L +5V #PWR1
+L +5V #PWR01
 U 1 1 5A6CAF8E
 P 3250 10750
-F 0 "#PWR1" H 3250 10600 50  0001 C CNN
+F 0 "#PWR01" H 3250 10600 50  0001 C CNN
 F 1 "+5V" H 3250 10890 50  0000 C CNN
 F 2 "" H 3250 10750 50  0000 C CNN
@@
 NoConn ~ 4750 12650
 $Comp
-L +3.3V #PWR3
+L +3.3V #PWR02
 U 1 1 5A6CB32D
 P 4250 11800
-F 0 "#PWR3" H 4250 11650 50  0001 C CNN
+F 0 "#PWR02" H 4250 11650 50  0001 C CNN
 F 1 "+3.3V" H 4250 11940 50  0000 C CNN
 F 2 "" H 4250 11800 50  0000 C CNN
@@
 	2400 18450 3950 18450
 $Comp
-L +3.3V #PWR2
+L +3.3V #PWR03
 U 1 1 5A6CC59B
 P 3350 17600
-F 0 "#PWR2" H 3350 17450 50  0001 C CNN
+F 0 "#PWR03" H 3350 17450 50  0001 C CNN
 F 1 "+3.3V" H 3350 17740 50  0000 C CNN
 F 2 "" H 3350 17600 50  0000 C CNN
@@
 	5300 18350 5600 18350
 $Comp
-L GND #PWR9
+L GND #PWR04
 U 1 1 5A6CC78A
 P 6800 18450
-F 0 "#PWR9" H 6800 18200 50  0001 C CNN
+F 0 "#PWR04" H 6800 18200 50  0001 C CNN
 F 1 "GND" H 6800 18300 50  0000 C CNN
 F 2 "" H 6800 18450 50  0000 C CNN
@@
 F 0 "R2" V 2780 17950 50  0000 C CNN
 F 1 "10kR" V 2700 17950 50  0000 C CNN
-F 2 "Resistors_THT:R_Axial_DIN0207_L6.3mm_D2.5mm_P10.16mm_Horizontal" V 2630 17950 50  0001 C CNN
+F 2 "Resistors_SMD:R_1206_HandSoldering" V 2630 17950 50  0001 C CNN
 F 3 "" H 2700 17950 50  0000 C CNN
 	1    2700 17950
@@
 F 0 "R1" V 2630 18200 50  0000 C CNN
 F 1 "10kR" V 2550 18200 50  0000 C CNN
-F 2 "Resistors_THT:R_Axial_DIN0207_L6.3mm_D2.5mm_P10.16mm_Horizontal" V 2480 18200 50  0001 C CNN
+F 2 "Resistors_SMD:R_1206_HandSoldering" V 2480 18200 50  0001 C CNN
 F 3 "" H 2550 18200 50  0000 C CNN
 	1    2550 18200
@@
 F 0 "R3" V 5280 17950 50  0000 C CNN
 F 1 "10kR" V 5200 17950 50  0000 C CNN
-F 2 "Resistors_THT:R_Axial_DIN0207_L6.3mm_D2.5mm_P10.16mm_Horizontal" V 5130 17950 50  0001 C CNN
+F 2 "Resistors_SMD:R_1206_HandSoldering" V 5130 17950 50  0001 C CNN
 F 3 "" H 5200 17950 50  0000 C CNN
 	1    5200 17950
@@
 F 0 "R4" V 5530 18150 50  0000 C CNN
 F 1 "10kR" V 5450 18150 50  0000 C CNN
-F 2 "Resistors_THT:R_Axial_DIN0207_L6.3mm_D2.5mm_P10.16mm_Horizontal" V 5380 18150 50  0001 C CNN
+F 2 "Resistors_SMD:R_1206_HandSoldering" V 5380 18150 50  0001 C CNN
 F 3 "" H 5450 18150 50  0000 C CNN
 	1    5450 18150
@@
 NoConn ~ 11500 4750
 $Comp
-L +3.3V #PWR4
+L +3.3V #PWR05
 U 1 1 5A7641EB
 P 4400 6450
-F 0 "#PWR4" H 4400 6300 50  0001 C CNN
+F 0 "#PWR05" H 4400 6300 50  0001 C CNN
 F 1 "+3.3V" H 4400 6590 50  0000 C CNN
 F 2 "" H 4400 6450 50  0000 C CNN
@@
 	4400 6450 4750 6450
 $Comp
-L GND #PWR8
+L GND #PWR06
 U 1 1 5A764D00
 P 4550 11050
-F 0 "#PWR8" H 4550 10800 50  0001 C CNN
+F 0 "#PWR06" H 4550 10800 50  0001 C CNN
 F 1 "GND" H 4550 10900 50  0000 C CNN
 F 2 "" H 4550 11050 50  0000 C CNN
@@
 	4550 11050 4750 11050
 $Comp
-L GND #PWR6
+L GND #PWR07
 U 1 1 5A7650C8
 P 4500 12250
-F 0 "#PWR6" H 4500 12000 50  0001 C CNN
+F 0 "#PWR07" H 4500 12000 50  0001 C CNN
 F 1 "GND" H 4500 12100 50  0000 C CNN
 F 2 "" H 4500 12250 50  0000 C CNN
@@
 $EndComp
 $Comp
-L GND #PWR7
+L GND #PWR08
 U 1 1 5A7650EA
 P 4500 12450
-F 0 "#PWR7" H 4500 12200 50  0001 C CNN
+F 0 "#PWR08" H 4500 12200 50  0001 C CNN
 F 1 "GND" H 4500 12300 50  0000 C CNN
 F 2 "" H 4500 12450 50  0000 C CNN
@@
 	4500 12450 4750 12450
 $Comp
-L GND #PWR16
+L GND #PWR09
 U 1 1 5A765594
 P 12100 11050
-F 0 "#PWR16" H 12100 10800 50  0001 C CNN
+F 0 "#PWR09" H 12100 10800 50  0001 C CNN
 F 1 "GND" H 12100 10900 50  0000 C CNN
 F 2 "" H 12100 11050 50  0000 C CNN
@@
 NoConn ~ 11850 10850
 $Comp
-L GND #PWR15
+L GND #PWR010
 U 1 1 5A765CB2
 P 11950 9050
-F 0 "#PWR15" H 11950 8800 50  0001 C CNN
+F 0 "#PWR010" H 11950 8800 50  0001 C CNN
 F 1 "GND" H 11950 8900 50  0000 C CNN
 F 2 "" H 11950 9050 50  0000 C CNN
@@
 	11850 9050 11950 9050
 $Comp
-L GND #PWR14
+L GND #PWR011
 U 1 1 5A766182
 P 11950 7850
-F 0 "#PWR14" H 11950 7600 50  0001 C CNN
+F 0 "#PWR011" H 11950 7600 50  0001 C CNN
 F 1 "GND" H 11950 7700 50  0000 C CNN
 F 2 "" H 11950 7850 50  0000 C CNN
@@
 $EndComp
 $Comp
-L GND #PWR20
+L GND #PWR012
 U 1 1 5A77470C
 P 13250 11650
-F 0 "#PWR20" H 13250 11400 50  0001 C CNN
+F 0 "#PWR012" H 13250 11400 50  0001 C CNN
 F 1 "GND" H 13250 11500 50  0000 C CNN
 F 2 "" H 13250 11650 50  0000 C CNN
@@
 $EndComp
 $Comp
-L GND #PWR19
+L GND #PWR013
 U 1 1 5A774732
 P 13250 11450
-F 0 "#PWR19" H 13250 11200 50  0001 C CNN
+F 0 "#PWR013" H 13250 11200 50  0001 C CNN
 F 1 "GND" H 13250 11300 50  0000 C CNN
 F 2 "" H 13250 11450 50  0000 C CNN
@@
 	11850 6050 12800 6050
 $Comp
-L GND #PWR17
+L GND #PWR014
 U 1 1 5A775D6B
 P 12700 6200
-F 0 "#PWR17" H 12700 5950 50  0001 C CNN
+F 0 "#PWR014" H 12700 5950 50  0001 C CNN
 F 1 "GND" H 12700 6050 50  0000 C CNN
 F 2 "" H 12700 6200 50  0000 C CNN
@@
 $EndComp
 $Comp
-L GND #PWR18
+L GND #PWR015
 U 1 1 5A776193
 P 13000 6700
-F 0 "#PWR18" H 13000 6450 50  0001 C CNN
+F 0 "#PWR015" H 13000 6450 50  0001 C CNN
 F 1 "GND" H 13000 6550 50  0000 C CNN
 F 2 "" H 13000 6700 50  0000 C CNN
@@
 F 0 "R10" V 5880 17550 50  0000 C CNN
 F 1 "47kR" V 5800 17550 50  0000 C CNN
-F 2 "Resistors_THT:R_Axial_DIN0207_L6.3mm_D2.5mm_P10.16mm_Horizontal" V 5730 17550 50  0001 C CNN
+F 2 "Resistors_SMD:R_1206_HandSoldering" V 5730 17550 50  0001 C CNN
 F 3 "" H 5800 17550 50  0000 C CNN
 	1    5800 17550
@@
 F 0 "R14" V 6080 17550 50  0000 C CNN
 F 1 "47kR" V 6000 17550 50  0000 C CNN
-F 2 "Resistors_THT:R_Axial_DIN0207_L6.3mm_D2.5mm_P10.16mm_Horizontal" V 5930 17550 50  0001 C CNN
+F 2 "Resistors_SMD:R_1206_HandSoldering" V 5930 17550 50  0001 C CNN
 F 3 "" H 6000 17550 50  0000 C CNN
 	1    6000 17550
@@
 	5900 18450 6050 18450
 $Comp
-L GND #PWR10
+L GND #PWR016
 U 1 1 5A777AFB
 P 6800 19150
-F 0 "#PWR10" H 6800 18900 50  0001 C CNN
+F 0 "#PWR016" H 6800 18900 50  0001 C CNN
 F 1 "GND" H 6800 19000 50  0000 C CNN
 F 2 "" H 6800 19150 50  0000 C CNN
@@
 $EndComp
 $Comp
-L GND #PWR11
+L GND #PWR017
 U 1 1 5A777B2F
 P 6800 19700
-F 0 "#PWR11" H 6800 19450 50  0001 C CNN
+F 0 "#PWR017" H 6800 19450 50  0001 C CNN
 F 1 "GND" H 6800 19550 50  0000 C CNN
 F 2 "" H 6800 19700 50  0000 C CNN
@@
 $EndComp
 $Comp
-L GND #PWR12
+L GND #PWR018
 U 1 1 5A777C23
 P 6800 20350
-F 0 "#PWR12" H 6800 20100 50  0001 C CNN
+F 0 "#PWR018" H 6800 20100 50  0001 C CNN
 F 1 "GND" H 6800 20200 50  0000 C CNN
 F 2 "" H 6800 20350 50  0000 C CNN
@@
 F 0 "R7" V 5580 18950 50  0000 C CNN
 F 1 "47kR" V 5500 18950 50  0000 C CNN
-F 2 "Resistors_THT:R_Axial_DIN0207_L6.3mm_D2.5mm_P10.16mm_Horizontal" V 5430 18950 50  0001 C CNN
+F 2 "Resistors_SMD:R_1206_HandSoldering" V 5430 18950 50  0001 C CNN
 F 3 "" H 5500 18950 50  0000 C CNN
 	1    5500 18950
@@
 F 0 "R11" V 5880 19050 50  0000 C CNN
 F 1 "47kR" V 5800 19050 50  0000 C CNN
-F 2 "Resistors_THT:R_Axial_DIN0207_L6.3mm_D2.5mm_P10.16mm_Horizontal" V 5730 19050 50  0001 C CNN
+F 2 "Resistors_SMD:R_1206_HandSoldering" V 5730 19050 50  0001 C CNN
 F 3 "" H 5800 19050 50  0000 C CNN
 	1    5800 19050
@@
 F 0 "R8" V 5580 19500 50  0000 C CNN
 F 1 "47kR" V 5500 19500 50  0000 C CNN
-F 2 "Resistors_THT:R_Axial_DIN0207_L6.3mm_D2.5mm_P10.16mm_Horizontal" V 5430 19500 50  0001 C CNN
+F 2 "Resistors_SMD:R_1206_HandSoldering" V 5430 19500 50  0001 C CNN
 F 3 "" H 5500 19500 50  0000 C CNN
 	1    5500 19500
@@
 F 0 "R12" V 5880 19600 50  0000 C CNN
 F 1 "47kR" V 5800 19600 50  0000 C CNN
-F 2 "Resistors_THT:R_Axial_DIN0207_L6.3mm_D2.5mm_P10.16mm_Horizontal" V 5730 19600 50  0001 C CNN
+F 2 "Resistors_SMD:R_1206_HandSoldering" V 5730 19600 50  0001 C CNN
 F 3 "" H 5800 19600 50  0000 C CNN
 	1    5800 19600
@@
 F 0 "R9" V 5580 20150 50  0000 C CNN
 F 1 "47kR" V 5500 20150 50  0000 C CNN
-F 2 "Resistors_THT:R_Axial_DIN0207_L6.3mm_D2.5mm_P10.16mm_Horizontal" V 5430 20150 50  0001 C CNN
+F 2 "Resistors_SMD:R_1206_HandSoldering" V 5430 20150 50  0001 C CNN
 F 3 "" H 5500 20150 50  0000 C CNN
 	1    5500 20150
@@
 F 0 "R13" V 5880 20250 50  0000 C CNN
 F 1 "47kR" V 5800 20250 50  0000 C CNN
-F 2 "Resistors_THT:R_Axial_DIN0207_L6.3mm_D2.5mm_P10.16mm_Horizontal" V 5730 20250 50  0001 C CNN
+F 2 "Resistors_SMD:R_1206_HandSoldering" V 5730 20250 50  0001 C CNN
 F 3 "" H 5800 20250 50  0000 C CNN
 	1    5800 20250
@@
 NoConn ~ 4750 7650
 $Comp
-L GND #PWR5
+L GND #PWR019
 U 1 1 5A77E370
 P 4500 7850
-F 0 "#PWR5" H 4500 7600 50  0001 C CNN
+F 0 "#PWR019" H 4500 7600 50  0001 C CNN
 F 1 "GND" H 4500 7700 50  0000 C CNN
 F 2 "" H 4500 7850 50  0000 C CNN
@@
 NoConn ~ 11850 6450
 $Comp
-L PWR_FLAG #FLG1
+L PWR_FLAG #FLG020
 U 1 1 5A783D0E
 P 4500 11800
-F 0 "#FLG1" H 4500 11895 50  0001 C CNN
+F 0 "#FLG020" H 4500 11895 50  0001 C CNN
 F 1 "PWR_FLAG" H 4500 11980 50  0000 C CNN
 F 2 "" H 4500 11800 50  0000 C CNN
@@
 $EndComp
 $Comp
-L GND #PWR13
+L GND #PWR021
 U 1 1 5A792B30
 P 11550 17850
-F 0 "#PWR13" H 11550 17600 50  0001 C CNN
+F 0 "#PWR021" H 11550 17600 50  0001 C CNN
 F 1 "GND" H 11550 17700 50  0000 C CNN
 F 2 "" H 11550 17850 50  0000 C CNN
@@
 F 0 "R5" V 12280 11450 50  0000 C CNN
 F 1 "500R" V 12200 11450 50  0000 C CNN
-F 2 "Resistors_THT:R_Axial_DIN0207_L6.3mm_D2.5mm_P10.16mm_Horizontal" V 12130 11450 50  0001 C CNN
+F 2 "Resistors_SMD:R_1206_HandSoldering" V 12130 11450 50  0001 C CNN
 F 3 "" H 12200 11450 50  0000 C CNN
 	1    12200 11450
@@
 F 0 "R6" V 12280 11650 50  0000 C CNN
 F 1 "500R" V 12200 11650 50  0000 C CNN
-F 2 "Resistors_THT:R_Axial_DIN0207_L6.3mm_D2.5mm_P10.16mm_Horizontal" V 12130 11650 50  0001 C CNN
+F 2 "Resistors_SMD:R_1206_HandSoldering" V 12130 11650 50  0001 C CNN
 F 3 "" H 12200 11650 50  0000 C CNN
 	1    12200 11650
