File: Electronique/Central_ancien/LED.sch (KiCad schematic (older format))
At the start: 4 parts, among them P4 CONN_jacky_led, P5 CONN_LED, Q1 IRF540N, U9 MC34152

Commit message: schéma ok
Connections:
- net labels added: BATT
- net labels removed: +9V
Changed lines of the file:
@@
 	1    0    0    -1
 $EndComp
+Text GLabel 5550 3700 2    60   Input ~ 0
+BATT
 NoConn ~ 5350 3500
 NoConn ~ 4000 3500
 NoConn ~ 5350 3800
 $Comp
-L GND #PWR46
+L GND #PWR049
 U 1 1 5A767FBA
 P 3900 3800
-F 0 "#PWR46" H 3900 3550 50  0001 C CNN
+F 0 "#PWR049" H 3900 3550 50  0001 C CNN
 F 1 "GND" H 3900 3650 50  0000 C CNN
 F 2 "" H 3900 3800 50  0000 C CNN
@@
 $EndComp
 $Comp
-L GND #PWR45
+L GND #PWR050
 U 1 1 5A767FD6
 P 3900 3700
-F 0 "#PWR45" H 3900 3450 50  0001 C CNN
+F 0 "#PWR050" H 3900 3450 50  0001 C CNN
 F 1 "GND" H 3900 3550 50  0000 C CNN
 F 2 "" H 3900 3700 50  0000 C CNN
@@
 Wire Wire Line
 	3900 3800 4000 3800
+Wire Wire Line
+	5350 3700 5550 3700
 Wire Wire Line
 	5350 3600 6000 3600
@@
 	3300 3600 4000 3600
 $Comp
-L GND #PWR44
+L GND #PWR051
 U 1 1 5A768319
 P 3000 3700
-F 0 "#PWR44" H 3000 3450 50  0001 C CNN
+F 0 "#PWR051" H 3000 3450 50  0001 C CNN
 F 1 "GND" H 3000 3550 50  0000 C CNN
 F 2 "" H 3000 3700 50  0000 C CNN
@@
 	3200 3700 3200 3750
 $Comp
-L GND #PWR49
+L GND #PWR052
 U 1 1 5A7685B8
 P 6300 3900
-F 0 "#PWR49" H 6300 3650 50  0001 C CNN
+F 0 "#PWR052" H 6300 3650 50  0001 C CNN
 F 1 "GND" H 6300 3750 50  0000 C CNN
 F 2 "" H 6300 3900 50  0000 C CNN
@@
 $EndComp
 $Comp
-L +5V #PWR48
+L +5V #PWR053
 U 1 1 5A768873
 P 6300 2850
-F 0 "#PWR48" H 6300 2700 50  0001 C CNN
+F 0 "#PWR053" H 6300 2700 50  0001 C CNN
 F 1 "+5V" H 6300 2990 50  0000 C CNN
 F 2 "" H 6300 2850 50  0000 C CNN
@@
 Wire Wire Line
 	6300 3100 6300 3350
-$Comp
-L +9V #PWR47
-U 1 1 5ABD7B5A
-P 5550 3700
-F 0 "#PWR47" H 5550 3550 50  0001 C CNN
-F 1 "+9V" H 5550 3840 50  0000 C CNN
-F 2 "" H 5550 3700 50  0000 C CNN
-F 3 "" H 5550 3700 50  0000 C CNN
-	1    5550 3700
-	0    1    1    0
-$EndComp
-Wire Wire Line
-	5350 3700 5550 3700
 $EndSCHEMATC
