File: Electronique/Central_ancien/Power.sch (KiCad schematic (older format))
At the start: 19 parts, among them P11 CONN_01X02, U2 LM317_SOT223, U3 LM317_SOT223, U5 B_Plug_5mm, U6 B_Plug_5mm, U7 DSN2596, U8 DSN2596

Commit message: schéma ok
Parts:
- removed C5: 10uC, symbol C
- removed R15: 3.3kR, symbol R
- removed R16: 470R, symbol R
- removed R17: 330R, symbol R
- removed R18: 270R, symbol R
- removed U2, U3: LM317_SOT223, symbol LM317_SOT223
- added U2: APE8865U5-28-HF-3, TO_SOT_Packages_SMD:SOT-23-5_HandSoldering, symbol APE8865U5-28-HF-3-RESCUE-central
Connections:
- net labels removed: +9V
- wire segments 54 -> 43
- no-connect marks 0 -> 1
Other:
- note removed: "FIXED!"
Changed lines of the file:
@@
 $EndDescr
 $Comp
-L +5V #PWR022
+L APE8865U5-28-HF-3-RESCUE-central U2
+U 1 1 5A6CA894
+P 8450 2000
+AR Path="/5A6CA894" Ref="U2"  Part="1"
+AR Path="/5A6CA888/5A6CA894" Ref="U2"  Part="1"
+F 0 "U2" H 8150 2250 50  0000 C CNN
+F 1 "APE8865U5-28-HF-3" H 8450 2200 50  0000 C CNN
+F 2 "TO_SOT_Packages_SMD:SOT-23-5_HandSoldering" H 8450 2100 50  0001 C CIN
+F 3 "" H 8450 2000 50  0000 C CNN
+	1    8450 2000
+	1    0    0    -1
+$EndComp
+$Comp
+L +5V #PWR023
 U 1 1 5A6CA927
 P 7100 1650
-F 0 "#PWR022" H 7100 1500 50  0001 C CNN
+F 0 "#PWR023" H 7100 1500 50  0001 C CNN
 F 1 "+5V" H 7100 1790 50  0000 C CNN
 F 2 "" H 7100 1650 50  0000 C CNN
@@
 Wire Wire Line
 	7100 1650 7100 1950
+Wire Wire Line
+	7100 1950 8000 1950
+Wire Wire Line
+	8000 2100 7800 2100
+Wire Wire Line
+	7800 2100 7800 1950
+Connection ~ 7800 1950
+$Comp
+L GND #PWR024
+U 1 1 5A6CA964
+P 8450 2450
+F 0 "#PWR024" H 8450 2200 50  0001 C CNN
+F 1 "GND" H 8450 2300 50  0000 C CNN
+F 2 "" H 8450 2450 50  0000 C CNN
+F 3 "" H 8450 2450 50  0000 C CNN
+	1    8450 2450
+	1    0    0    -1
+$EndComp
+Wire Wire Line
+	8450 2300 8450 2450
 Text GLabel 9200 1950 2    60   Input ~ 0
 +2.8V
+Wire Wire Line
+	8900 1950 9200 1950
+NoConn ~ 8900 2100
 $Comp
 L C C1
@@
 $EndComp
 $Comp
-L GND #PWR023
+L GND #PWR025
 U 1 1 5A6CB546
 P 7400 2550
-F 0 "#PWR023" H 7400 2300 50  0001 C CNN
+F 0 "#PWR025" H 7400 2300 50  0001 C CNN
 F 1 "GND" H 7400 2400 50  0000 C CNN
 F 2 "" H 7400 2550 50  0000 C CNN
@@
 $EndComp
 $Comp
-L GND #PWR024
+L GND #PWR026
 U 1 1 5A6CB560
 P 9100 2550
-F 0 "#PWR024" H 9100 2300 50  0001 C CNN
+F 0 "#PWR026" H 9100 2300 50  0001 C CNN
 F 1 "GND" H 9100 2400 50  0000 C CNN
 F 2 "" H 9100 2550 50  0000 C CNN
@@
 Wire Wire Line
 	9100 2100 9100 1950
+Connection ~ 9100 1950
 Wire Wire Line
 	9100 2400 9100 2550
 Wire Wire Line
 	7400 2050 7400 1950
+Connection ~ 7400 1950
 Wire Wire Line
 	7400 2350 7400 2550
@@
 	1250 2300 1850 2300
 $Comp
-L GND #PWR025
+L GND #PWR027
 U 1 1 5A74E256
 P 1550 1750
-F 0 "#PWR025" H 1550 1500 50  0001 C CNN
+F 0 "#PWR027" H 1550 1500 50  0001 C CNN
 F 1 "GND" H 1550 1600 50  0000 C CNN
 F 2 "" H 1550 1750 50  0000 C CNN
@@
 $EndComp
 $Comp
-L GND #PWR026
+L GND #PWR028
 U 1 1 5A74E280
 P 1550 2500
-F 0 "#PWR026" H 1550 2250 50  0001 C CNN
+F 0 "#PWR028" H 1550 2250 50  0001 C CNN
 F 1 "GND" H 1550 2350 50  0000 C CNN
 F 2 "" H 1550 2500 50  0000 C CNN
@@
 	2500 2300 2500 2500
 $Comp
-L GND #PWR027
+L GND #PWR029
 U 1 1 5A74E3F6
 P 2500 2050
-F 0 "#PWR027" H 2500 1800 50  0001 C CNN
+F 0 "#PWR029" H 2500 1800 50  0001 C CNN
 F 1 "GND" H 2500 1900 50  0000 C CNN
 F 2 "" H 2500 2050 50  0000 C CNN
@@
 $EndComp
 $Comp
-L GND #PWR028
+L GND #PWR030
 U 1 1 5A74E420
 P 2500 2850
-F 0 "#PWR028" H 2500 2600 50  0001 C CNN
+F 0 "#PWR030" H 2500 2600 50  0001 C CNN
 F 1 "GND" H 2500 2700 50  0000 C CNN
 F 2 "" H 2500 2850 50  0000 C CNN
@@
 Connection ~ 2500 2300
 $Comp
-L GND #PWR029
+L GND #PWR031
 U 1 1 5A74E67A
 P 3400 1850
-F 0 "#PWR029" H 3400 1600 50  0001 C CNN
+F 0 "#PWR031" H 3400 1600 50  0001 C CNN
 F 1 "GND" H 3400 1700 50  0000 C CNN
 F 2 "" H 3400 1850 50  0000 C CNN
@@
 $EndComp
 $Comp
-L GND #PWR030
+L GND #PWR032
 U 1 1 5A74E804
 P 3400 2600
-F 0 "#PWR030" H 3400 2350 50  0001 C CNN
+F 0 "#PWR032" H 3400 2350 50  0001 C CNN
 F 1 "GND" H 3400 2450 50  0000 C CNN
 F 2 "" H 3400 2600 50  0000 C CNN
@@
 	3400 2500 3500 2500
 $Comp
-L GND #PWR031
+L GND #PWR033
 U 1 1 5A74EC12
 P 4700 1850
-F 0 "#PWR031" H 4700 1600 50  0001 C CNN
+F 0 "#PWR033" H 4700 1600 50  0001 C CNN
 F 1 "GND" H 4700 1700 50  0000 C CNN
 F 2 "" H 4700 1850 50  0000 C CNN
@@
 $EndComp
 $Comp
-L GND #PWR032
+L GND #PWR034
 U 1 1 5A74ED5A
 P 4700 2600
-F 0 "#PWR032" H 4700 2350 50  0001 C CNN
+F 0 "#PWR034" H 4700 2350 50  0001 C CNN
 F 1 "GND" H 4700 2450 50  0000 C CNN
 F 2 "" H 4700 2600 50  0000 C CNN
@@
 	4700 2500 4700 2600
 $Comp
-L +5V #PWR033
+L +5V #PWR035
 U 1 1 5A74F2CA
 P 5000 1500
-F 0 "#PWR033" H 5000 1350 50  0001 C CNN
+F 0 "#PWR035" H 5000 1350 50  0001 C CNN
 F 1 "+5V" H 5000 1640 50  0000 C CNN
 F 2 "" H 5000 1500 50  0000 C CNN
@@
 	5000 1550 5000 1500
 $Comp
-L PWR_FLAG #FLG034
+L PWR_FLAG #FLG036
 U 1 1 5A74F572
 P 1500 1400
-F 0 "#FLG034" H 1500 1495 50  0001 C CNN
+F 0 "#FLG036" H 1500 1495 50  0001 C CNN
 F 1 "PWR_FLAG" H 1500 1580 50  0000 C CNN
 F 2 "" H 1500 1400 50  0000 C CNN
@@
 $EndComp
 $Comp
-L PWR_FLAG #FLG035
+L PWR_FLAG #FLG037
 U 1 1 5A74F59C
 P 1600 2200
-F 0 "#FLG035" H 1600 2295 50  0001 C CNN
+F 0 "#FLG037" H 1600 2295 50  0001 C CNN
 F 1 "PWR_FLAG" H 1600 2380 50  0000 C CNN
 F 2 "" H 1600 2200 50  0000 C CNN
@@
 $EndComp
 $Comp
-L PWR_FLAG #FLG036
+L PWR_FLAG #FLG038
 U 1 1 5A74F5C6
 P 1600 2450
-F 0 "#FLG036" H 1600 2545 50  0001 C CNN
+F 0 "#FLG038" H 1600 2545 50  0001 C CNN
 F 1 "PWR_FLAG" H 1600 2630 50  0000 C CNN
 F 2 "" H 1600 2450 50  0000 C CNN
@@
 $EndComp
 $Comp
-L GND #PWR037
+L GND #PWR039
 U 1 1 5A77C1FF
 P 5700 2000
-F 0 "#PWR037" H 5700 1750 50  0001 C CNN
+F 0 "#PWR039" H 5700 1750 50  0001 C CNN
 F 1 "GND" H 5700 1850 50  0000 C CNN
 F 2 "" H 5700 2000 50  0000 C CNN
@@
 	5200 2500 5350 2500
 $Comp
-L GND #PWR038
+L GND #PWR040
 U 1 1 5A782A30
 P 5250 2700
-F 0 "#PWR038" H 5250 2450 50  0001 C CNN
+F 0 "#PWR040" H 5250 2450 50  0001 C CNN
 F 1 "GND" H 5250 2550 50  0000 C CNN
 F 2 "" H 5250 2700 50  0000 C CNN
@@
 Text Label 5050 2300 0    60   ~ 0
 Rasp_power
-$Comp
-L LM317_SOT223 U3
-U 1 1 5ABD55CE
-P 8150 2100
-F 0 "U3" H 8150 2400 50  0000 C CNN
-F 1 "LM317_SOT223" H 8200 1850 50  0000 L CNN
-F 2 "" H 8150 2100 50  0000 C CNN
-F 3 "" H 8150 2100 50  0000 C CNN
-	1    8150 2100
-	1    0    0    -1
-$EndComp
-Wire Wire Line
-	7100 1950 7750 1950
-Connection ~ 7400 1950
-Wire Wire Line
-	8550 1950 9200 1950
-Connection ~ 9100 1950
-$Comp
-L R R18
-U 1 1 5ABD5713
-P 8800 2350
-F 0 "R18" V 8880 2350 50  0000 C CNN
-F 1 "270R" V 8800 2350 50  0000 C CNN
-F 2 "" V 8730 2350 50  0000 C CNN
-F 3 "" H 8800 2350 50  0000 C CNN
-	1    8800 2350
-	1    0    0    -1
-$EndComp
-$Comp
-L R R17
-U 1 1 5ABD5756
-P 8150 2850
-F 0 "R17" V 8230 2850 50  0000 C CNN
-F 1 "330R" V 8150 2850 50  0000 C CNN
-F 2 "" V 8080 2850 50  0000 C CNN
-F 3 "" H 8150 2850 50  0000 C CNN
-	1    8150 2850
-	1    0    0    -1
-$EndComp
-$Comp
-L GND #PWR039
-U 1 1 5ABD58D3
-P 8150 3250
-F 0 "#PWR039" H 8150 3000 50  0001 C CNN
-F 1 "GND" H 8150 3100 50  0000 C CNN
-F 2 "" H 8150 3250 50  0000 C CNN
-F 3 "" H 8150 3250 50  0000 C CNN
-	1    8150 3250
-	1    0    0    -1
-$EndComp
-Wire Wire Line
-	8150 3250 8150 3000
-Wire Wire Line
-	8150 2700 8150 2450
-Wire Wire Line
-	8150 2600 8800 2600
-Wire Wire Line
-	8800 2600 8800 2500
-Connection ~ 8150 2600
-Wire Wire Line
-	8800 2200 8800 1950
-Connection ~ 8800 1950
-Text Notes 8500 1750 0    60   ~ 0
-FIXED!
-$Comp
-L LM317_SOT223 U2
-U 1 1 5ABD8063
-P 6900 4150
-F 0 "U2" H 6900 4450 50  0000 C CNN
-F 1 "LM317_SOT223" H 6950 3900 50  0000 L CNN
-F 2 "" H 6900 4150 50  0000 C CNN
-F 3 "" H 6900 4150 50  0000 C CNN
-	1    6900 4150
-	1    0    0    -1
-$EndComp
-Text GLabel 5950 4000 0    60   Input ~ 0
-BATT
-Wire Wire Line
-	5950 4000 6500 4000
-$Comp
-L +9V #PWR040
-U 1 1 5ABD83E3
-P 7900 4000
-F 0 "#PWR040" H 7900 3850 50  0001 C CNN
-F 1 "+9V" H 7900 4140 50  0000 C CNN
-F 2 "" H 7900 4000 50  0000 C CNN
-F 3 "" H 7900 4000 50  0000 C CNN
-	1    7900 4000
-	0    1    1    0
-$EndComp
-$Comp
-L GND #PWR041
-U 1 1 5ABD8417
-P 6900 5000
-F 0 "#PWR041" H 6900 4750 50  0001 C CNN
-F 1 "GND" H 6900 4850 50  0000 C CNN
-F 2 "" H 6900 5000 50  0000 C CNN
-F 3 "" H 6900 5000 50  0000 C CNN
-	1    6900 5000
-	1    0    0    -1
-$EndComp
-Wire Wire Line
-	7300 4000 7900 4000
-$Comp
-L R R16
-U 1 1 5ABD8496
-P 7650 4300
-F 0 "R16" V 7730 4300 50  0000 C CNN
-F 1 "470R" V 7650 4300 50  0000 C CNN
-F 2 "" V 7580 4300 50  0000 C CNN
-F 3 "" H 7650 4300 50  0000 C CNN
-	1    7650 4300
-	1    0    0    -1
-$EndComp
-$Comp
-L R R15
-U 1 1 5ABD84F7
-P 6900 4800
-F 0 "R15" V 6980 4800 50  0000 C CNN
-F 1 "3.3kR" V 6900 4800 50  0000 C CNN
-F 2 "" V 6830 4800 50  0000 C CNN
-F 3 "" H 6900 4800 50  0000 C CNN
-	1    6900 4800
-	1    0    0    -1
-$EndComp
-Wire Wire Line
-	6900 4650 6900 4500
-Wire Wire Line
-	6900 5000 6900 4950
-Wire Wire Line
-	6900 4600 7650 4600
-Wire Wire Line
-	7650 4600 7650 4450
-Connection ~ 6900 4600
-Wire Wire Line
-	7650 4150 7650 4000
-Connection ~ 7650 4000
-$Comp
-L C C5
-U 1 1 5ABE132F
-P 4950 2950
-F 0 "C5" H 4975 3050 50  0000 L CNN
-F 1 "10uC" H 4975 2850 50  0000 L CNN
-F 2 "" H 4988 2800 50  0000 C CNN
-F 3 "" H 4950 2950 50  0000 C CNN
-	1    4950 2950
-	1    0    0    -1
-$EndComp
-$Comp
-L GND #PWR042
-U 1 1 5ABE142E
-P 4950 3150
-F 0 "#PWR042" H 4950 2900 50  0001 C CNN
-F 1 "GND" H 4950 3000 50  0000 C CNN
-F 2 "" H 4950 3150 50  0000 C CNN
-F 3 "" H 4950 3150 50  0000 C CNN
-	1    4950 3150
-	1    0    0    -1
-$EndComp
-Wire Wire Line
-	4950 2800 4950 2300
-Connection ~ 4950 2300
-Wire Wire Line
-	4950 3150 4950 3100
 $EndSCHEMATC
