File: Electronique/Central_ancien/central.sch (KiCad schematic (older format))
At the start: 35 parts, among them P1 CONN_02X03, P10 CONN_Selec, P12 CONN_01X02, P13 CONN_01X02, P14 CONN_01X02, P15 CONN_01X02, P6 CONN_02X03, P7 CONN_02X03, P8 CONN_02X03, P9 CONN_jack_start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

Commit message: schéma ok
Parts:
- removed Q2, Q3: Q_NMOS_DGS, symbol Q_NMOS_DGS
- removed R5, R6: 500R, symbol R
- added U3: I2C_repeater, Housings_SOIC:SOIC-8_3.9x4.9mm_Pitch1.27mm, symbol I2C_repeater
Connections:
- net labels added: I2C_TOF_EN
- wire segments 119 -> 117
- no-connect marks 60 -> 59
Other:
- note added: "PCA9515"
- note removed: "FIXED!"
- note removed: "Use BSS138"
- moved on the sheet: D3, R1, R2
